File: tragiclaser-phy/bootconfig.sch (KiCad schematic (older format))
At the start: 15 parts, among them U1 XC6SLX25-2FTG256C, U3 DNP, U4 100 MHz

Commit message: Began layout on TRAGICLASER PHY
Parts:
- C1, C2: footprint (none) -> azonenberg_pcb:EIA_0402_CAP_NOSILK
- R19, R20, R21, R22, R23, R24, R25, R26, R27, R28: footprint (none) -> azonenberg_pcb:EIA_0402_RES_NOSILK
- U1: footprint (none) -> azonenberg_pcb:BGA_256_17x17_FULLARRAY_1MM
- U3: footprint (none) -> azonenberg_pcb:SOIC_8_3.9MM
- U4: footprint (none) -> azonenberg_pcb:OSCILLATOR_3.2x2.5
Changed lines of the file:
@@
 Sheet 5 5
 Title "TRAGICLASER Ethernet PHY Prototype"
-Date "2017-09-27"
+Date "2017-09-28"
 Rev "0.1"
 Comp "Andrew Zonenberg"
@@
 F 0 "U1" H 2100 7037 60  0000 C CNN
 F 1 "XC6SLX25-2FTG256C" H 2100 6931 60  0000 C CNN
-F 2 "" H 2100 3850 60  0000 C CNN
+F 2 "azonenberg_pcb:BGA_256_17x17_FULLARRAY_1MM" H 2100 3850 60  0001 C CNN
 F 3 "" H 2100 3850 60  0000 C CNN
 	3    2100 3850
@@
 F 0 "U3" H 7400 2037 60  0000 C CNN
 F 1 "DNP" H 7400 1931 60  0000 C CNN
-F 2 "" H 7400 1350 60  0000 C CNN
+F 2 "azonenberg_pcb:SOIC_8_3.9MM" H 7400 1350 60  0001 C CNN
 F 3 "" H 7400 1350 60  0000 C CNN
 	1    7400 1350
@@
 F 0 "R21" V 3650 1650 50  0000 C CNN
 F 1 "0" V 3700 1850 50  0000 C CNN
-F 2 "" V 3630 1850 50  0000 C CNN
+F 2 "azonenberg_pcb:EIA_0402_RES_NOSILK" V 3630 1850 50  0001 C CNN
 F 3 "" H 3700 1850 50  0000 C CNN
 	1    3700 1850
@@
 F 0 "R20" V 3600 950 50  0000 C CNN
 F 1 "0" V 3650 1150 50  0000 C CNN
-F 2 "" V 3580 1150 50  0000 C CNN
+F 2 "azonenberg_pcb:EIA_0402_RES_NOSILK" V 3580 1150 50  0001 C CNN
 F 3 "" H 3650 1150 50  0000 C CNN
 	1    3650 1150
@@
 F 0 "R24" V 6300 850 50  0000 C CNN
 F 1 "DNP" V 6350 1050 50  0000 C CNN
-F 2 "" V 6280 1050 50  0000 C CNN
+F 2 "azonenberg_pcb:EIA_0402_RES_NOSILK" V 6280 1050 50  0001 C CNN
 F 3 "" H 6350 1050 50  0000 C CNN
 	1    6350 1050
@@
 F 0 "R23" V 6300 750 50  0000 C CNN
 F 1 "DNP" V 6350 950 50  0000 C CNN
-F 2 "" V 6280 950 50  0000 C CNN
+F 2 "azonenberg_pcb:EIA_0402_RES_NOSILK" V 6280 950 50  0001 C CNN
 F 3 "" H 6350 950 50  0000 C CNN
 	1    6350 950
@@
 F 0 "R25" V 6300 950 50  0000 C CNN
 F 1 "DNP" V 6350 1150 50  0000 C CNN
-F 2 "" V 6280 1150 50  0000 C CNN
+F 2 "azonenberg_pcb:EIA_0402_RES_NOSILK" V 6280 1150 50  0001 C CNN
 F 3 "" H 6350 1150 50  0000 C CNN
 	1    6350 1150
@@
 F 0 "C2" H 6515 1446 50  0000 L CNN
 F 1 "DNP" H 6515 1355 50  0000 L CNN
-F 2 "" H 6438 1250 50  0000 C CNN
+F 2 "azonenberg_pcb:EIA_0402_CAP_NOSILK" H 6438 1250 50  0001 C CNN
 F 3 "" H 6400 1400 50  0000 C CNN
 	1    6400 1400
@@
 F 0 "U4" H 7425 3087 60  0000 C CNN
 F 1 "100 MHz" H 7425 2981 60  0000 C CNN
-F 2 "" H 7450 2800 60  0000 C CNN
+F 2 "azonenberg_pcb:OSCILLATOR_3.2x2.5" H 7450 2800 60  0001 C CNN
 F 3 "" H 7450 2800 60  0000 C CNN
 	1    7450 2800
@@
 F 0 "C1" H 6465 3096 50  0000 L CNN
 F 1 "0.47 uF" H 6465 3005 50  0000 L CNN
-F 2 "" H 6388 2900 50  0000 C CNN
+F 2 "azonenberg_pcb:EIA_0402_CAP_NOSILK" H 6388 2900 50  0001 C CNN
 F 3 "" H 6350 3050 50  0000 C CNN
 	1    6350 3050
@@
 F 0 "R28" V 8400 2600 50  0000 C CNN
 F 1 "33" V 8450 2800 50  0000 C CNN
-F 2 "" V 8380 2800 50  0000 C CNN
+F 2 "azonenberg_pcb:EIA_0402_RES_NOSILK" V 8380 2800 50  0001 C CNN
 F 3 "" H 8450 2800 50  0000 C CNN
 	1    8450 2800
@@
 F 0 "R26" V 8400 850 50  0000 C CNN
 F 1 "DNP" V 8450 1050 50  0000 C CNN
-F 2 "" V 8380 1050 50  0000 C CNN
+F 2 "azonenberg_pcb:EIA_0402_RES_NOSILK" V 8380 1050 50  0001 C CNN
 F 3 "" H 8450 1050 50  0000 C CNN
 	1    8450 1050
@@
 F 0 "R27" V 8400 1050 50  0000 C CNN
 F 1 "DNP" V 8450 1250 50  0000 C CNN
-F 2 "" V 8380 1250 50  0000 C CNN
+F 2 "azonenberg_pcb:EIA_0402_RES_NOSILK" V 8380 1250 50  0001 C CNN
 F 3 "" H 8450 1250 50  0000 C CNN
 	1    8450 1250
@@
 F 0 "R19" V 3600 850 50  0000 C CNN
 F 1 "DNP" V 3650 1050 50  0000 C CNN
-F 2 "" V 3580 1050 50  0000 C CNN
+F 2 "azonenberg_pcb:EIA_0402_RES_NOSILK" V 3580 1050 50  0001 C CNN
 F 3 "" H 3650 1050 50  0000 C CNN
 	1    3650 1050
@@
 F 0 "R22" V 3650 4450 50  0000 C CNN
 F 1 "4.7k" V 3700 4650 50  0000 C CNN
-F 2 "" V 3630 4650 50  0000 C CNN
+F 2 "azonenberg_pcb:EIA_0402_RES_NOSILK" V 3630 4650 50  0001 C CNN
 F 3 "" H 3700 4650 50  0000 C CNN
 	1    3700 4650
