File: tragiclaser-phy/fpga-support.sch (KiCad schematic (older format))
At the start: 5 parts, among them J1 XILINX_JTAG, U1 XC6SLX25-2FTG256C

Commit message: Began layout on TRAGICLASER PHY
Parts:
- D1: footprint (none) -> azonenberg_pcb:EIA_0603_LED
- J1: footprint (none) -> azonenberg_pcb:XILINX_JTAG_PTH_MOLEX_0878311420
- R1, R2: footprint (none) -> azonenberg_pcb:EIA_0402_RES_NOSILK
- U1: footprint (none) -> azonenberg_pcb:BGA_256_17x17_FULLARRAY_1MM
Changed lines of the file:
@@
 Sheet 2 5
 Title "TRAGICLASER Ethernet PHY Prototype"
-Date "2017-09-27"
+Date "2017-09-28"
 Rev "0.1"
 Comp "Andrew Zonenberg"
@@
 F 0 "U1" H 4650 7187 60  0000 C CNN
 F 1 "XC6SLX25-2FTG256C" H 4650 7081 60  0000 C CNN
-F 2 "" H 4650 4000 60  0000 C CNN
+F 2 "azonenberg_pcb:BGA_256_17x17_FULLARRAY_1MM" H 4650 4000 60  0001 C CNN
 F 3 "" H 4650 4000 60  0000 C CNN
 	5    4650 4000
@@
 F 0 "J1" H 2718 2908 60  0000 L CNN
 F 1 "XILINX_JTAG" H 2718 2802 60  0000 L CNN
-F 2 "" H 2000 2200 60  0000 C CNN
+F 2 "azonenberg_pcb:XILINX_JTAG_PTH_MOLEX_0878311420" H 2000 2200 60  0001 C CNN
 F 3 "" H 2000 2200 60  0000 C CNN
 	1    2000 2200
@@
 F 0 "R1" V 1600 2800 50  0000 C CNN
 F 1 "470" V 1700 2800 50  0000 C CNN
-F 2 "" V 1630 2800 50  0000 C CNN
+F 2 "azonenberg_pcb:EIA_0402_RES_NOSILK" V 1630 2800 50  0001 C CNN
 F 3 "" H 1700 2800 50  0000 C CNN
 	1    1700 2800
@@
 F 0 "D1" H 1291 3016 50  0000 C CNN
 F 1 "GREEN" H 1291 2925 50  0000 C CNN
-F 2 "" H 1300 2800 50  0000 C CNN
+F 2 "azonenberg_pcb:EIA_0603_LED" H 1300 2800 50  0001 C CNN
 F 3 "" H 1300 2800 50  0000 C CNN
 	1    1300 2800
@@
 F 0 "R2" V 1600 3100 50  0000 C CNN
 F 1 "1k" V 1700 3100 50  0000 C CNN
-F 2 "" V 1630 3100 50  0000 C CNN
+F 2 "azonenberg_pcb:EIA_0402_RES_NOSILK" V 1630 3100 50  0001 C CNN
 F 3 "" H 1700 3100 50  0000 C CNN
 	1    1700 3100
