File: pic32mx-jtag/pic32mx-jtag.kicad_pcb (KiCad board)
At the start: 4 copper layers, 73 x 54 mm, 40 parts, among them J1 BARREL_JACK, J10 U.FL, J2 CONN_01X05, J3 PMOD_HOST, J4 PMOD_HOST, J5 PMOD_HOST, J6 XILINX_JTAG, J7 PMOD_HOST, J8 CONN_01X03, J9 U.FL, U1 PIC32MX6xxFxxxH, U2 LDO1117-33_SOT223

Commit message: Finished v0.1 of pic32mx-jtag
Parts:
- added G***: LOGO, azonenberg_pcb:LONGTHING-1200DPI, F.Cu at (63.0, 112.0)
- moved J10 46.5 mm to (107.0, 102.3), turned to -90 degrees
- moved R2 29.2 mm to (97.3, 91.8), turned to 90 degrees
- moved C10 25.9 mm to (100.8, 100.8)
- moved C5 24.5 mm to (102.0, 102.3)
- moved C7 21.3 mm to (98.2, 91.8), turned to -90 degrees
- moved C1 20.8 mm to (85.2, 94.7)
- moved C11 20.2 mm to (92.5, 108.0)
- moved C9 19.6 mm to (63.4, 95.2), turned to 90 degrees
- moved R1 18.3 mm to (93.8, 92.5), turned to 90 degrees
- moved C6 15.3 mm to (92.5, 93.8)
- moved C3 12.9 mm to (63.1, 99.5), turned to -90 degrees
- moved C8 12.5 mm to (90.3, 108.8), turned to -90 degrees
- moved C4 11.8 mm to (85.8, 98.5), turned to -90 degrees
- moved R4 11.2 mm to (83.5, 100.9)
- moved J9 11.2 mm to (76.1, 96.5), turned to 90 degrees
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Connections:
- C7 pad 1: Net-(C7-Pad1) -> /MCLR_EXT
- J2 pad 1: /MCLR -> /MCLR_EXT
- J4 pad 1: /GPIO4 -> /GPIO14
- J4 pad 10: /GPIO9 -> /GPIO21
- J4 pad 2: /GPIO5 -> /GPIO15
- J4 pad 3: /I2C_SCL -> /GPIO16
- J4 pad 4: /I2C_SDA -> /GPIO17
- J4 pad 7: /GPIO6 -> /GPIO18
- J4 pad 8: /GPIO7 -> /GPIO19
- J4 pad 9: /GPIO8 -> /GPIO20
- J5 pad 1: /PUART_CTS -> /GPIO4
- J5 pad 10: /GPIO13 -> /GPIO9
- J5 pad 2: /PUART_TXD -> /GPIO5
- J5 pad 3: /PUART_RXD -> /I2C_SCL
- J5 pad 4: /PUART_RTS -> /I2C_SDA
- J5 pad 7: /GPIO10 -> /GPIO6
- J5 pad 8: /GPIO11 -> /GPIO7
- J5 pad 9: /GPIO12 -> /GPIO8
- J7 pad 1: /GPIO14 -> /PUART_CTS
- J7 pad 10: /GPIO21 -> /GPIO13
- J7 pad 2: /GPIO15 -> /PUART_TXD
- J7 pad 3: /GPIO16 -> /PUART_RXD
- J7 pad 4: /GPIO17 -> /PUART_RTS
- J7 pad 7: /GPIO18 -> /GPIO10
- J7 pad 8: /GPIO19 -> /GPIO11
- J7 pad 9: /GPIO20 -> /GPIO12
- R1 pad 2: Net-(C7-Pad1) -> /MCLR_EXT
- R2 pad 2: Net-(C7-Pad1) -> /MCLR_EXT
- U1 pad 1: /GPIO13 -> /GPIO6
- U1 pad 11: unconnected-(U1-Pad11) -> /GPIO17
- U1 pad 12: unconnected-(U1-Pad12) -> /GPIO20
- U1 pad 13: unconnected-(U1-Pad13) -> /GPIO16
- U1 pad 14: /GPIO21 -> /GPIO19
- U1 pad 17: unconnected-(U1-Pad17) -> /GPIO18
- U1 pad 18: unconnected-(U1-Pad18) -> /GPIO14
- U1 pad 2: /GPIO2 -> /GPIO4
- U1 pad 22: unconnected-(U1-Pad22) -> /GPIO15
- U1 pad 3: /GPIO3 -> /GPIO21
- U1 pad 30: unconnected-(U1-Pad30) -> /LED0
- U1 pad 33: /GPIO18 -> /LED1
- U1 pad 34: /3V3 -> unconnected-(U1-Pad34)
- U1 pad 36: /GPIO15 -> /LED2
- U1 pad 37: /GPIO14 -> /LED3
- U1 pad 39: /LED0 -> /GPIO3
- U1 pad 40: /LED3 -> /GPIO2
- U1 pad 42: /GPIO8 -> /GPIO1
- U1 pad 44: /GPIO1 -> /GPIO0
- U1 pad 45: /GPIO9 -> /GPIO13
- U1 pad 46: /GPIO0 -> /GPIO12
- U1 pad 47: /LED1 -> /GPIO11
- U1 pad 48: /LED2 -> /GPIO10
- U1 pad 52: /GPIO4 -> unconnected-(U1-Pad52)
- U1 pad 53: /GPIO5 -> unconnected-(U1-Pad53)
- U1 pad 54: /GPIO6 -> unconnected-(U1-Pad54)
- U1 pad 55: /GPIO7 -> unconnected-(U1-Pad55)
- U1 pad 58: /GPIO16 -> unconnected-(U1-Pad58)
- U1 pad 59: /GPIO17 -> unconnected-(U1-Pad59)
- U1 pad 60: /GPIO19 -> unconnected-(U1-Pad60)
- U1 pad 61: /GPIO20 -> /GPIO9
- U1 pad 62: /GPIO10 -> /GPIO8
- U1 pad 63: /GPIO11 -> /GPIO7
- U1 pad 64: /GPIO12 -> /GPIO5
Routing:
- net /GND: track 0.00 -> 282.4 mm, vias 0 -> 16
- net /3V3: track 0.00 -> 244.8 mm, vias 0 -> 19
- net /LED0: track 0.00 -> 40.7 mm, vias 0 -> 2
- net /LED1: track 0.00 -> 39.1 mm, vias 0 -> 2
- net /JTAG_TDI: track 0.00 -> 38.0 mm
- net /LED2: track 0.00 -> 37.6 mm, vias 0 -> 2
- net /JTAG_TMS: track 0.00 -> 36.5 mm
- net /JTAG_TCK: track 0.00 -> 36.5 mm
- net /JTAG_TDO: track 0.00 -> 36.4 mm
- net /LED3: track 0.00 -> 34.7 mm, vias 0 -> 2
- net /UART_RX: track 0.00 -> 30.8 mm, vias 0 -> 1
- net /UART_TX: track 0.00 -> 28.2 mm, vias 0 -> 1
- net /PGD: track 0.00 -> 28.2 mm, vias 0 -> 1
- net /GPIO3: track 0.00 -> 27.6 mm, vias 0 -> 1
- net /PGC: track 0.00 -> 27.3 mm, vias 0 -> 1
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- added copper zone on In2.Cu, net /3V3
- added copper zone on In1.Cu, net /GND
Other:
- board text added: "3V3"
- board text added: "5V DC"
- board text added: "CS#"
- board text added: "CTS"
- board text added: "GND"
- board text added: "JTAG"
- board text added: "LED0"
- board text added: "LED1"
- board text added: "LED2"
- board text added: "LED3"
- board text added: "MCLR"
- board text added: "PGC"
- board text added: "PGD"
- board text added: "PIC32MX6xx JTAG Dev Board A. Zonenberg / v0.1 2022-03-28"
- board text added: "RTS"
- board text added: "RX"
- board text added: "SCK"
- board text added: "SCL"
- board text added: "SDA"
- board text added: "SI"
- board text added: "SO"
- board text added: "TX"
- board text added: "VCORE"
