File: pic32mx-jtag/pic32mx-jtag.kicad_sch (KiCad schematic)
At the start: 36 parts, among them J1 BARREL_JACK, J10 U.FL, J2 CONN_01X05, J3 PMOD_HOST, J4 PMOD_HOST, J5 PMOD_HOST, J6 XILINX_JTAG, J7 PMOD_HOST, J8 CONN_01X03, J9 U.FL, U1 PIC32MX6xxFxxxH, U2 LDO1117-33_SOT223

Commit message: Finished v0.1 of pic32mx-jtag
Connections:
- net 3V3: no longer U1.34 (VBUS)
- net GPIO0: now also U1.44 (RD10); no longer U1.46 (RD0)
- net GPIO1: now also U1.42 (RD8); no longer U1.44 (RD10)
- net GPIO10: now also J7.7 (D4), U1.48 (RC14); no longer J5.7 (D4), U1.62 (RE2)
- net GPIO11: now also J7.8 (D5), U1.47 (RC13); no longer J5.8 (D5), U1.63 (RE3)
- net GPIO12: now also J7.9 (D6), U1.46 (RD0); no longer J5.9 (D6), U1.64 (RE4)
- net GPIO13: now also J7.10 (D7), U1.45 (RD11); no longer J5.10 (D7), U1.1 (RE5)
- net GPIO14: now also J4.1 (D0), U1.18 (RB7); no longer J7.1 (D0), U1.37 (RG2)
- net GPIO15: now also J4.2 (D1), U1.22 (RB9); no longer J7.2 (D1), U1.36 (RG3)
- net GPIO16: now also J4.3 (D2), U1.13 (RB3); no longer J7.3 (D2), U1.58 (RF0)
- net GPIO17: now also J4.4 (D3), U1.11 (RB5); no longer J7.4 (D3), U1.59 (RF1)
- net GPIO18: now also J4.7 (D4), U1.17 (RB6); no longer J7.7 (D4), U1.33 (RF3)
- net GPIO19: now also J4.8 (D5), U1.14 (RB2); no longer J7.8 (D5), U1.60 (RE0)
- net GPIO2: now also U1.40 (RC15); no longer U1.2 (RE6)
- net GPIO20: now also J4.9 (D6), U1.12 (RB4); no longer J7.9 (D6), U1.61 (RE1)
- net GPIO21: now also J4.10 (D7), U1.3 (RE7); no longer J7.10 (D7), U1.14 (RB2)
- net GPIO3: now also U1.39 (RC12); no longer U1.3 (RE7)
- net GPIO4: now also J5.1 (D0), U1.2 (RE6); no longer J4.1 (D0), U1.52 (RD4)
- net GPIO5: now also J5.2 (D1), U1.64 (RE4); no longer J4.2 (D1), U1.53 (RD5)
- net GPIO6: now also J5.7 (D4), U1.1 (RE5); no longer J4.7 (D4), U1.54 (RD6)
- net GPIO7: now also J5.8 (D5), U1.63 (RE3); no longer J4.8 (D5), U1.55 (RD7)
- net GPIO8: now also J5.9 (D6), U1.62 (RE2); no longer J4.9 (D6), U1.42 (RD8)
- net GPIO9: now also J5.10 (D7), U1.61 (RE1); no longer J4.10 (D7), U1.45 (RD11)
- net I2C_SCL: now also J5.3 (D2); no longer J4.3 (D2)
- net I2C_SDA: now also J5.4 (D3); no longer J4.4 (D3)
- net LED0: now also U1.30 (RB15); no longer U1.39 (RC12)
- net LED1: now also U1.33 (RF3); no longer U1.47 (RC13)
- net LED2: now also U1.36 (RG3); no longer U1.48 (RC14)
- net LED3: now also U1.37 (RG2); no longer U1.40 (RC15)
- net MCLR: no longer J2.1 (P1)
- net PUART_CTS: now also J7.1 (D0); no longer J5.1 (D0)
- net PUART_RTS: now also J7.4 (D3); no longer J5.4 (D3)
- net PUART_RXD: now also J7.3 (D2); no longer J5.3 (D2)
- net PUART_TXD: now also J7.2 (D1); no longer J5.2 (D1)
- net MCLR_EXT: now reaches C7.1, R1.2, R2.2
- net MCLR_EXT: now also J2.1 (P1)
- no-connect marks 10 -> 11
Other:
- moved on the sheet: J4, J5, J7
