File: baset1-media-converter/baset-phy.kicad_sch (KiCad schematic)
At the start: 63 parts, among them J3 0826-1G1T-23-F, U4 KSZ9031RN, U5 ECS-1612MV-250-CN, U6 RCLAMP0514M, U7 RCLAMP0514M

Commit message: Continued layout on media converter
Parts:
- removed TP16: U.FL, azonenberg_pcb:CONN_U.FL_TE_1909763-1, symbol conn:CONN_COAXIAL
Changed lines of the file:
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@@
   (title_block
     (title "BaseT to BaseT1 Media Converter")
-    (date "2024-01-25")
+    (date "2024-01-27")
     (rev "0.1")
     (company "Antikernel Labs")
@@
   (junction (at 97.79 26.67) (diameter 0) (color 0 0 0 0)
   )
-  (junction (at 111.76 184.15) (diameter 0) (color 0 0 0 0)
-  )
   (junction (at 83.82 184.15) (diameter 0) (color 0 0 0 0)
   )
@@
   )
   (junction (at 60.96 171.45) (diameter 0) (color 0 0 0 0)
-  )
-  (junction (at 111.76 191.77) (diameter 0) (color 0 0 0 0)
   )
   (junction (at 69.85 191.77) (diameter 0) (color 0 0 0 0)
@@
     (stroke (width 0) (type default) (color 0 0 0 0))
   )
-  (wire (pts (xy 127 191.77) (xy 127 189.23))
-    (stroke (width 0) (type default) (color 0 0 0 0))
-  )
   (wire (pts (xy 171.45 29.21) (xy 154.94 29.21))
     (stroke (width 0) (type default) (color 0 0 0 0))
@@
     (stroke (width 0) (type default) (color 0 0 0 0))
   )
-  (wire (pts (xy 111.76 191.77) (xy 127 191.77))
-    (stroke (width 0) (type default) (color 0 0 0 0))
-  )
   (wire (pts (xy 127 163.83) (xy 139.7 163.83))
     (stroke (width 0) (type default) (color 0 0 0 0))
@@
   )
   (wire (pts (xy 53.34 71.12) (xy 45.72 71.12))
-    (stroke (width 0) (type default) (color 0 0 0 0))
-  )
-  (wire (pts (xy 111.76 184.15) (xy 123.19 184.15))
     (stroke (width 0) (type default) (color 0 0 0 0))
   )
@@
     (pin "9")
   )
-  (symbol (lib_id "conn:CONN_COAXIAL") (at 127 184.15 0) (unit 1)
-    (in_bom yes) (on_board yes) (fields_autoplaced)
-    (property "Reference" "TP16" (id 0) (at 129.5401 183.6085 0)
-      (effects (font (size 1.27 1.27)) (justify left))
-    )
-    (property "Value" "U.FL" (id 1) (at 129.5401 186.1454 0)
-      (effects (font (size 1.27 1.27)) (justify left))
-    )
-    (property "Footprint" "azonenberg_pcb:CONN_U.FL_TE_1909763-1" (id 2) (at 127 184.15 0)
-      (effects (font (size 1.27 1.27)) hide)
-    )
-    (property "Datasheet" "" (id 3) (at 127 184.15 0)
-      (effects (font (size 1.27 1.27)) hide)
-    )
-    (pin "1")
-    (pin "2")
-  )
   (symbol (lib_id "device:C") (at 44.45 113.03 0) (unit 1)
