File: baset1-media-converter/psu.kicad_sch (KiCad schematic)
At the start: 22 parts, among them U3 LTC3374-QFN

Commit message: Updating file: baset1-media-converter.kicad_pcb with current fully routed design
Connections:
- net GND: now also C62.2, C63.2, C64.2, C65.2
Changed lines of the file:
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@@
   (title_block
     (title "BaseT to BaseT1 Media Converter")
-    (date "2024-01-27")
+    (date "2024-01-28")
     (rev "0.1")
     (company "Antikernel Labs")
@@
     (stroke (width 0) (type default) (color 0 0 0 0))
   )
+  (label "GND" (at 135.89 55.88 180)
+    (effects (font (size 1.27 1.27)) (justify right bottom))
+  )
   (label "5V0" (at 135.89 48.26 180)
