File: baset1-media-converter/baset1-media-converter.kicad_pcb (KiCad board)
At the start: 4 copper layers, 100.5 x 62.5 mm, 180 parts, among them J1 CONN_01X05, J2 UX60SX-MB-5ST, J3 0826-1G1T-23-F, J4 CONN_01X02, M1 LOGO, M2 LOGO, M3 LOGO, Q1 SSM6N58NU, U1 STM32F031-QFN28, U10 NCP45521-H, U2 FT234XD, U3 LTC3374-QFN, U4 KSZ9031RN, U5 ECS-1612MV-250-CN, U6 RCLAMP0514M, U7 RCLAMP0514M, U8 DP83TG720S-Q1, U9 ECS-1612MV-250-CN

Commit message: Added note about incorrect FTDI footprint
Other:
- board text added: "FIXME-v0.2 FTDI footprint is 0.5mm, real chip is 0.45"
Changed lines of the file:
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@@
       (primitives
         (gr_poly (pts
-            (xy 0.077 -0.15)
-            (xy -0.275 -0.15)
-            (xy -0.275 0.15)
-            (xy 0.275 0.15)
             (xy 0.275 0.048)
+            (xy 0.275 0.15)
+            (xy -0.275 0.15)
+            (xy -0.275 -0.15)
+            (xy 0.077 -0.15)
           ) (width 0) (fill yes))
       ))
@@
       (primitives
         (gr_poly (pts
-            (xy -0.077 -0.15)
-            (xy 0.275 -0.15)
             (xy 0.275 0.15)
             (xy -0.275 0.15)
             (xy -0.275 0.048)
+            (xy -0.077 -0.15)
+            (xy 0.275 -0.15)
           ) (width 0) (fill yes))
       ))
@@
       (primitives
         (gr_poly (pts
-            (xy 0.077 -0.15)
-            (xy -0.275 -0.15)
-            (xy -0.275 0.15)
-            (xy 0.275 0.15)
             (xy 0.275 0.048)
+            (xy 0.275 0.15)
+            (xy -0.275 0.15)
+            (xy -0.275 -0.15)
+            (xy 0.077 -0.15)
           ) (width 0) (fill yes))
       ))
@@
       (primitives
         (gr_poly (pts
-            (xy -0.077 -0.15)
-            (xy 0.275 -0.15)
             (xy 0.275 0.15)
             (xy -0.275 0.15)
             (xy -0.275 0.048)
+            (xy -0.077 -0.15)
+            (xy 0.275 -0.15)
           ) (width 0) (fill yes))
       ))
@@
       (primitives
         (gr_poly (pts
-            (xy 0.077 -0.15)
-            (xy -0.275 -0.15)
-            (xy -0.275 0.15)
-            (xy 0.275 0.15)
             (xy 0.275 0.048)
+            (xy 0.275 0.15)
+            (xy -0.275 0.15)
+            (xy -0.275 -0.15)
+            (xy 0.077 -0.15)
           ) (width 0) (fill yes))
       ))
@@
       (primitives
         (gr_poly (pts
-            (xy -0.077 -0.15)
-            (xy 0.275 -0.15)
             (xy 0.275 0.15)
             (xy -0.275 0.15)
             (xy -0.275 0.048)
+            (xy -0.077 -0.15)
+            (xy 0.275 -0.15)
           ) (width 0) (fill yes))
       ))
@@
       (primitives
         (gr_poly (pts
-            (xy 0.077 -0.15)
-            (xy -0.275 -0.15)
-            (xy -0.275 0.15)
-            (xy 0.275 0.15)
             (xy 0.275 0.048)
+            (xy 0.275 0.15)
+            (xy -0.275 0.15)
+            (xy -0.275 -0.15)
+            (xy 0.077 -0.15)
           ) (width 0) (fill yes))
       ))
@@
       (primitives
         (gr_poly (pts
-            (xy -0.077 -0.15)
-            (xy 0.275 -0.15)
             (xy 0.275 0.15)
             (xy -0.275 0.15)
             (xy -0.275 0.048)
+            (xy -0.077 -0.15)
+            (xy 0.275 -0.15)
           ) (width 0) (fill yes))
       ))
@@
     (effects (font (size 0.75 0.75) (thickness 0.1)))
   )
+  (gr_text "FIXME-v0.2\nFTDI footprint is 0.5mm, real chip is 0.45" (at 80.5 32.5) (layer "Eco1.User")
+    (effects (font (size 1.5 1.5) (thickness 0.1)) (justify left))
+  )
   (segment (start 111.25 44.83) (end 115.08 41) (width 0.125) (layer "F.Cu") (net 1))
