File: kup-lulz/sfp28.kicad_sch (KiCad schematic)
At the start: 69 parts, among them J10 SFP_CAGE, J11 CONN_SFP_HOST, J12 SFP_CAGE, J33 CONN_SFP_HOST, J34 SFP_CAGE, J7 CONN_SFP_HOST, J8 SFP_CAGE, J9 CONN_SFP_HOST, U9 XILINX_ULTRASCALEPLUS_B676

Commit message: Continued initial work on kup-lulz devboard
Connections:
- net SFP0_RX_N: now also J11.13 (RX_P), U9.P1 (MGTYRXN3_225); no longer J11.12 (RX_N), U9.Y1 (MGTYRXN0_225)
- net SFP0_RX_P: now also J11.12 (RX_N), U9.P2 (MGTYRXP3_225); no longer J11.13 (RX_P), U9.Y2 (MGTYRXP0_225)
- net SFP0_TX_N: now also U9.R4 (MGTYTXN3_225); no longer U9.AA4 (MGTYTXN0_225)
- net SFP0_TX_P: now also U9.R5 (MGTYTXP3_225); no longer U9.AA5 (MGTYTXP0_225)
- net SFP1_RX_N: now also J9.13 (RX_P), U9.T1 (MGTYRXN2_225); no longer J9.12 (RX_N), U9.V1 (MGTYRXN1_225)
- net SFP1_RX_P: now also J9.12 (RX_N), U9.T2 (MGTYRXP2_225); no longer J9.13 (RX_P), U9.V2 (MGTYRXP1_225)
- net SFP1_TX_N: now also U9.U4 (MGTYTXN2_225); no longer U9.W4 (MGTYTXN1_225)
- net SFP1_TX_P: now also U9.U5 (MGTYTXP2_225); no longer U9.W5 (MGTYTXP1_225)
- net SFP2_RX_N: now also J7.13 (RX_P), U9.V1 (MGTYRXN1_225); no longer J7.12 (RX_N), U9.T1 (MGTYRXN2_225)
- net SFP2_RX_P: now also J7.12 (RX_N), U9.V2 (MGTYRXP1_225); no longer J7.13 (RX_P), U9.T2 (MGTYRXP2_225)
- net SFP2_TX_N: now also U9.W4 (MGTYTXN1_225); no longer U9.U4 (MGTYTXN2_225)
- net SFP2_TX_P: now also U9.W5 (MGTYTXP1_225); no longer U9.U5 (MGTYTXP2_225)
- net SFP3_RX_N: now also J33.13 (RX_P), U9.Y1 (MGTYRXN0_225); no longer J33.12 (RX_N), U9.P1 (MGTYRXN3_225)
- net SFP3_RX_P: now also J33.12 (RX_N), U9.Y2 (MGTYRXP0_225); no longer J33.13 (RX_P), U9.P2 (MGTYRXP3_225)
- net SFP3_TX_N: now also U9.AA4 (MGTYTXN0_225); no longer U9.R4 (MGTYTXN3_225)
- net SFP3_TX_P: now also U9.AA5 (MGTYTXP0_225); no longer U9.R5 (MGTYTXP3_225)
- net SFP28_REFCLK1_N: no longer names the net of U9.T6 (MGTREFCLK1N_225)
- net SFP28_REFCLK1_P: no longer names the net of U9.T7 (MGTREFCLK1P_225)
- no-connect marks 0 -> 2
Other:
- note added: "Pair swap for routing"
Changed lines of the file:
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@@
   (title_block
     (title "Kintex Ultrascale+ OshPark For The Lulz")
-    (date "2024-01-31")
+    (date "2024-02-01")
     (rev "0.1")
     (company "Antikernel Labs")
@@
   (junction (at 194.31 46.99) (diameter 0) (color 0 0 0 0)
   )
+  (no_connect (at 208.28 205.74))
+  (no_connect (at 208.28 203.2))
   (wire (pts (xy 284.48 139.7) (xy 262.89 139.7))
     (stroke (width 0) (type default) (color 0 0 0 0))
@@
     (stroke (width 0) (type default) (color 0 0 0 0))
   )
+  (text "Pair swap for routing" (at 101.6 57.15 180)
+    (effects (font (size 1.27 1.27)) (justify right bottom))
+  )
+  (text "Pair swap for routing" (at 260.35 57.15 180)
+    (effects (font (size 1.27 1.27)) (justify right bottom))
+  )
   (text "SFP+ power filtering" (at 334.01 162.56 0)
     (effects (font (size 1.27 1.27)) (justify left bottom))
@@
     (effects (font (size 1.27 1.27)) (justify left bottom))
   )
+  (text "Pair swap for routing" (at 181.61 57.15 180)
+    (effects (font (size 1.27 1.27)) (justify right bottom))
+  )
+  (text "Pair swap for routing" (at 339.09 57.15 180)
+    (effects (font (size 1.27 1.27)) (justify right bottom))
+  )
   (text "SFP+ power filtering" (at 97.79 162.56 0)
     (effects (font (size 1.27 1.27)) (justify left bottom))
@@
     (effects (font (size 1.27 1.27)) (justify right bottom))
   )
-  (label "SFP1_RX_N" (at 273.05 59.69 180)
+  (label "SFP1_RX_N" (at 273.05 57.15 180)
     (effects (font (size 1.27 1.27)) (justify right bottom))
   )
@@
     (effects (font (size 1.27 1.27)) (justify right bottom))
   )
-  (label "SFP2_RX_P" (at 194.31 57.15 180)
-    (effects (font (size 1.27 1.27)) (justify right bottom))
-  )
-  (label "SFP0_RX_N" (at 208.28 220.98 180)
+  (label "SFP2_RX_P" (at 194.31 59.69 180)
+    (effects (font (size 1.27 1.27)) (justify right bottom))
+  )
+  (label "SFP0_RX_N" (at 208.28 243.84 180)
     (effects (font (size 1.27 1.27)) (justify right bottom))
   )
@@
     (effects (font (size 1.27 1.27)) (justify right bottom))
   )
-  (label "SFP2_RX_N" (at 194.31 59.69 180)
-    (effects (font (size 1.27 1.27)) (justify right bottom))
-  )
-  (label "SFP2_RX_N" (at 208.28 236.22 180)
+  (label "SFP2_RX_N" (at 194.31 57.15 180)
+    (effects (font (size 1.27 1.27)) (justify right bottom))
+  )
+  (label "SFP2_RX_N" (at 208.28 228.6 180)
     (effects (font (size 1.27 1.27)) (justify right bottom))
   )
@@
     (effects (font (size 1.27 1.27)) (justify right bottom))
   )
-  (label "SFP3_RX_N" (at 208.28 243.84 180)
+  (label "SFP3_RX_N" (at 208.28 220.98 180)
     (effects (font (size 1.27 1.27)) (justify right bottom))
   )
@@
     (effects (font (size 1.27 1.27)) (justify right bottom))
   )
-  (label "SFP1_RX_P" (at 208.28 226.06 180)
-    (effects (font (size 1.27 1.27)) (justify right bottom))
-  )
-  (label "SFP0_RX_P" (at 208.28 218.44 180)
+  (label "SFP1_RX_P" (at 208.28 233.68 180)
+    (effects (font (size 1.27 1.27)) (justify right bottom))
+  )
+  (label "SFP0_RX_P" (at 208.28 241.3 180)
     (effects (font (size 1.27 1.27)) (justify right bottom))
   )
@@
     (effects (font (size 1.27 1.27)) (justify right bottom))
   )
-  (label "SFP1_RX_N" (at 208.28 228.6 180)
-    (effects (font (size 1.27 1.27)) (justify right bottom))
-  )
-  (label "SFP1_TX_N" (at 208.28 259.08 180)
+  (label "SFP1_RX_N" (at 208.28 236.22 180)
+    (effects (font (size 1.27 1.27)) (justify right bottom))
+  )
+  (label "SFP1_TX_N" (at 208.28 266.7 180)
     (effects (font (size 1.27 1.27)) (justify right bottom))
   )
@@
     (effects (font (size 1.27 1.27)) (justify right bottom))
   )
-  (label "SFP1_RX_P" (at 273.05 57.15 180)
-    (effects (font (size 1.27 1.27)) (justify right bottom))
-  )
-  (label "SFP3_TX_P" (at 208.28 271.78 180)
+  (label "SFP1_RX_P" (at 273.05 59.69 180)
+    (effects (font (size 1.27 1.27)) (justify right bottom))
+  )
+  (label "SFP3_TX_P" (at 208.28 248.92 180)
     (effects (font (size 1.27 1.27)) (justify right bottom))
   )
@@
     (effects (font (size 1.27 1.27)) (justify right bottom))
   )
-  (label "SFP3_TX_N" (at 208.28 274.32 180)
+  (label "SFP3_TX_N" (at 208.28 251.46 180)
     (effects (font (size 1.27 1.27)) (justify right bottom))
   )
@@
     (effects (font (size 1.27 1.27)) (justify right bottom))
   )
-  (label "SFP2_RX_P" (at 208.28 233.68 180)
+  (label "SFP2_RX_P" (at 208.28 226.06 180)
     (effects (font (size 1.27 1.27)) (justify right bottom))
   )
@@
     (effects (font (size 1.27 1.27)) (justify right bottom))
   )
-  (label "SFP2_TX_N" (at 208.28 266.7 180)
-    (effects (font (size 1.27 1.27)) (justify right bottom))
-  )
-  (label "SFP3_RX_P" (at 208.28 241.3 180)
+  (label "SFP2_TX_N" (at 208.28 259.08 180)
+    (effects (font (size 1.27 1.27)) (justify right bottom))
+  )
+  (label "SFP3_RX_P" (at 208.28 218.44 180)
     (effects (font (size 1.27 1.27)) (justify right bottom))
   )
@@
     (effects (font (size 1.27 1.27)) (justify right bottom))
   )
-  (label "SFP0_TX_P" (at 208.28 248.92 180)
-    (effects (font (size 1.27 1.27)) (justify right bottom))
-  )
-  (label "SFP0_RX_P" (at 351.79 57.15 180)
+  (label "SFP0_TX_P" (at 208.28 271.78 180)
+    (effects (font (size 1.27 1.27)) (justify right bottom))
+  )
+  (label "SFP0_RX_P" (at 351.79 59.69 180)
     (effects (font (size 1.27 1.27)) (justify right bottom))
   )
@@
     (effects (font (size 1.27 1.27)) (justify right bottom))
   )
-  (label "SFP0_RX_N" (at 351.79 59.69 180)
+  (label "SFP0_RX_N" (at 351.79 57.15 180)
     (effects (font (size 1.27 1.27)) (justify right bottom))
   )
@@
     (effects (font (size 1.27 1.27)) (justify left bottom))
   )
-  (label "SFP1_TX_P" (at 208.28 256.54 180)
+  (label "SFP1_TX_P" (at 208.28 264.16 180)
     (effects (font (size 1.27 1.27)) (justify right bottom))
   )
@@
     (effects (font (size 1.27 1.27)) (justify right bottom))
   )
-  (label "SFP2_TX_P" (at 208.28 264.16 180)
+  (label "SFP2_TX_P" (at 208.28 256.54 180)
     (effects (font (size 1.27 1.27)) (justify right bottom))
   )
@@
     (effects (font (size 1.27 1.27)) (justify right bottom))
   )
-  (label "SFP3_RX_P" (at 115.57 57.15 180)
+  (label "SFP3_RX_P" (at 115.57 59.69 180)
     (effects (font (size 1.27 1.27)) (justify right bottom))
   )
@@
     (effects (font (size 1.27 1.27)) (justify left bottom))
   )
-  (label "SFP3_RX_N" (at 115.57 59.69 180)
-    (effects (font (size 1.27 1.27)) (justify right bottom))
-  )
-  (label "SFP0_TX_N" (at 208.28 251.46 180)
+  (label "SFP3_RX_N" (at 115.57 57.15 180)
+    (effects (font (size 1.27 1.27)) (justify right bottom))
+  )
+  (label "SFP0_TX_N" (at 208.28 274.32 180)
     (effects (font (size 1.27 1.27)) (justify right bottom))
   )
@@
     (effects (font (size 1.27 1.27)) (justify right))
   )
-  (hierarchical_label "SFP28_REFCLK1_P" (shape input) (at 208.28 203.2 180)
-    (effects (font (size 1.27 1.27)) (justify right))
-  )
   (hierarchical_label "SFP3_RS1" (shape input) (at 115.57 74.93 180)
     (effects (font (size 1.27 1.27)) (justify right))
@@
     (effects (font (size 1.27 1.27)) (justify right))
   )
-  (hierarchical_label "SFP28_REFCLK1_N" (shape input) (at 208.28 205.74 180)
-    (effects (font (size 1.27 1.27)) (justify right))
-  )
