File: kup-lulz/kup-lulz.kicad_pcb (KiCad board)
At the start: 4 copper layers, 144.5 x 137 mm, 229 parts, among them J1 CONN_PCIE_PWR_8PIN, J10 SFP_CAGE, J11 CONN_SFP_HOST, J12 SFP_CAGE, J13 PMOD_HOST, J14 PMOD_HOST, J15 CONN_QSFP_HOST, J16 CONN_QSFP_HOST, J17 SMPM, J18 SMPM, J19 SMPM, J2 CONN_IBC_MGMT, J20 SMPM, J21 SMPM, J22 SMPM, J23 SMPM, J24 SMPM, J25 SMPM, J26 SMPM, J27 SMPM, J28 SMPM, J29 SMPM, J3 CONN_01X03, J30 SMPM, J31 SMPM, J32 SMPM, J33 CONN_SFP_HOST, J34 SFP_CAGE, J35 QSFP_CAGE, J36 QSFP_CAGE, J4 CONN_01X05, J7 CONN_SFP_HOST, J8 SFP_CAGE, J9 CONN_SFP_HOST, M1 HEATSINK, M2 SCREWHOLE, M3 SCREWHOLE, M4 SCREWHOLE, M5 SCREWHOLE, SW1 SWITCH, SW2 SWITCH, U1 STM32L031C6U6, U2 MYMGK1R812ERSR, U3 MYMGK1R812ERSR, U4 MYMGK00506ERSR, U5 MYMGK00504ERSR, U6 MYMGK00504ERSR, U7 MYMGK00504ERSR, U9 XILINX_ULTRASCALEPLUS_B676

Commit message: Continued initial work on kup-lulz devboard
Parts:
- added C118: 0.47 uF, azonenberg_pcb:EIA_0402_CAP_NOSILK, F.Cu at (208.6, 82.8)
- added C119: 0.47 uF, azonenberg_pcb:EIA_0402_CAP_NOSILK, F.Cu at (211.1, 82.8)
- added C120: 0.47 uF, azonenberg_pcb:EIA_0402_CAP_NOSILK, F.Cu at (229.4, 74.3)
- added C121: 0.47 uF, azonenberg_pcb:EIA_0402_CAP_NOSILK, F.Cu at (218.6, 84.3)
- added C122: 0.47 uF, azonenberg_pcb:EIA_0402_CAP_NOSILK, F.Cu at (230.2, 72.5)
- added C123: 0.47 uF, azonenberg_pcb:EIA_0402_CAP_NOSILK, F.Cu at (226.9, 77.3)
- added C124: 4.7 uF, azonenberg_pcb:EIA_0603_CAP_NOSILK, F.Cu at (237.7, 80.0)
- added C125: 4.7 uF, azonenberg_pcb:EIA_0603_CAP_NOSILK, F.Cu at (241.0, 80.0)
- added C126: 0.47 uF, azonenberg_pcb:EIA_0402_CAP_NOSILK, F.Cu at (239.8, 81.6)
- added C127: 0.47 uF, azonenberg_pcb:EIA_0402_CAP_NOSILK, F.Cu at (247.3, 79.8)
- added C128: 0.47 uF, azonenberg_pcb:EIA_0402_CAP_NOSILK, F.Cu at (243.9, 79.8)
- added C129: 0.47 uF, azonenberg_pcb:EIA_0402_CAP_NOSILK, F.Cu at (239.8, 83.1)
- added C130: 0.47 uF, azonenberg_pcb:EIA_0402_CAP_NOSILK, F.Cu at (237.3, 83.1)
- added C131: 0.47 uF, azonenberg_pcb:EIA_0402_CAP_NOSILK, F.Cu at (237.3, 81.6)
- added C132: 0.47 uF, azonenberg_pcb:EIA_0402_CAP_NOSILK, F.Cu at (244.8, 81.3)
- added C133: 0.47 uF, azonenberg_pcb:EIA_0402_CAP_NOSILK, F.Cu at (242.3, 81.6)
- added C40: 4.7 uF, azonenberg_pcb:EIA_0603_CAP_NOSILK, F.Cu at (233.8, 103.2)
- added C41: 4.7 uF, azonenberg_pcb:EIA_0603_CAP_NOSILK, F.Cu at (237.2, 99.4)
- added C59: 4.7 uF, azonenberg_pcb:EIA_0603_CAP_NOSILK, F.Cu at (227.3, 72.7)
- added C60: 0.47 uF, azonenberg_pcb:EIA_0402_CAP_NOSILK, F.Cu at (223.6, 81.3)
- added C81: 0.1 uF, azonenberg_pcb:EIA_0402_CAP_NOSILK, F.Cu at (208.6, 100.7)
- added C82: 0.1 uF, azonenberg_pcb:EIA_0402_CAP_NOSILK, F.Cu at (211.1, 100.7)
- added FB3: MI0603J601R-10, azonenberg_pcb:EIA_0603_INDUCTOR_NOSILK, F.Cu at (256.0, 72.7)
- added J37: XILINX_JTAG, azonenberg_pcb:XILINX_JTAG_PTH_MOLEX_0878311420, F.Cu at (245.2, 75.4)
- added J38: PMOD_HOST, azonenberg_pcb:CONN_HEADER_2.54MM_2x6_RA_PMOD_HOST, F.Cu at (216.8, 112.5)
- added J5: JUMPER_0402, azonenberg_pcb:EIA_0402_JUMPER, F.Cu at (209.1, 79.8)
- added J6: XILINX_JTAG, azonenberg_pcb:XILINX_JTAG_PTH_MOLEX_0878311420, F.Cu at (216.5, 75.4)
- added Q1: SSM6N58NU, azonenberg_pcb:DFN_6_0.65MM_2x2MM_GDS, F.Cu at (233.8, 100.4)
- added R31: 1K, azonenberg_pcb:EIA_0402_RES_NOSILK, F.Cu at (236.8, 101.0)
- added R40: 0, azonenberg_pcb:EIA_0402_RES_NOSILK, F.Cu at (211.1, 81.3)
- added R41: 0, azonenberg_pcb:EIA_0402_RES_NOSILK, F.Cu at (229.4, 75.8)
- added R42: 0, azonenberg_pcb:EIA_0402_RES_NOSILK, F.Cu at (226.9, 74.3)
- added R43: 4.7K, azonenberg_pcb:EIA_0402_RES_NOSILK, F.Cu at (216.1, 82.8)
- added R44: 33, azonenberg_pcb:EIA_0402_RES_NOSILK, F.Cu at (216.1, 84.3)
- added R45: 33, azonenberg_pcb:EIA_0402_RES_NOSILK, F.Cu at (222.1, 79.8)
- added R46: 33, azonenberg_pcb:EIA_0402_RES_NOSILK, F.Cu at (213.6, 81.3)
- added R47: 33, azonenberg_pcb:EIA_0402_RES_NOSILK, F.Cu at (218.6, 82.8)
- added R48: 33, azonenberg_pcb:EIA_0402_RES_NOSILK, F.Cu at (221.1, 82.8)
- added R49: 33, azonenberg_pcb:EIA_0402_RES_NOSILK, F.Cu at (208.6, 84.3)
- added R50: 33, azonenberg_pcb:EIA_0402_RES_NOSILK, F.Cu at (217.1, 79.8)
- added R51: 33, azonenberg_pcb:EIA_0402_RES_NOSILK, F.Cu at (212.1, 79.8)
- added R52: 33, azonenberg_pcb:EIA_0402_RES_NOSILK, F.Cu at (224.6, 79.8)
- added R53: 33, azonenberg_pcb:EIA_0402_RES_NOSILK, F.Cu at (211.1, 84.3)
- added R54: 33, azonenberg_pcb:EIA_0402_RES_NOSILK, F.Cu at (226.9, 75.8)
- added R55: 4.7K, azonenberg_pcb:EIA_0402_RES_NOSILK, F.Cu at (218.6, 81.3)
- added R56: 4.7K, azonenberg_pcb:EIA_0402_RES_NOSILK, F.Cu at (219.6, 79.8)
- added R57: 4.7K, azonenberg_pcb:EIA_0402_RES_NOSILK, F.Cu at (214.6, 79.8)
- added R58: 4.7K, azonenberg_pcb:EIA_0402_RES_NOSILK, F.Cu at (208.6, 81.3)
- added R59: 4.7K, azonenberg_pcb:EIA_0402_RES_NOSILK, F.Cu at (213.6, 82.8)
- added R81: 100, azonenberg_pcb:EIA_0402_RES_NOSILK, F.Cu at (233.4, 90.0)
- added R89: 4.7K, azonenberg_pcb:EIA_0402_RES_NOSILK, F.Cu at (221.1, 81.3)
- added R90: 4.7K, azonenberg_pcb:EIA_0402_RES_NOSILK, F.Cu at (216.1, 81.3)
- added R91: 4.7K, azonenberg_pcb:EIA_0402_RES_NOSILK, F.Cu at (213.6, 84.3)
- added R92: 33, azonenberg_pcb:EIA_0402_RES_NOSILK, F.Cu at (255.6, 74.3)
- added TP18: U.FL, azonenberg_pcb:CONN_U.FL_TE_1909763-1, F.Cu at (210.1, 91.8)
- added TP19: U.FL, azonenberg_pcb:CONN_U.FL_TE_1909763-1, F.Cu at (221.2, 91.8)
- added TP20: U.FL, azonenberg_pcb:CONN_U.FL_TE_1909763-1, F.Cu at (215.7, 97.1)
- added TP21: U.FL, azonenberg_pcb:CONN_U.FL_TE_1909763-1, F.Cu at (221.2, 97.1)
- added TP22: U.FL, azonenberg_pcb:CONN_U.FL_TE_1909763-1, F.Cu at (210.1, 97.1)
- added TP23: U.FL, azonenberg_pcb:CONN_U.FL_TE_1909763-1, F.Cu at (215.7, 91.8)
- added U10: MT25QU256ABA8E12-0AUT, azonenberg_pcb:BGA_24_6x8_DEPOP1_1MM, F.Cu at (206.0, 129.5)
- added U11: 74LVC1T45, azonenberg_pcb:DFN_6_0.5MM_1.6x1.6MM_TI_DPK, F.Cu at (211.4, 129.3)
- added U12: 74LVC1T45, azonenberg_pcb:DFN_6_0.5MM_1.6x1.6MM_TI_DPK, F.Cu at (211.4, 126.0)
- added U13: 74LVC1T45, azonenberg_pcb:DFN_6_0.5MM_1.6x1.6MM_TI_DPK, F.Cu at (213.9, 126.0)
- added U14: STM32L431VxIx, azonenberg_pcb:BGA_100_7x7_DEPOP_0.5MM_STM32_UFBGA100_OSHPARK, F.Cu at (163.8, 75.0)
- R10: moved to B.Cu
- moved R23 213.0 mm to (64.5, 104.0), turned to 90 degrees
- moved TP6 210.5 mm to (64.5, 92.8)
- moved R19 191.9 mm to (64.5, 102.0), turned to -90 degrees
- moved TP1 182.2 mm to (64.2, 68.5)
- moved R5 182.0 mm to (64.0, 58.5), turned to 180 degrees
- moved C15 178.1 mm to (57.2, 97.0), turned to 90 degrees
- moved C8 176.4 mm to (76.7, 64.5), turned to -90 degrees
- moved C3 175.4 mm to (60.2, 71.0), turned to 180 degrees
- moved C10 170.0 mm to (73.2, 64.5), turned to -90 degrees
- moved U7 164.6 mm to (64.5, 96.8), turned to 90 degrees
- moved C6 162.8 mm to (73.2, 60.0), turned to 90 degrees
- moved C37 156.9 mm to (74.5, 96.2), turned to 90 degrees
- moved R10 149.0 mm to (108.0, 87.5)
- moved R7 148.4 mm to (64.0, 57.5)
- moved C33 147.6 mm to (71.0, 96.2), turned to 90 degrees
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Connections:
- net /Power Supply/12V0 renamed /12V0
- net /Power Supply/2V5 renamed /2V5
- net /Power Supply/3V3_SB renamed /3V3_SB
- net /SFP28 interfaces/3V3 renamed /3V3
- C112 pad 2: /SFP28 interfaces/GND -> /GND
- C113 pad 2: /SFP28 interfaces/GND -> /GND
- C116 pad 2: /SFP28 interfaces/GND -> /GND
- C117 pad 2: /SFP28 interfaces/GND -> /GND
- C61 pad 2: /SFP28 interfaces/GND -> /GND
- C62 pad 2: /SFP28 interfaces/GND -> /GND
- C65 pad 2: /SFP28 interfaces/GND -> /GND
- C66 pad 2: /SFP28 interfaces/GND -> /GND
- C67 pad 2: /SFP28 interfaces/GND -> /GND
- C68 pad 2: /SFP28 interfaces/GND -> /GND
- C71 pad 2: /SFP28 interfaces/GND -> /GND
- C72 pad 2: /SFP28 interfaces/GND -> /GND
- C73 pad 2: /SFP28 interfaces/GND -> /GND
- C74 pad 2: /SFP28 interfaces/GND -> /GND
- C77 pad 2: /SFP28 interfaces/GND -> /GND
- C78 pad 2: /SFP28 interfaces/GND -> /GND
- J10 pad 1: /SFP28 interfaces/GND -> /GND
- J11 pad 1: /SFP28 interfaces/GND -> /GND
- J11 pad 10: /SFP28 interfaces/GND -> /GND
- J11 pad 11: /SFP28 interfaces/GND -> /GND
- J11 pad 12: /SFP28 interfaces/SFP0_RX_N -> /SFP28 interfaces/SFP0_RX_P
- J11 pad 13: /SFP28 interfaces/SFP0_RX_P -> /SFP28 interfaces/SFP0_RX_N
- J11 pad 14: /SFP28 interfaces/GND -> /GND
- J11 pad 17: /SFP28 interfaces/GND -> /GND
- J11 pad 20: /SFP28 interfaces/GND -> /GND
- J12 pad 1: /SFP28 interfaces/GND -> /GND
- J17 pad 2: /SMPM ports/GND -> /GND
- J18 pad 2: /SMPM ports/GND -> /GND
- J19 pad 2: /SMPM ports/GND -> /GND
- J20 pad 2: /SMPM ports/GND -> /GND
- J21 pad 2: /SMPM ports/GND -> /GND
- J22 pad 2: /SMPM ports/GND -> /GND
- J23 pad 2: /SMPM ports/GND -> /GND
- J24 pad 2: /SMPM ports/GND -> /GND
- J25 pad 2: /SMPM ports/GND -> /GND
- J26 pad 2: /SMPM ports/GND -> /GND
- J27 pad 2: /SMPM ports/GND -> /GND
- J28 pad 2: /SMPM ports/GND -> /GND
- J29 pad 2: /SMPM ports/GND -> /GND
- J30 pad 2: /SMPM ports/GND -> /GND
- J31 pad 2: /SMPM ports/GND -> /GND
- J32 pad 2: /SMPM ports/GND -> /GND
- J33 pad 1: /SFP28 interfaces/GND -> /GND
- J33 pad 10: /SFP28 interfaces/GND -> /GND
- J33 pad 11: /SFP28 interfaces/GND -> /GND
- J33 pad 12: /SFP28 interfaces/SFP3_RX_N -> /SFP28 interfaces/SFP3_RX_P
- J33 pad 13: /SFP28 interfaces/SFP3_RX_P -> /SFP28 interfaces/SFP3_RX_N
- J33 pad 14: /SFP28 interfaces/GND -> /GND
- J33 pad 17: /SFP28 interfaces/GND -> /GND
- J33 pad 20: /SFP28 interfaces/GND -> /GND
- J34 pad 1: /SFP28 interfaces/GND -> /GND
- J7 pad 1: /SFP28 interfaces/GND -> /GND
- J7 pad 10: /SFP28 interfaces/GND -> /GND
- J7 pad 11: /SFP28 interfaces/GND -> /GND
- J7 pad 12: /SFP28 interfaces/SFP2_RX_N -> /SFP28 interfaces/SFP2_RX_P
- J7 pad 13: /SFP28 interfaces/SFP2_RX_P -> /SFP28 interfaces/SFP2_RX_N
- J7 pad 14: /SFP28 interfaces/GND -> /GND
- J7 pad 17: /SFP28 interfaces/GND -> /GND
- J7 pad 20: /SFP28 interfaces/GND -> /GND
- J8 pad 1: /SFP28 interfaces/GND -> /GND
- J9 pad 1: /SFP28 interfaces/GND -> /GND
- J9 pad 10: /SFP28 interfaces/GND -> /GND
- J9 pad 11: /SFP28 interfaces/GND -> /GND
- J9 pad 12: /SFP28 interfaces/SFP1_RX_N -> /SFP28 interfaces/SFP1_RX_P
- J9 pad 13: /SFP28 interfaces/SFP1_RX_P -> /SFP28 interfaces/SFP1_RX_N
- J9 pad 14: /SFP28 interfaces/GND -> /GND
- J9 pad 17: /SFP28 interfaces/GND -> /GND
- J9 pad 20: /SFP28 interfaces/GND -> /GND
- R63 pad 1: /SFP28 interfaces/GND -> /GND
- R64 pad 1: /SFP28 interfaces/GND -> /GND
- R70 pad 1: /SFP28 interfaces/GND -> /GND
- R71 pad 1: /SFP28 interfaces/GND -> /GND
- R77 pad 1: /SFP28 interfaces/GND -> /GND
- R78 pad 1: /SFP28 interfaces/GND -> /GND
- R85 pad 1: /SFP28 interfaces/GND -> /GND
- R86 pad 1: /SFP28 interfaces/GND -> /GND
- U1 pad 11: /Power Supply/FPGA_RST_N -> /FPGA support/FPGA_RESET_N_3V3
- U1 pad 22: /Power Supply/FPGA_DONE -> /FPGA support/FPGA_DONE_3V3
- U1 pad 25: /Power Supply/FPGA_INIT -> /FPGA support/FPGA_INIT_3V3
- U4 pad 5: /FPGA support/1V8 -> /FPGA support/3V3
- U9 pad AA4: /SFP28 interfaces/SFP0_TX_N -> /SFP28 interfaces/SFP3_TX_N
- U9 pad AA5: /SFP28 interfaces/SFP0_TX_P -> /SFP28 interfaces/SFP3_TX_P
- U9 pad AB6: /SMPM ports/K_REFCLK_0_N -> unconnected-(U9-PadAB6)
- U9 pad AB7: /SMPM ports/K_REFCLK_0_P -> unconnected-(U9-PadAB7)
- U9 pad K6: /QSFP28 interface/QSFP28A_REFCLK0_N -> unconnected-(U9-PadK6)
- U9 pad K7: /QSFP28 interface/QSFP28A_REFCLK0_P -> unconnected-(U9-PadK7)
- U9 pad M6: /QSFP28 interface/QSFP28B_REFCLK1_N -> unconnected-(U9-PadM6)
- U9 pad M7: /QSFP28 interface/QSFP28B_REFCLK1_P -> unconnected-(U9-PadM7)
- U9 pad P1: /SFP28 interfaces/SFP3_RX_N -> /SFP28 interfaces/SFP0_RX_N
- U9 pad P2: /SFP28 interfaces/SFP3_RX_P -> /SFP28 interfaces/SFP0_RX_P
- U9 pad P6: /QSFP28 interface/QSFP28B_REFCLK0_N -> unconnected-(U9-PadP6)
- U9 pad P7: /QSFP28 interface/QSFP28B_REFCLK0_P -> unconnected-(U9-PadP7)
- U9 pad R4: /SFP28 interfaces/SFP3_TX_N -> /SFP28 interfaces/SFP0_TX_N
- U9 pad R5: /SFP28 interfaces/SFP3_TX_P -> /SFP28 interfaces/SFP0_TX_P
- U9 pad T1: /SFP28 interfaces/SFP2_RX_N -> /SFP28 interfaces/SFP1_RX_N
- U9 pad T2: /SFP28 interfaces/SFP2_RX_P -> /SFP28 interfaces/SFP1_RX_P
- U9 pad T6: /SFP28 interfaces/SFP28_REFCLK1_N -> unconnected-(U9-PadT6)
- U9 pad T7: /SFP28 interfaces/SFP28_REFCLK1_P -> unconnected-(U9-PadT7)
- U9 pad U4: /SFP28 interfaces/SFP2_TX_N -> /SFP28 interfaces/SFP1_TX_N
- U9 pad U5: /SFP28 interfaces/SFP2_TX_P -> /SFP28 interfaces/SFP1_TX_P
- U9 pad V1: /SFP28 interfaces/SFP1_RX_N -> /SFP28 interfaces/SFP2_RX_N
- U9 pad V2: /SFP28 interfaces/SFP1_RX_P -> /SFP28 interfaces/SFP2_RX_P
- U9 pad W4: /SFP28 interfaces/SFP1_TX_N -> /SFP28 interfaces/SFP2_TX_N
- U9 pad W5: /SFP28 interfaces/SFP1_TX_P -> /SFP28 interfaces/SFP2_TX_P
- U9 pad Y1: /SFP28 interfaces/SFP0_RX_N -> /SFP28 interfaces/SFP3_RX_N
- U9 pad Y2: /SFP28 interfaces/SFP0_RX_P -> /SFP28 interfaces/SFP3_RX_P
- U9 pad Y6: /SMPM ports/K_REFCLK_1_N -> unconnected-(U9-PadY6)
- U9 pad Y7: /SMPM ports/K_REFCLK_1_P -> unconnected-(U9-PadY7)
Routing:
- net /GND: track 0.00 -> 595.4 mm, vias 0 -> 89
- net /FPGA support/3V3: track 35.6 -> 337.4 mm
- net /FPGA support/GND: track 347.6 -> 528.9 mm, vias 175 -> 203
- net /SFP28 interfaces/SFP3_RX_P: track 0.00 -> 80.8 mm
- net /SFP28 interfaces/SFP3_RX_N: track 0.00 -> 80.8 mm
- net /SFP28 interfaces/SFP3_TX_N: track 0.49 -> 78.4 mm, vias 1 -> 2
- net /SFP28 interfaces/SFP3_TX_P: track 0.49 -> 78.4 mm, vias 1 -> 2
- net /SFP28 interfaces/SFP2_TX_FAULT: track 0.00 -> 60.8 mm, vias 0 -> 1
- net /SFP28 interfaces/SFP2_TX_DISABLE: track 0.00 -> 59.6 mm, vias 0 -> 1
- net /SFP28 interfaces/SFP2_RX_P: track 5.03 -> 64.4 mm
- net /SFP28 interfaces/SFP2_RX_N: track 4.93 -> 64.3 mm
- net /SFP28 interfaces/SFP2_I2C_SDA: track 0.00 -> 58.4 mm, vias 0 -> 1
- net /SFP28 interfaces/SFP2_I2C_SCL: track 0.00 -> 54.3 mm, vias 0 -> 1
- net /SFP28 interfaces/SFP2_TX_P: track 8.59 -> 62.5 mm, vias 1 -> 2
- net /SFP28 interfaces/SFP2_TX_N: track 8.55 -> 62.4 mm, vias 1 -> 2
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Other:
- board text added: "(-)RX3(+)"
- board text added: "3V3"
- board text added: "GTY_VCC"
- board text added: "SFP0"
- board text added: "SFP1"
- board text added: "SFP2"
- board text added: "SFP3"
- board text added: "VCCINT"
- board text removed: "TODO: Replace with SFP28 cages (this is temporary for floorplanning)"

Commit message: Continued initial layout of kup-lulz
Parts:
- added C111: 10 uF, azonenberg_pcb:EIA_0805_CAP_NOSILK, F.Cu at (101.0, 78.8)
- added C134: 0.47 uF, azonenberg_pcb:EIA_0402_CAP_NOSILK, F.Cu at (263.8, 113.2)
- added C135: 0.47 uF, azonenberg_pcb:EIA_0402_CAP_NOSILK, F.Cu at (244.7, 107.4)
- added C136: 0.47 uF, azonenberg_pcb:EIA_0402_CAP_NOSILK, F.Cu at (254.0, 102.8)
- added C137: 0.1 uF, azonenberg_pcb:EIA_0402_CAP_NOSILK, F.Cu at (249.7, 107.4)
- added C138: 0.1 uF, azonenberg_pcb:EIA_0402_CAP_NOSILK, F.Cu at (252.2, 107.4)
- added C139: 0.1 uF, azonenberg_pcb:EIA_0402_CAP_NOSILK, F.Cu at (247.2, 107.4)
- added C140: 0.1 uF, azonenberg_pcb:EIA_0402_CAP_NOSILK, F.Cu at (254.0, 104.3)
- added C141: 0.47 uF, azonenberg_pcb:EIA_0402_CAP_NOSILK, F.Cu at (267.8, 102.8)
- added C142: 0.1 uF, azonenberg_pcb:EIA_0402_CAP_NOSILK, F.Cu at (265.3, 105.8)
- added C143: 0.1 uF, azonenberg_pcb:EIA_0402_CAP_NOSILK, F.Cu at (267.8, 104.3)
- added C39: DNP, azonenberg_pcb:EIA_0402_CAP_NOSILK, F.Cu at (181.8, 119.5)
- added C42: 330 uF, azonenberg_pcb:EIA_1210_CAP_NOSILK, F.Cu at (211.8, 134.8)
- added C43: 47 uF, azonenberg_pcb:EIA_1210_CAP_NOSILK, F.Cu at (206.8, 134.8)
- added C44: 47 uF, azonenberg_pcb:EIA_1210_CAP_NOSILK, F.Cu at (211.8, 127.0)
- added C45: 47 uF, azonenberg_pcb:EIA_1210_CAP_NOSILK, F.Cu at (221.8, 127.0)
- added C46: 47 uF, azonenberg_pcb:EIA_1210_CAP_NOSILK, F.Cu at (206.8, 127.0)
- added C47: 10 uF, azonenberg_pcb:EIA_0805_CAP_NOSILK, B.Cu at (89.8, 76.0)
- added C48: 10 uF, azonenberg_pcb:EIA_0805_CAP_NOSILK, F.Cu at (101.0, 76.2)
- added C49: 10 uF, azonenberg_pcb:EIA_0805_CAP_NOSILK, F.Cu at (101.0, 74.2)
- added C50: 10 uF, azonenberg_pcb:EIA_0805_CAP_NOSILK, B.Cu at (68.0, 79.8)
- added C51: 100 uF, azonenberg_pcb:EIA_1210_CAP_NOSILK, F.Cu at (216.8, 127.0)
- added C52: 10 uF, azonenberg_pcb:EIA_0805_CAP_NOSILK, F.Cu at (68.5, 68.5)
- added C53: 100 uF, azonenberg_pcb:EIA_1210_CAP_NOSILK, F.Cu at (216.8, 134.8)
- added C54: 100 uF, azonenberg_pcb:EIA_1210_CAP_NOSILK, F.Cu at (206.8, 130.9)
- added C55: 100 uF, azonenberg_pcb:EIA_1210_CAP_NOSILK, F.Cu at (216.8, 130.9)
- added C56: 100 uF, azonenberg_pcb:EIA_1210_CAP_NOSILK, F.Cu at (211.8, 130.9)
- added C57: 47 uF, azonenberg_pcb:EIA_1210_CAP_NOSILK, F.Cu at (221.8, 130.9)
- added C58: 10 uF, azonenberg_pcb:EIA_0805_CAP_NOSILK, B.Cu at (80.1, 86.0)
- added C79: 22 uF, azonenberg_pcb:EIA_1210_CAP_NOSILK, F.Cu at (45.5, 149.5)
- added C80: 22 uF, azonenberg_pcb:EIA_1210_CAP_NOSILK, F.Cu at (64.0, 150.0)
- added C83: 22 uF, azonenberg_pcb:EIA_1210_CAP_NOSILK, F.Cu at (42.5, 132.4)
- added C84: 22 uF, azonenberg_pcb:EIA_1210_CAP_NOSILK, F.Cu at (43.0, 139.0)
- added C85: 22 uF, azonenberg_pcb:EIA_1210_CAP_NOSILK, F.Cu at (42.0, 126.5)
- added C86: 22 uF, azonenberg_pcb:EIA_1210_CAP_NOSILK, F.Cu at (63.0, 141.0)
- added C87: 22 uF, azonenberg_pcb:EIA_1210_CAP_NOSILK, F.Cu at (72.5, 134.5)
- added C88: 22 uF, azonenberg_pcb:EIA_1210_CAP_NOSILK, F.Cu at (63.5, 131.0)
- added J39: CONN_01X03, azonenberg_pcb:CONN_HEADER_2.54MM_1x3, F.Cu at (253.2, 95.0)
- added L10: 1 uH, azonenberg_pcb:EIA_0805_INDUCTOR_NOSILK, F.Cu at (66.0, 137.0)
- added L11: 1 uH, azonenberg_pcb:EIA_0805_INDUCTOR_NOSILK, F.Cu at (74.0, 130.5)
- added L12: 1 uH, azonenberg_pcb:EIA_0805_INDUCTOR_NOSILK, F.Cu at (68.0, 134.0)
- added L7: 1 uH, azonenberg_pcb:EIA_0805_INDUCTOR_NOSILK, F.Cu at (38.5, 142.5)
- added L8: 1 uH, azonenberg_pcb:EIA_0805_INDUCTOR_NOSILK, F.Cu at (43.0, 143.0)
- added L9: 1 uH, azonenberg_pcb:EIA_0805_INDUCTOR_NOSILK, F.Cu at (48.0, 145.0)
- added M6: LOGO, azonenberg_pcb:LONGTHING-1200DPI, F.Cu at (26.9, 109.0)
- added M7: LOGO, w_logo:Logo_silk_ROHS_5x2.8mm, F.Cu at (28.2, 131.8)
- added M8: LOGO, w_logo:Logo_silk_OSHW_6x6mm, F.Cu at (26.5, 118.5)
- added M9: LOGO, w_logo:Logo_silk_WEEE_3.4x5mm, F.Cu at (27.0, 126.0)
- added R93: 10K, azonenberg_pcb:EIA_0402_RES_NOSILK, F.Cu at (134.7, 49.6)
- added R94: 4.7K, azonenberg_pcb:EIA_0402_RES_NOSILK, F.Cu at (266.2, 113.2)
- added R95: 1K, azonenberg_pcb:EIA_0402_RES_NOSILK, F.Cu at (267.8, 105.8)
- added R96: 1K, azonenberg_pcb:EIA_0402_RES_NOSILK, F.Cu at (265.3, 104.3)
- added R97: 1K, azonenberg_pcb:EIA_0402_RES_NOSILK, F.Cu at (265.3, 102.8)
- added TP24: TESTCLIP, azonenberg_pcb:TESTPOINT_SMT_KEYSTONE_5016, F.Cu at (238.5, 149.5)
- added TP25: TESTCLIP, azonenberg_pcb:TESTPOINT_SMT_KEYSTONE_5016, F.Cu at (244.2, 149.5)
- added U15: AT24MAC402, azonenberg_pcb:DFN_8_0.5MM_2x3MM_TALL, F.Cu at (260.9, 113.2)
- added U16: SIT9121AI-2BF-XXS156.250000G, azonenberg_pcb:OSCILLATOR_LVDS_3.2x2.5, F.Cu at (245.8, 104.4)
- added U17: SIT9121AI-2BF-XXS156.250000G, azonenberg_pcb:OSCILLATOR_LVDS_3.2x2.5, F.Cu at (250.4, 104.4)
- added U18: SIT9121AI-2BF-XXS156.250000G, azonenberg_pcb:OSCILLATOR_LVDS_3.2x2.5, F.Cu at (261.7, 104.4)
- added U8: ADP1740ACPZ-1.8-R7, azonenberg_pcb:QFN_16_0.65MM_4x4MM, F.Cu at (179.2, 115.8)
- C116, C117, C71, C72, C77, C78, R25, R27, R32, R39, R44, R49, R50, R52, R60, R61, R65, R66, R67, R68, R72, R73, R74, R75, R79, R80, R81, R82, R83, R87, R88: moved to B.Cu
- J15, J16: footprint azonenberg_pcb:CONN_QSFP+_TE_2110819-1 -> azonenberg_pcb:CONN_ZQSFP+_TE_1551920-2
- J35, J36: footprint azonenberg_pcb:CONN_QSFP_CAGE_TE_2110487-1 -> azonenberg_pcb:CONN_ZQSFP+_CAGE_TE_4-2170705-5
- R40, R41, R42: value 0 -> 4.7K
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Connections:
- C1 pad 2: /FPGA support/GND -> /GND
- C10 pad 2: /FPGA support/GND -> /GND
- C103 pad 2: /SMPM ports/K_TX_0_P -> /SMPM ports/K_TX_0_N
- C104 pad 2: /SMPM ports/K_TX_0_N -> /SMPM ports/K_TX_0_P
- C105 pad 2: /SMPM ports/K_TX_1_P -> /SMPM ports/K_TX_1_N
- C106 pad 2: /SMPM ports/K_TX_1_N -> /SMPM ports/K_TX_1_P
- C107 pad 2: /SMPM ports/K_TX_2_P -> /SMPM ports/K_TX_2_N
- C108 pad 2: /SMPM ports/K_TX_2_N -> /SMPM ports/K_TX_2_P
- C109 pad 2: /SMPM ports/K_TX_3_P -> /SMPM ports/K_TX_3_N
- C11 pad 2: /FPGA support/GND -> /GND
- C110 pad 2: /SMPM ports/K_TX_3_N -> /SMPM ports/K_TX_3_P
- C118 pad 2: /FPGA support/GND -> /GND
- C119 pad 2: /FPGA support/GND -> /GND
- C12 pad 2: /FPGA support/GND -> /GND
- C120 pad 2: /FPGA support/GND -> /GND
- C121 pad 1: /FPGA support/3V3 -> /3V3
- C121 pad 2: /FPGA support/GND -> /GND
- C122 pad 1: /FPGA support/3V3 -> /3V3
- C122 pad 2: /FPGA support/GND -> /GND
- C123 pad 1: /FPGA support/3V3 -> /3V3
- C123 pad 2: /FPGA support/GND -> /GND
- C124 pad 1: /Management/3V3 -> /3V3
- C124 pad 2: /Management/GND -> /GND
- C125 pad 2: /Management/GND -> /GND
- C126 pad 1: /Management/3V3 -> /3V3
- C126 pad 2: /Management/GND -> /GND
- C127 pad 2: /Management/GND -> /GND
- C128 pad 1: /Management/3V3 -> /3V3
- C128 pad 2: /Management/GND -> /GND
- C129 pad 1: /Management/3V3 -> /3V3
- C129 pad 2: /Management/GND -> /GND
- C13 pad 2: /FPGA support/GND -> /GND
- C130 pad 1: /Management/3V3 -> /3V3
- C130 pad 2: /Management/GND -> /GND
- C131 pad 1: /Management/3V3 -> /3V3
- C131 pad 2: /Management/GND -> /GND
- C132 pad 1: /Management/3V3 -> /3V3
- C132 pad 2: /Management/GND -> /GND
- C133 pad 1: /Management/3V3 -> /3V3
- C133 pad 2: /Management/GND -> /GND
- C14 pad 2: /FPGA support/GND -> /GND
- C15 pad 2: /FPGA support/GND -> /GND
- C16 pad 2: /FPGA support/GND -> /GND
- C17 pad 2: /FPGA support/GND -> /GND
- C18 pad 2: /FPGA support/GND -> /GND
- C19 pad 2: /FPGA support/GND -> /GND
- C2 pad 2: /FPGA support/GND -> /GND
- C20 pad 2: /FPGA support/GND -> /GND
- C21 pad 2: /FPGA support/GND -> /GND
- C22 pad 2: /FPGA support/GND -> /GND
- C23 pad 2: /FPGA support/GND -> /GND
- C24 pad 2: /FPGA support/GND -> /GND
- C25 pad 2: /FPGA support/GND -> /GND
- C26 pad 1: /FPGA support/3V3 -> /3V3
- C26 pad 2: /FPGA support/GND -> /GND
- C27 pad 2: /FPGA support/GND -> /GND
- C28 pad 2: /FPGA support/GND -> /GND
- C29 pad 2: /FPGA support/GND -> /GND
- C3 pad 2: /FPGA support/GND -> /GND
- C30 pad 1: /FPGA support/3V3 -> /3V3
- C30 pad 2: /FPGA support/GND -> /GND
- C31 pad 2: /FPGA support/GND -> /GND
- C32 pad 2: /FPGA support/GND -> /GND
- C33 pad 2: /FPGA support/GND -> /GND
- C34 pad 1: /FPGA support/3V3 -> /3V3
- C34 pad 2: /FPGA support/GND -> /GND
- C35 pad 2: /FPGA support/GND -> /GND
- C36 pad 2: /FPGA support/GND -> /GND
- C37 pad 2: /FPGA support/GND -> /GND
- C38 pad 1: /FPGA support/3V3 -> /3V3
- C38 pad 2: /FPGA support/GND -> /GND
- C4 pad 2: /FPGA support/GND -> /GND
- C40 pad 2: /FPGA support/GND -> /GND
- C41 pad 2: /FPGA support/GND -> /GND
- C5 pad 2: /FPGA support/GND -> /GND
- C59 pad 2: /FPGA support/GND -> /GND
- C6 pad 2: /FPGA support/GND -> /GND
- C60 pad 2: /FPGA support/GND -> /GND
- C7 pad 2: /FPGA support/GND -> /GND
- C8 pad 2: /FPGA support/GND -> /GND
- C81 pad 1: /QSFP28 interface/3V3 -> /3V3
- C81 pad 2: /QSFP28 interface/GND -> /GND
- C82 pad 1: /QSFP28 interface/3V3 -> /3V3
- C82 pad 2: /QSFP28 interface/GND -> /GND
- C89 pad 2: /QSFP28 interface/GND -> /GND
- C9 pad 2: /FPGA support/GND -> /GND
- C90 pad 2: /QSFP28 interface/GND -> /GND
- C91 pad 2: /QSFP28 interface/GND -> /GND
- C92 pad 2: /QSFP28 interface/GND -> /GND
- C93 pad 2: /QSFP28 interface/GND -> /GND
- C94 pad 2: /QSFP28 interface/GND -> /GND
- C95 pad 2: /SMPM ports/K_RX_0_P -> /SMPM ports/K_RX_0_N
- C96 pad 2: /SMPM ports/K_RX_0_N -> /SMPM ports/K_RX_0_P
- D1 pad 1: /FPGA support/GND -> /GND
- D2 pad 1: /FPGA support/GND -> /GND
- FB3 pad 1: /Management/3V3 -> /3V3
- J1 pad 5: /FPGA support/GND -> /GND
- J1 pad 6: /FPGA support/GND -> /GND
- J1 pad 7: /FPGA support/GND -> /GND
- J1 pad 8: /FPGA support/GND -> /GND
- J11 pad 2: /SFP28 interfaces/SFP0_TX_FAULT -> /Management/SFP0_TX_FAULT
- J11 pad 3: /SFP28 interfaces/SFP0_TX_DISABLE -> /Management/SFP0_TX_DISABLE
- J11 pad 6: /SFP28 interfaces/SFP0_MOD_ABS -> /Management/SFP0_MOD_ABS
- J11 pad 7: /SFP28 interfaces/SFP0_RS0 -> /Management/SFP0_RS0
- J11 pad 8: /SFP28 interfaces/SFP0_RX_LOS -> /Management/SFP0_RX_LOS
- J11 pad 9: /SFP28 interfaces/SFP0_RS1 -> /Management/SFP0_RS1
- J13 pad 11: /Management/GND -> /GND
- J13 pad 12: /Management/3V3 -> /3V3
- J13 pad 5: /Management/GND -> /GND
- J13 pad 6: /Management/3V3 -> /3V3
- J14 pad 11: /Management/GND -> /GND
- J14 pad 12: /Management/3V3 -> /3V3
- J14 pad 5: /Management/GND -> /GND
- J14 pad 6: /Management/3V3 -> /3V3
- J15 pad 1: /QSFP28 interface/GND -> /GND
- J15 pad 11: /QSFP28 interface/QSFP_I2C_SCL -> /Management/QSFP_I2C_SCL
- J15 pad 12: /QSFP28 interface/QSFP_I2C_SDA -> /Management/QSFP_I2C_SDA
- J15 pad 13: /QSFP28 interface/GND -> /GND
- J15 pad 16: /QSFP28 interface/GND -> /GND
- J15 pad 19: /QSFP28 interface/GND -> /GND
- J15 pad 20: /QSFP28 interface/GND -> /GND
- J15 pad 21: /QSFP28 interface/QSFP28A_RX2_N -> /QSFP28 interface/QSFP28A_RX2_P
- J15 pad 22: /QSFP28 interface/QSFP28A_RX2_P -> /QSFP28 interface/QSFP28A_RX2_N
- J15 pad 23: /QSFP28 interface/GND -> /GND
- J15 pad 26: /QSFP28 interface/GND -> /GND
- J15 pad 27: /QSFP28 interface/QSFP0_PRESENT_N -> /Management/QSFP0_PRESENT_N
- J15 pad 28: /QSFP28 interface/QSFP0_INT_N -> /Management/QSFP0_INT_N
- J15 pad 31: /QSFP28 interface/QSFP0_LPMODE -> /Management/QSFP0_LPMODE
- J15 pad 32: /QSFP28 interface/GND -> /GND
- J15 pad 35: /QSFP28 interface/GND -> /GND
- J15 pad 38: /QSFP28 interface/GND -> /GND
- J15 pad 4: /QSFP28 interface/GND -> /GND
- J15 pad 7: /QSFP28 interface/GND -> /GND
- J15 pad 8: /QSFP28 interface/QSFP0_I2C_SEL_N -> /Management/QSFP0_I2C_SEL_N
- J15 pad 9: /QSFP28 interface/QSFP0_RST_N -> /Management/QSFP0_RST_N
- J16 pad 1: /QSFP28 interface/GND -> /GND
- J16 pad 11: /QSFP28 interface/QSFP_I2C_SCL -> /Management/QSFP_I2C_SCL
- J16 pad 12: /QSFP28 interface/QSFP_I2C_SDA -> /Management/QSFP_I2C_SDA
- J16 pad 13: /QSFP28 interface/GND -> /GND
- J16 pad 14: /QSFP28 interface/QSFP28B_RX3_P -> /QSFP28 interface/QSFP28B_RX3_N
- J16 pad 15: /QSFP28 interface/QSFP28B_RX3_N -> /QSFP28 interface/QSFP28B_RX3_P
- J16 pad 16: /QSFP28 interface/GND -> /GND
- J16 pad 17: /QSFP28 interface/QSFP28B_RX1_P -> /QSFP28 interface/QSFP28B_RX1_N
- J16 pad 18: /QSFP28 interface/QSFP28B_RX1_N -> /QSFP28 interface/QSFP28B_RX1_P
- J16 pad 19: /QSFP28 interface/GND -> /GND
- J16 pad 2: /QSFP28 interface/QSFP28B_TX2_N -> /QSFP28 interface/QSFP28B_TX3_N
- J16 pad 20: /QSFP28 interface/GND -> /GND
- J16 pad 21: /QSFP28 interface/QSFP28B_RX2_N -> /QSFP28 interface/QSFP28B_RX2_P
- J16 pad 22: /QSFP28 interface/QSFP28B_RX2_P -> /QSFP28 interface/QSFP28B_RX2_N
- J16 pad 23: /QSFP28 interface/GND -> /GND
- J16 pad 24: /QSFP28 interface/QSFP28B_RX4_N -> /QSFP28 interface/QSFP28B_RX4_P
- J16 pad 25: /QSFP28 interface/QSFP28B_RX4_P -> /QSFP28 interface/QSFP28B_RX4_N
- J16 pad 26: /QSFP28 interface/GND -> /GND
- J16 pad 27: /QSFP28 interface/QSFP1_PRESENT_N -> /Management/QSFP1_PRESENT_N
- J16 pad 28: /QSFP28 interface/QSFP1_INT_N -> /Management/QSFP1_INT_N
- J16 pad 3: /QSFP28 interface/QSFP28B_TX2_P -> /QSFP28 interface/QSFP28B_TX3_P
- J16 pad 31: /QSFP28 interface/QSFP1_LPMODE -> /Management/QSFP1_LPMODE
- J16 pad 32: /QSFP28 interface/GND -> /GND
- J16 pad 33: /QSFP28 interface/QSFP28B_TX3_P -> /QSFP28 interface/QSFP28B_TX2_N
- J16 pad 34: /QSFP28 interface/QSFP28B_TX3_N -> /QSFP28 interface/QSFP28B_TX2_P
- J16 pad 35: /QSFP28 interface/GND -> /GND
- J16 pad 36: /QSFP28 interface/QSFP28B_TX1_P -> /QSFP28 interface/QSFP28B_TX4_P
- J16 pad 37: /QSFP28 interface/QSFP28B_TX1_N -> /QSFP28 interface/QSFP28B_TX4_N
- J16 pad 38: /QSFP28 interface/GND -> /GND
- J16 pad 4: /QSFP28 interface/GND -> /GND
- J16 pad 5: /QSFP28 interface/QSFP28B_TX4_N -> /QSFP28 interface/QSFP28B_TX1_P
- J16 pad 6: /QSFP28 interface/QSFP28B_TX4_P -> /QSFP28 interface/QSFP28B_TX1_N
- J16 pad 7: /QSFP28 interface/GND -> /GND
- J16 pad 8: /QSFP28 interface/QSFP1_I2C_SEL_N -> /Management/QSFP1_I2C_SEL_N
- J16 pad 9: /QSFP28 interface/QSFP1_RST_N -> /Management/QSFP1_RST_N
- J2 pad 2: /FPGA support/GND -> /GND
- J3 pad 3: /FPGA support/GND -> /GND
- J33 pad 2: /SFP28 interfaces/SFP3_TX_FAULT -> /Management/SFP3_TX_FAULT
- J33 pad 3: /SFP28 interfaces/SFP3_TX_DISABLE -> /Management/SFP3_TX_DISABLE
- J33 pad 6: /SFP28 interfaces/SFP3_MOD_ABS -> /Management/SFP3_MOD_ABS
- J33 pad 7: /SFP28 interfaces/SFP3_RS0 -> /Management/SFP3_RS0
- J33 pad 8: /SFP28 interfaces/SFP3_RX_LOS -> /Management/SFP3_RX_LOS
- J33 pad 9: /SFP28 interfaces/SFP3_RS1 -> /Management/SFP3_RS1
- J35 pad 1: /QSFP28 interface/GND -> /GND
- J36 pad 1: /QSFP28 interface/GND -> /GND
- J37 pad 11: /Management/GND -> /GND
- J37 pad 2: /Management/3V3 -> /3V3
- J37 pad 3: /Management/GND -> /GND
- J37 pad 5: /Management/GND -> /GND
- J37 pad 7: /Management/GND -> /GND
- J37 pad 9: /Management/GND -> /GND
- J38 pad 11: /Management/GND -> /GND
- J38 pad 12: /Management/3V3 -> /3V3
- J38 pad 5: /Management/GND -> /GND
- J38 pad 6: /Management/3V3 -> /3V3
- J4 pad 2: /FPGA support/GND -> /GND
- J5 pad 3: /FPGA support/GND -> /GND
- J6 pad 11: /FPGA support/GND -> /GND
- J6 pad 13: /FPGA support/GND -> unconnected-(J6-Pad13)
- J6 pad 3: /FPGA support/GND -> /GND
- J6 pad 5: /FPGA support/GND -> /GND
- J6 pad 7: /FPGA support/GND -> /GND
- J6 pad 9: /FPGA support/GND -> /GND
- J7 pad 2: /SFP28 interfaces/SFP2_TX_FAULT -> /Management/SFP2_TX_FAULT
- J7 pad 3: /SFP28 interfaces/SFP2_TX_DISABLE -> /Management/SFP2_TX_DISABLE
- J7 pad 6: /SFP28 interfaces/SFP2_MOD_ABS -> /Management/SFP2_MOD_ABS
- J7 pad 7: /SFP28 interfaces/SFP2_RS0 -> /Management/SFP2_RS0
- J7 pad 8: /SFP28 interfaces/SFP2_RX_LOS -> /Management/SFP2_RX_LOS
- J7 pad 9: /SFP28 interfaces/SFP2_RS1 -> /Management/SFP2_RS1
- J9 pad 2: /SFP28 interfaces/SFP1_TX_FAULT -> /Management/SFP1_TX_FAULT
- J9 pad 3: /SFP28 interfaces/SFP1_TX_DISABLE -> /Management/SFP1_TX_DISABLE
- J9 pad 6: /SFP28 interfaces/SFP1_MOD_ABS -> /Management/SFP1_MOD_ABS
- J9 pad 7: /SFP28 interfaces/SFP1_RS0 -> /Management/SFP1_RS0
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Routing:
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- added copper zone on F.Cu, net /12V0
- added copper zone on F.Cu, net /3V3
- added copper zone on F.Cu, net /FPGA support/1V8
- added copper zone on F.Cu, net /FPGA support/VCCINT
- added copper zone on F.Cu, net /GND
- added copper zone on F.Cu, net /GTY_VTT
- added copper zone on F.Cu, net /Power Supply/GTY_VCC
Other:
- board text added: "(+)RX0(-)"
- board text added: "(+)TX2(-)"
- board text added: "(+)TX3(-)"
- board text added: "(-)RX1(+)"
- board text added: "(-)RX2(+)"
- board text added: "(-)TX0(+)"
- board text added: "(-)TX1(+)"
- board text added: "1V8"
- board text added: "3V3_SB"
- board text added: "GND"
- board text added: "SUPER_SCL"
- board text added: "SUPER_SDA"
- board text removed: "TODO: Replace with QSFP28 cages (this is temporary for floorplanning)"

Commit message: Continued initial layout
Parts:
- removed C14, C18: 22 uF 25V, azonenberg_pcb:EIA_1812_CAP_NOSILK
- removed C28, C32: 220 uF, azonenberg_pcb:EIA_1210_CAP_NOSILK
- removed C36: DNP, azonenberg_pcb:EIA_1210_CAP_NOSILK
- removed R18: 3k, azonenberg_pcb:EIA_0402_RES_NOSILK
- removed R22: 160, azonenberg_pcb:EIA_0402_RES_NOSILK
- removed R36: 10K, azonenberg_pcb:EIA_0402_RES_NOSILK
- removed R37: 1K, azonenberg_pcb:EIA_0402_RES_NOSILK
- removed R58, R59: 4.7K, azonenberg_pcb:EIA_0402_RES_NOSILK
- removed TP17: U.FL, azonenberg_pcb:CONN_U.FL_TE_1909763-1
- removed TP5: TESTPOINT, azonenberg_pcb:TESTPOINT_SMT_0.5MM
- removed U6: MYMGK00504ERSR, azonenberg_pcb:MODULE_MURATA_MYMGK00504ERSR
- C135, C137, C138, C139, C40, C41, C43, C54, C56, C59, C60, C80, C82, C86, C87, C88, C92, C93, C94, J5, L10, L11, L12, R31, R43, R45, R46, R47, R48, R55, R56, R57, TP21, TP22, TP23, U16: moved to B.Cu
- moved C141 208.8 mm to (61.6, 69.8)
- moved C143 206.9 mm to (63.4, 72.0)
- moved C142 204.5 mm to (63.4, 73.0)
- moved U18 204.1 mm to (60.2, 72.0), turned to -90 degrees
- moved TP16 190.5 mm to (64.4, 83.0), turned to 180 degrees
- moved C138 167.0 mm to (85.3, 100.0), turned to 90 degrees
- moved C137 165.2 mm to (84.6, 100.0), turned to 90 degrees
- moved U16 162.6 mm to (83.4, 113.6), turned to 180 degrees
- moved C56 161.5 mm to (59.5, 77.2), turned to 90 degrees
- moved C43 161.2 mm to (56.2, 77.2), turned to 90 degrees
- moved C135 159.0 mm to (85.8, 112.2), turned to 90 degrees
- moved J13 156.4 mm to (170.5, 142.0), turned to 90 degrees
- moved C54 153.7 mm to (62.8, 77.2), turned to 90 degrees
- moved C44 148.4 mm to (76.5, 66.0)
- moved C45 144.3 mm to (91.0, 66.0)
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Connections:
- net /Power Supply/GVEN_2V5 renamed /Power Supply/GVEN_3V3
- C40 pad 1: /2V5 -> /3V3
- J15 pad 17: /QSFP28 interface/QSFP28A_RX1_P -> /QSFP28 interface/QSFP28A_RX2_N
- J15 pad 18: /QSFP28 interface/QSFP28A_RX1_N -> /QSFP28 interface/QSFP28A_RX2_P
- J15 pad 21: /QSFP28 interface/QSFP28A_RX2_P -> /QSFP28 interface/QSFP28A_RX1_P
- J15 pad 22: /QSFP28 interface/QSFP28A_RX2_N -> /QSFP28 interface/QSFP28A_RX1_N
- J16 pad 2: /QSFP28 interface/QSFP28B_TX3_N -> /QSFP28 interface/QSFP28B_TX3_P
- J16 pad 3: /QSFP28 interface/QSFP28B_TX3_P -> /QSFP28 interface/QSFP28B_TX3_N
- J16 pad 36: /QSFP28 interface/QSFP28B_TX4_P -> /QSFP28 interface/QSFP28B_TX4_N
- J16 pad 37: /QSFP28 interface/QSFP28B_TX4_N -> /QSFP28 interface/QSFP28B_TX4_P
- R31 pad 1: /2V5 -> /3V3
- U1 pad 1: /Power Supply/2V5_EN -> unconnected-(U1-Pad1)
- U1 pad 2: /Power Supply/2V5_PGOOD -> unconnected-(U1-Pad2)
- U8 pad 1: /2V5 -> /3V3
- U8 pad 15: /2V5 -> /3V3
- U8 pad 16: /2V5 -> /3V3
- U8 pad 2: /2V5 -> /3V3
- U8 pad 3: /2V5 -> /3V3
- U9 pad A12: /Management/PMOD_DQ2 -> /Management/SFP0_RX_LOS
- U9 pad A13: /Management/PMOD_DQ3 -> /Management/SFP0_MOD_ABS
- U9 pad A14: /Management/PMOD_DQ0 -> /SFP28 interfaces/SFP0_I2C_SDA
- U9 pad AA13: /Management/SFP0_RX_LOS -> /Management/PMOD_DQ2
- U9 pad AA14: /SFP28 interfaces/SFP2_I2C_SCL -> /Management/PMODB_DQ1
- U9 pad AA15: /Management/SFP2_RX_LOS -> /Management/PMODB_DQ2
- U9 pad AB14: /SFP28 interfaces/SFP2_I2C_SDA -> /Management/PMODB_DQ0
- U9 pad AB15: /SFP28 interfaces/SFP3_I2C_SCL -> /Management/PMODB_DQ5
- U9 pad AB16: /SFP28 interfaces/SFP3_I2C_SDA -> /Management/PMODB_DQ4
- U9 pad AC13: /Management/SFP3_MOD_ABS -> /Management/PMODB_DQ7
- U9 pad AC14: /Management/SFP3_RX_LOS -> /Management/PMODB_DQ6
- U9 pad B12: /Management/PMOD_DQ4 -> /SFP28 interfaces/SFP1_I2C_SDA
- U9 pad B14: /Management/PMOD_DQ1 -> /SFP28 interfaces/SFP0_I2C_SCL
- U9 pad C12: /Management/PMOD_DQ5 -> /SFP28 interfaces/SFP1_I2C_SCL
- U9 pad C13: /Management/PMOD_DQ6 -> /Management/SFP1_RX_LOS
- U9 pad C14: /Management/PMOD_DQ7 -> /Management/SFP1_MOD_ABS
- U9 pad C18: /HP IOs/REFCLK3_N -> /HP IOs/REFCLK3_P
- U9 pad C19: /HP IOs/REFCLK3_P -> /HP IOs/REFCLK3_N
- U9 pad D13: /Management/PMODB_DQ0 -> /SFP28 interfaces/SFP2_I2C_SDA
- U9 pad D14: /Management/PMODB_DQ1 -> /SFP28 interfaces/SFP2_I2C_SCL
- U9 pad E12: /Management/PMODB_DQ2 -> /Management/SFP2_RX_LOS
- U9 pad E13: /Management/PMODB_DQ3 -> /Management/SFP2_MOD_ABS
- U9 pad F12: /Management/PMODB_DQ6 -> /Management/SFP3_RX_LOS
- U9 pad F13: /Management/PMODB_DQ4 -> /SFP28 interfaces/SFP3_I2C_SDA
- U9 pad F14: /Management/PMODB_DQ5 -> /SFP28 interfaces/SFP3_I2C_SCL
- U9 pad G12: /Management/PMODB_DQ7 -> /Management/SFP3_MOD_ABS
- U9 pad W12: /SFP28 interfaces/SFP0_I2C_SCL -> /Management/PMOD_DQ1
- U9 pad W13: /SFP28 interfaces/SFP0_I2C_SDA -> /Management/PMOD_DQ0
- U9 pad W14: /SFP28 interfaces/SFP1_I2C_SCL -> /Management/PMOD_DQ5
- U9 pad W15: /SFP28 interfaces/SFP1_I2C_SDA -> /Management/PMOD_DQ4
- U9 pad W16: /Management/SFP1_MOD_ABS -> /Management/PMOD_DQ7
- U9 pad Y13: /Management/SFP0_MOD_ABS -> /Management/PMOD_DQ3
- U9 pad Y15: /Management/SFP2_MOD_ABS -> /Management/PMODB_DQ3
- U9 pad Y16: /Management/SFP1_RX_LOS -> /Management/PMOD_DQ6
Routing:
- net /GND: track 2059.3 -> 2599.0 mm, vias 880 -> 1022
- net /3V3: track 429.8 -> 592.2 mm, vias 28 -> 57
- net /FPGA support/1V8: track 169.4 -> 290.0 mm, vias 65 -> 86
- net /Management/SFP0_RS0: track 101.1 -> 3.45 mm
- net /Management/SFP0_RX_LOS: track 98.5 -> 2.10 mm
- net /Management/SFP0_RS1: track 98.1 -> 2.85 mm
- net /Management/SFP1_TX_FAULT: track 89.5 -> 2.10 mm
- net /Management/SFP1_TX_DISABLE: track 89.2 -> 2.95 mm
- net /SFP28 interfaces/SFP1_I2C_SDA: track 86.7 -> 1.60 mm
- net /SFP28 interfaces/SFP1_I2C_SCL: track 82.9 -> 1.60 mm
- net /FPGA support/FPGA_JTAG_TMS: track 5.88 -> 86.1 mm
- net /Management/SFP1_MOD_ABS: track 82.7 -> 2.95 mm
- net /Management/SFP1_RS0: track 77.9 -> 3.20 mm
- net /Management/SFP1_RX_LOS: track 74.9 -> 2.10 mm
- net /Management/SFP1_RS1: track 71.8 -> 2.60 mm
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Other:
- board size 144.5 x 137 mm -> 154.5 x 137 mm
- board text added: "12V0"
- board text added: "FPGA JTAG"
- board text added: "FPGA PMOD A"
- board text added: "FPGA PMOD B"
- board text added: "GTY_VTT"
- board text added: "MCU JTAG"

Commit message: Continued initial routing
Parts:
- C20, C23, C24, C25, FB2, R24, R26: moved to B.Cu
- moved J4 70.8 mm to (116.2, 28.5)
- moved C20 65.9 mm to (75.1, 54.9), turned to 180 degrees
- moved C25 63.8 mm to (86.8, 57.6), turned to -90 degrees
- moved C24 61.4 mm to (79.9, 54.9)
- moved FB2 59.9 mm to (77.3, 54.9), turned to 180 degrees
- moved C23 59.9 mm to (87.4, 51.0)
- moved R13 58.3 mm to (78.5, 53.0)
- moved D1 57.1 mm to (76.2, 52.8)
- moved R14 53.6 mm to (78.5, 54.0)
- moved D2 53.2 mm to (76.2, 54.2)
- moved R26 49.8 mm to (79.6, 49.9), turned to 45 degrees
- moved R24 49.8 mm to (81.5, 55.7), turned to 90 degrees
- moved U1 41.5 mm to (83.8, 54.0)
- moved R12 38.1 mm to (83.0, 49.2), turned to 90 degrees
- moved J3 33.6 mm to (100.2, 28.5)
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Connections:
- J15 pad 14: /QSFP28 interface/QSFP28A_RX3_P -> /QSFP28 interface/QSFP28A_RX4_P
- J15 pad 15: /QSFP28 interface/QSFP28A_RX3_N -> /QSFP28 interface/QSFP28A_RX4_N
- J15 pad 17: /QSFP28 interface/QSFP28A_RX2_N -> /QSFP28 interface/QSFP28A_RX2_P
- J15 pad 18: /QSFP28 interface/QSFP28A_RX2_P -> /QSFP28 interface/QSFP28A_RX2_N
- J15 pad 2: /QSFP28 interface/QSFP28A_TX2_N -> /QSFP28 interface/QSFP28A_TX4_P
- J15 pad 24: /QSFP28 interface/QSFP28A_RX4_N -> /QSFP28 interface/QSFP28A_RX3_P
- J15 pad 25: /QSFP28 interface/QSFP28A_RX4_P -> /QSFP28 interface/QSFP28A_RX3_N
- J15 pad 3: /QSFP28 interface/QSFP28A_TX2_P -> /QSFP28 interface/QSFP28A_TX4_N
- J15 pad 33: /QSFP28 interface/QSFP28A_TX3_P -> /QSFP28 interface/QSFP28A_TX2_N
- J15 pad 34: /QSFP28 interface/QSFP28A_TX3_N -> /QSFP28 interface/QSFP28A_TX2_P
- J15 pad 5: /QSFP28 interface/QSFP28A_TX4_N -> /QSFP28 interface/QSFP28A_TX3_P
- J15 pad 6: /QSFP28 interface/QSFP28A_TX4_P -> /QSFP28 interface/QSFP28A_TX3_N
- U1 pad 1: unconnected-(U1-Pad1) -> /Power Supply/VCCINT_PGOOD
- U1 pad 10: /Management/MCU_READY -> /Power Supply/3V3_EN
- U1 pad 11: /FPGA support/FPGA_RESET_N_3V3 -> /Power Supply/3V3_PGOOD
- U1 pad 12: /Management/MCU_RST_N -> /Power Supply/GTY_VCC_EN
- U1 pad 18: /Power Supply/3V3_PGOOD -> /FPGA support/FPGA_RESET_N_3V3
- U1 pad 2: unconnected-(U1-Pad2) -> /Power Supply/VCCINT_EN
- U1 pad 20: /Power Supply/3V3_EN -> /Management/MCU_READY
- U1 pad 21: /Power Supply/GTY_VCC_EN -> /Management/MCU_RST_N
- U1 pad 27: /Power Supply/1V8_EN -> /Power Supply/GTY_VCCAUX_PGOOD
- U1 pad 28: /Power Supply/1V8_PGOOD -> /Power Supply/GTY_VCCAUX_EN_N
- U1 pad 3: /Power Supply/GTY_VCCAUX_EN_N -> /Power Supply/1V8_PGOOD
- U1 pad 30: /Power Supply/SUPER_I2C_SCL -> /Power Supply/GTY_VTT_EN
- U1 pad 31: /Power Supply/SUPER_I2C_SDA -> unconnected-(U1-Pad31)
- U1 pad 32: /Power Supply/VCCINT_PGOOD -> unconnected-(U1-Pad32)
- U1 pad 39: /Power Supply/VCCINT_EN -> unconnected-(U1-Pad39)
- U1 pad 4: /Power Supply/GTY_VCCAUX_PGOOD -> /Power Supply/1V8_EN
- U1 pad 41: /Power Supply/GTY_VTT_EN -> unconnected-(U1-Pad41)
- U1 pad 45: unconnected-(U1-Pad45) -> /Power Supply/SUPER_I2C_SCL
- U1 pad 46: unconnected-(U1-Pad46) -> /Power Supply/SUPER_I2C_SDA
Routing:
- net /3V3_SB: track 17.6 -> 198.2 mm, vias 2 -> 8
- net /GND: track 2599.0 -> 2732.0 mm, vias 1022 -> 1055
- net /Power Supply/RST_N: track 0.00 -> 64.9 mm, vias 0 -> 1
- net /Power Supply/SUPER_I2C_SCL: track 3.62 -> 66.8 mm, vias 0 -> 2
- net /Power Supply/SUPER_I2C_SDA: track 4.12 -> 64.5 mm, vias 0 -> 2
- net /QSFP28 interface/QSFP28A_TX4_P: track 5.87 -> 55.3 mm, vias 1 -> 2
- net /QSFP28 interface/QSFP28A_TX4_N: track 5.82 -> 54.6 mm, vias 1 -> 2
- net /Power Supply/SUPER_SWDIO: track 0.00 -> 48.8 mm, vias 0 -> 1
- net /Power Supply/SUPER_SWCLK: track 0.00 -> 45.4 mm, vias 0 -> 1
- net /Power Supply/SOFT_POWER: track 1.00 -> 44.1 mm, vias 0 -> 3
- net /QSFP28 interface/QSFP28A_TX3_P: track 13.1 -> 54.3 mm, vias 1 -> 2
- net /QSFP28 interface/QSFP28A_TX3_N: track 13.1 -> 54.2 mm, vias 1 -> 2
- net /QSFP28 interface/QSFP28A_TX1_P: track 16.8 -> 57.4 mm, vias 1 -> 2
- net /QSFP28 interface/QSFP28A_TX1_N: track 16.9 -> 57.5 mm, vias 1 -> 2
- net /QSFP28 interface/QSFP28A_RX3_N: track 7.66 -> 44.4 mm
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Other:
- board text added: "POWER"
- board text added: "RESET"
- board text added: "RST#"
- board text added: "RX"
- board text added: "SUPER UART"
- board text added: "SWCLK"
- board text added: "SWDIO"
- board text added: "TX"
