File: kup-lulz/smpm.kicad_sch (KiCad schematic)
At the start: 34 parts, among them J17 SMPM, J18 SMPM, J19 SMPM, J20 SMPM, J21 SMPM, J22 SMPM, J23 SMPM, J24 SMPM, J25 SMPM, J26 SMPM, J27 SMPM, J28 SMPM, J29 SMPM, J30 SMPM, J31 SMPM, J32 SMPM, U9 XILINX_ULTRASCALEPLUS_B676

Commit message: Continued initial work on kup-lulz devboard
Parts:
- R81: footprint (none) -> azonenberg_pcb:EIA_0402_RES_NOSILK
Connections:
- net K_REFCLK_0_N: no longer names the net of U9.AB6 (MGTREFCLK0N_224)
- net K_REFCLK_0_P: no longer names the net of U9.AB7 (MGTREFCLK0P_224)
- net K_REFCLK_1_N: no longer names the net of U9.Y6 (MGTREFCLK1N_224)
- net K_REFCLK_1_P: no longer names the net of U9.Y7 (MGTREFCLK1P_224)
- no-connect marks 0 -> 4
Changed lines of the file:
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@@
   (title_block
     (title "Kintex Ultrascale+ OshPark For The Lulz")
-    (date "2024-01-31")
+    (date "2024-02-01")
     (rev "0.1")
   )
   (junction (at 189.23 49.53) (diameter 0) (color 0 0 0 0)
   )
+  (no_connect (at 204.47 34.29))
+  (no_connect (at 204.47 41.91))
+  (no_connect (at 204.47 36.83))
+  (no_connect (at 204.47 44.45))
   (wire (pts (xy 38.1 119.38) (xy 38.1 121.92))
     (stroke (width 0) (type default) (color 0 0 0 0))
@@
   (label "K_RX_1_N" (at 204.47 67.31 180)
     (effects (font (size 1.27 1.27)) (justify right bottom))
-  )
-  (hierarchical_label "K_REFCLK_0_N" (shape input) (at 204.47 36.83 180)
-    (effects (font (size 1.27 1.27)) (justify right))
   )
   (hierarchical_label "GTY_VTT" (shape input) (at 187.96 49.53 180)
     (effects (font (size 1.27 1.27)) (justify right))
   )
-  (hierarchical_label "K_REFCLK_1_P" (shape input) (at 204.47 41.91 180)
-    (effects (font (size 1.27 1.27)) (justify right))
-  )
-  (hierarchical_label "K_REFCLK_0_P" (shape input) (at 204.47 34.29 180)
-    (effects (font (size 1.27 1.27)) (justify right))
-  )
   (hierarchical_label "GND" (shape input) (at 38.1 44.45 180)
-    (effects (font (size 1.27 1.27)) (justify right))
-  )
-  (hierarchical_label "K_REFCLK_1_N" (shape input) (at 204.47 44.45 180)
     (effects (font (size 1.27 1.27)) (justify right))
   )
@@
     (property "Reference" "R81" (id 0) (at 198.12 48.26 90))
     (property "Value" "100" (id 1) (at 194.31 49.53 90))
-    (property "Footprint" "" (id 2) (at 194.31 51.308 90)
-      (effects (font (size 1.27 1.27)) hide)
-    )
+    (property "Footprint" "azonenberg_pcb:EIA_0402_RES_NOSILK" (id 2) (at 194.31 51.308 90)
+      (effects (font (size 1.27 1.27)) hide)
+    )

Commit message: Continued initial layout of kup-lulz
Connections:
- net K_RX_0_N: now also C95.2; no longer C96.2
- net K_RX_0_P: now also C96.2; no longer C95.2
- net K_TX_0_N: now also C103.2; no longer C104.2
- net K_TX_0_P: now also C104.2; no longer C103.2
- net K_TX_1_N: now also C105.2; no longer C106.2
- net K_TX_1_P: now also C106.2; no longer C105.2
- net K_TX_2_N: now also C107.2; no longer C108.2
- net K_TX_2_P: now also C108.2; no longer C107.2
- net K_TX_3_N: now also C109.2; no longer C110.2
- net K_TX_3_P: now also C110.2; no longer C109.2
Other:
- company: (none) -> Antikernel Labs
Changed lines of the file:
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@@
   (title_block
     (title "Kintex Ultrascale+ OshPark For The Lulz")
-    (date "2024-02-01")
+    (date "2024-02-05")
     (rev "0.1")
+    (company "Antikernel Labs")
+    (comment 1 "Andrew D. Zonenberg")
   )
   (junction (at 189.23 49.53) (diameter 0) (color 0 0 0 0)
@@
     (effects (font (size 1.27 1.27)) (justify right bottom))
   )
-  (label "K_TX_0_P" (at 104.14 38.1 0)
-    (effects (font (size 1.27 1.27)) (justify left bottom))
-  )
-  (label "K_RX_0_P" (at 58.42 38.1 0)
+  (label "K_TX_0_P" (at 104.14 50.8 0)
+    (effects (font (size 1.27 1.27)) (justify left bottom))
+  )
+  (label "K_RX_0_P" (at 58.42 50.8 0)
     (effects (font (size 1.27 1.27)) (justify left bottom))
   )
@@
     (effects (font (size 1.27 1.27)) (justify right bottom))
   )
-  (label "K_TX_0_N" (at 104.14 50.8 0)
+  (label "K_TX_0_N" (at 104.14 38.1 0)
     (effects (font (size 1.27 1.27)) (justify left bottom))
   )
@@
     (effects (font (size 1.27 1.27)) (justify left bottom))
   )
-  (label "K_TX_2_N" (at 104.14 101.6 0)
+  (label "K_TX_2_N" (at 104.14 88.9 0)
     (effects (font (size 1.27 1.27)) (justify left bottom))
   )
@@
     (effects (font (size 1.27 1.27)) (justify left bottom))
   )
-  (label "K_TX_2_P" (at 104.14 88.9 0)
+  (label "K_TX_2_P" (at 104.14 101.6 0)
     (effects (font (size 1.27 1.27)) (justify left bottom))
   )
@@
     (effects (font (size 1.27 1.27)) (justify right bottom))
   )
-  (label "K_RX_0_N" (at 58.42 50.8 0)
+  (label "K_RX_0_N" (at 58.42 38.1 0)
     (effects (font (size 1.27 1.27)) (justify left bottom))
   )
@@
     (effects (font (size 1.27 1.27)) (justify left bottom))
   )
-  (label "K_TX_3_P" (at 104.14 114.3 0)
+  (label "K_TX_3_P" (at 104.14 127 0)
     (effects (font (size 1.27 1.27)) (justify left bottom))
   )
@@
     (effects (font (size 1.27 1.27)) (justify right bottom))
   )
-  (label "K_TX_1_P" (at 104.14 63.5 0)
-    (effects (font (size 1.27 1.27)) (justify left bottom))
-  )
-  (label "K_TX_3_N" (at 104.14 127 0)
+  (label "K_TX_1_P" (at 104.14 76.2 0)
+    (effects (font (size 1.27 1.27)) (justify left bottom))
+  )
+  (label "K_TX_3_N" (at 104.14 114.3 0)
     (effects (font (size 1.27 1.27)) (justify left bottom))
   )
@@
     (effects (font (size 1.27 1.27)) (justify right bottom))
   )
-  (label "K_TX_1_N" (at 104.14 76.2 0)
-    (effects (font (size 1.27 1.27)) (justify left bottom))
-  )
+  (label "K_TX_1_N" (at 104.14 63.5 0)
+    (effects (font (size 1.27 1.27)) (justify left bottom))
+  )
