File: kup-lulz/mgmt.kicad_sch (KiCad schematic)
At the start: 55 parts, among them J38 PMOD_HOST, J39 CONN_01X03, J4 CORTEX_DEBUG_ETM, U14 STM32H735-UFBGA176-25, U15 AT24MAC402, U6 ECS-1612MV-250-CN, U9 XILINX_ULTRASCALEPLUS_B676

Commit message: Finished initial routing of new processor
Connections:
- net MCU_PMOD_DQ0: now also U14.B3 (PB9); no longer U14.R6 (PC4)
- net MCU_PMOD_DQ1: now also U14.C1 (PC13); no longer U14.C6 (PB5)
- net MCU_PMOD_DQ2: now also U14.A2 (PB8); no longer U14.P1 (PA0)
- net MCU_PMOD_DQ4: now also U14.D1 (PC15); no longer U14.C7 (PG14)
- net MCU_PMOD_DQ5: now also U14.B1 (PE4); no longer U14.P7 (PB2)
- net MCU_PMOD_DQ6: now also U14.B4 (PE0); no longer U14.R7 (PA6)
- net MCU_READY: now also U14.R12 (PE11); no longer U14.P6 (PA5)
- net MGMT_SPI_CS_N: now also U9.AB15 (IO_L6P_HDGC_AD6P_84); no longer U9.W15 (IO_L10N_AD2N_84)
- net MGMT_SPI_DQ0: now also U9.Y15 (IO_L7P_HDGC_AD5P_84); no longer U9.AA15 (IO_L7N_HDGC_AD5N_84)
- net MGMT_SPI_DQ1: now also U9.AB16 (IO_L6N_HDGC_AD6N_84); no longer U9.AB15 (IO_L6P_HDGC_AD6P_84)
- net MGMT_SPI_DQ2: now also U9.W15 (IO_L10N_AD2N_84); no longer U9.W13 (IO_L12N_AD0N_84)
- net MGMT_SPI_DQ3: now also U9.W13 (IO_L12N_AD0N_84); no longer U9.Y15 (IO_L7P_HDGC_AD5P_84)
- net MGMT_SPI_SCK: now also U9.AA14 (IO_L8P_HDGC_AD4P_84); no longer U9.AB16 (IO_L6N_HDGC_AD6N_84)
- net SOFT_RESET: now also U14.P2 (PA1); no longer U14.M7 (PC5)
- net SUPER_SPI_CS_N: now also U14.P1 (PA0); no longer U14.H1 (PF6)
Changed lines of the file:
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@@
 	)
 	(no_connect
+		(at 142.24 166.37)
+	)
+	(no_connect
 		(at 92.71 280.67)
 	)
@@
 	)
 	(no_connect
-		(at 92.71 173.99)
-	)
-	(no_connect
 		(at 387.35 320.04)
 	)
@@
 	)
 	(no_connect
-		(at 41.91 153.67)
-	)
-	(no_connect
 		(at 101.6 85.09)
 	)
@@
 	)
 	(no_connect
+		(at 142.24 219.71)
+	)
+	(no_connect
 		(at 142.24 232.41)
 	)
@@
 	)
 	(no_connect
+		(at 41.91 168.91)
+	)
+	(no_connect
 		(at 142.24 158.75)
 	)
@@
 	)
 	(no_connect
-		(at 92.71 205.74)
-	)
-	(no_connect
 		(at 382.27 167.64)
 	)
@@
 	)
 	(no_connect
-		(at 92.71 176.53)
+		(at 142.24 189.23)
 	)
 	(no_connect
-		(at 142.24 189.23)
+		(at 92.71 158.75)
 	)
 	(no_connect
@@
 	)
 	(no_connect
+		(at 92.71 166.37)
+	)
+	(no_connect
 		(at 382.27 106.68)
 	)
@@
 	)
 	(no_connect
-		(at 92.71 215.9)
-	)
-	(no_connect
 		(at 382.27 109.22)
 	)
@@
 	)
 	(no_connect
-		(at 142.24 186.69)
+		(at 382.27 165.1)
 	)
 	(no_connect
-		(at 382.27 165.1)
+		(at 142.24 163.83)
 	)
 	(no_connect
@@
 	)
 	(no_connect
-		(at 171.45 85.09)
-	)
-	(no_connect
-		(at 92.71 233.68)
+		(at 92.71 210.82)
 	)
 	(no_connect
-		(at 92.71 210.82)
+		(at 41.91 166.37)
 	)
 	(no_connect
@@
 	)
 	(no_connect
-		(at 142.24 191.77)
-	)
-	(no_connect
 		(at 382.27 99.06)
 	)
@@
 	)
 	(no_connect
+		(at 41.91 295.91)
+	)
+	(no_connect
 		(at 41.91 179.07)
 	)
@@
 	)
 	(no_connect
+		(at 171.45 87.63)
+	)
+	(no_connect
 		(at 101.6 82.55)
 	)
@@
 	)
 	(label "MCU_PMOD_DQ4"
-		(at 41.91 295.91 180)
+		(at 142.24 191.77 180)
 		(fields_autoplaced yes)
 		(effects
@@
 	)
 	(label "MCU_PMOD_DQ0"
-		(at 142.24 163.83 180)
+		(at 92.71 176.53 180)
 		(fields_autoplaced yes)
 		(effects
@@
 	)
 	(label "MCU_PMOD_DQ5"
-		(at 92.71 158.75 180)
+		(at 92.71 215.9 180)
 		(fields_autoplaced yes)
 		(effects
@@
 		)
 	)
-	(label "MCU_RST_N"
-		(at 387.35 309.88 180)
-		(fields_autoplaced yes)
-		(effects
-			(font
-				(size 1.27 1.27)
-			)
-			(justify right bottom)
-		)
-	)
 	(label "MCU_JTAG_TMS"
 		(at 41.91 186.69 180)
@@
 	)
 	(label "MGMT_SPI_DQ3"
-		(at 171.45 90.17 180)
+		(at 171.45 62.23 180)
 		(fields_autoplaced yes)
 		(effects
@@
 	)
 	(label "MGMT_SPI_DQ0"
-		(at 171.45 87.63 180)
+		(at 171.45 90.17 180)
 		(fields_autoplaced yes)
 		(effects
@@
 	)
 	(label "MGMT_SPI_DQ2"
-		(at 171.45 62.23 180)
+		(at 171.45 72.39 180)
 		(fields_autoplaced yes)
 		(effects
@@
 	)
 	(label "MGMT_SPI_DQ1"
-		(at 171.45 95.25 180)
+		(at 171.45 92.71 180)
 		(fields_autoplaced yes)
 		(effects
@@
 	)
 	(label "MCU_PMOD_DQ2"
-		(at 41.91 148.59 180)
+		(at 92.71 173.99 180)
 		(fields_autoplaced yes)
 		(effects
@@
 	)
 	(label "MGMT_SPI_CS_N"
-		(at 171.45 72.39 180)
+		(at 171.45 95.25 180)
 		(fields_autoplaced yes)
 		(effects
@@
 	)
 	(label "MCU_PMOD_DQ6"
-		(at 41.91 168.91 180)
+		(at 92.71 205.74 180)
 		(fields_autoplaced yes)
 		(effects
@@
 	)
 	(label "MCU_PMOD_DQ1"
-		(at 92.71 166.37 180)
+		(at 142.24 186.69 180)
 		(fields_autoplaced yes)
 		(effects
@@
 	)
 	(label "MGMT_SPI_SCK"
-		(at 171.45 92.71 180)
+		(at 171.45 85.09 180)
 		(fields_autoplaced yes)
 		(effects
@@
 	(hierarchical_label "SOFT_RESET"
 		(shape output)
-		(at 142.24 166.37 180)
+		(at 41.91 153.67 180)
 		(fields_autoplaced yes)
 		(effects
@@
 	(hierarchical_label "MCU_READY"
 		(shape output)
-		(at 41.91 166.37 180)
+		(at 92.71 233.68 180)
 		(fields_autoplaced yes)
 		(effects
@@
 	(hierarchical_label "SUPER_SPI_CS_N"
 		(shape output)
-		(at 142.24 219.71 180)
+		(at 41.91 148.59 180)
 		(fields_autoplaced yes)
 		(effects
@@
 		)
 	)
+	(hierarchical_label "MCU_RST_N"
+		(shape input)
+		(at 387.35 309.88 180)
+		(fields_autoplaced yes)
+		(effects
+			(font
+				(size 1.27 1.27)
+			)
+			(justify right)
+		)
+	)
 	(hierarchical_label "SFP2_TX_DISABLE"
 		(shape output)
@@
 		)
 		(pin "H1"
-			(alternate "SPI5_NSS")
 		)
 		(pin "P4"
@@
 		)
 		(pin "H1"
-			(alternate "SPI5_NSS")
 		)
 		(pin "P4"
@@
 		)
 		(pin "H1"
-			(alternate "SPI5_NSS")
 		)
 		(pin "P4"
@@
 		)
 		(pin "H1"
-			(alternate "SPI5_NSS")
 		)
 		(pin "P4"
@@
 		)
 		(pin "H1"
-			(alternate "SPI5_NSS")
 		)
 		(pin "P4"
@@
 		)
 		(pin "H1"
-			(alternate "SPI5_NSS")
 		)
 		(pin "P4"
@@
 		)
 		(pin "H1"
-			(alternate "SPI5_NSS")
 		)
 		(pin "P4"
@@
 		)
 		(pin "H1"
-			(alternate "SPI5_NSS")
 		)
 		(pin "P4"
@@
 		)
 		(pin "H1"
-			(alternate "SPI5_NSS")
 		)
 		(pin "P4"
@@
 		)
 		(pin "H1"
-			(alternate "SPI5_NSS")
 		)
 		(pin "P4"
@@
 		)
 		(pin "H1"
-			(alternate "SPI5_NSS")
 		)
 		(pin "P4"
