File: kup-lulz/fpgasupport.kicad_sch (KiCad schematic)
At the start: 51 parts, among them J5 JUMPER_0402, J6 XILINX_JTAG, U10 MT25QU256ABA8E12-0AUT, U11 74LVC1T45, U12 74LVC1T45, U13 74LVC1T45, U9 XILINX_ULTRASCALEPLUS_B676

Commit message: Final kup-lulz design ready for fab
Parts:
- added C157, C158, C159, C160, C161, C162: 4.7 uF, azonenberg_pcb:EIA_0603_CAP_NOSILK, symbol device:C
Connections:
- net GND: now also C157.2, C158.2, C159.2, C160.2, C161.2, C162.2
- net GTY_VCC: now also C157.1, C162.1
- net GTY_VCCAUX: now also C159.1, C160.1
- net GTY_VTT: now also C158.1, C161.1
Other:
- note added: "GTY decoupling We have only one power supply group, so one set of caps is probably enough on a good board Add two to compensate for very inductive PDN layout"
