File: kup-lulz/psu.kicad_sch (KiCad schematic)
At the start: 110 parts, among them J1 CONN_PCIE_PWR_8PIN, J13 FAN_01, J2 CONN_IBC_MGMT, J3 CONN_01X03, J4 CONN_01X05, Q1 SSM6N58NU, SW1 SWITCH, SW2 SWITCH, U1 STM32L031C6U6, U2 MYMGK1R812ERSR, U3 MYMGK1R812ERSR, U4 MYMGK00506ERSR, U5 MYMGK00504ERSR, U7 MYMGK00504ERSR, U8 ADP1740ACPZ-1.8-R7

Commit message: Replaced supervisor with L431
Parts:
- removed J4: CONN_01X05, azonenberg_pcb:CONN_HEADER_2.54MM_1x5, symbol conn:CONN_01X05
- removed U1: STM32L031C6U6, azonenberg_pcb:QFN_48_0.5MM_7x7MM, symbol st-azonenberg:STM32L031-UFQFPN48
- added C18: 0.47 uF, azonenberg_pcb:EIA_0402_CAP_NOSILK, symbol device:C
- added J41: CORTEX_DEBUG_ETM, azonenberg_pcb:CONN_HEADER_1.27MM_2x10_SMT_SAMTEC_FTSH-110-01-L-DV-K, symbol special-azonenberg:CORTEX_DEBUG_ETM
- added unit 2 of Q1
- added R22: 10K, azonenberg_pcb:EIA_0402_RES_NOSILK, symbol device:R
- added U1: STM32L431-QFN48, azonenberg_pcb:QFN_48_0.5MM_7x7MM, symbol st-azonenberg:STM32L431-QFN48
Connections:
- net 12V0_VMON: now also U1.19 (PB1)
- net 1V8_EN: now also U1.4 (PC15)
- net 1V8_PGOOD: now also U1.3 (PC14)
- net 3V3_EN: now also U1.10 (PA0)
- net 3V3_PGOOD: now also U1.11 (PA1)
- net 3V3_SB: now also C18.1, J41.1 (VCC), R22.2, U1.1 (VBAT), U1.24 (VDD), U1.36 (VDD), U1.48 (VDD)
- net A3V3_SUPER: now also U1.9 (VDDA)
- net BOOT0: now also U1.44 (BOOT0)
- net FAN1_PWM: now also U1.12 (PA2)
- net FAN1_TACH: now also U1.45 (PB8)
- net FPGA_DONE: now also U1.21 (PB10)
- net FPGA_INIT: now also U1.20 (PB2)
- net FPGA_RST_N: now also U1.25 (PB12)
- net GND: now also C18.2, J41.11 (GND), J41.13 (GND), J41.15 (GND), J41.17 (GND), J41.19 (GND), J41.3 (GND), J41.5 (GND), J41.9 (GNDdet), Q1.D2 (D), Q1.G2 (G), Q1.S2 (S), U1.23 (GND), U1.35 (GND), U1.47 (GND), U1.8 (VSSA), U1.PAD (GND)
- net GTY_VCCAUX_EN_N: now also U1.32 (PA11)
- net GTY_VCCAUX_PGOOD: now also U1.29 (PA8)
- net GTY_VCC_EN: now also U1.13 (PA3)
- net GTY_VCC_PGOOD: now also U1.18 (PB0)
- net GTY_VTT_EN: now also U1.27 (PB14)
- net GTY_VTT_PGOOD: now also U1.28 (PB15)
- net MCU_READY: now also U1.22 (PB11)
- net MCU_RST_N: now also U1.46 (PB9)
- net SOFT_POWER: now also U1.33 (PA12)
- net SOFT_RESET: now also U1.41 (PB5)
- net SUPER_I2C_SCL: now also U1.42 (PB6)
- net SUPER_I2C_SDA: now also U1.43 (PB7)
- net SUPER_LED0: now also U1.5 (PH0)
- net SUPER_LED1: now also U1.6 (PH1)
- net SUPER_SPI_CS_N: now also U1.14 (PA4)
- net SUPER_SPI_MISO: now also U1.16 (PA6)
- net SUPER_SPI_MOSI: now also U1.17 (PA7)
- net SUPER_SPI_SCK: now also U1.15 (PA5)
- net SUPER_UART_RX: now also U1.31 (PA10)
- net SUPER_UART_TX: now also U1.30 (PA9)
- net VCCINT_EN: now also U1.2 (PC13)
- net VCCINT_PGOOD: now also U1.26 (PB13)
- net RST_N renamed SUPER_RST_N
- net SUPER_RST_N: now also J41.10 (~{RST}), U1.7 (NRST)
- new net SUPER_JTAG_TCK: J41.4 (TCK), U1.37 (PA14)
- new net SUPER_JTAG_TDI: J41.8 (TDI), U1.38 (PA15)
- new net SUPER_JTAG_TDO: J41.6 (TDO), U1.39 (PB3)
- new net SUPER_JTAG_TMS: J41.2 (TMS), U1.34 (PA13)
- new net SUPER_JTAG_TRST: R22.1, U1.40 (PB4)
- no-connect marks 4 -> 5
Other:
- note added: "PGOOD pin for all MYMGK1R812 rails (VCCINT, GTY_VTT) is pulled up to 5V internally, need to be on 5V tolerant pin. Other regs have external pullups to 3V3_SB"
- note removed: "PGOOD pin for all MYMGK1R812 rails is pulled up to 5V internally, need to be on 5V tolerant pin. Other regs have external pullups to 3V3_SB"
- moved on the sheet: C22, R12, R15, R9, TP7, TP8

Commit message: Final kup-lulz design ready for fab
Parts:
- D1, D2: footprint azonenberg_pcb:EIA_0603_LED -> azonenberg_pcb:EIA_0402_LED
- J3, TP7: footprint azonenberg_pcb:CONN_HEADER_2.54MM_1x3 -> azonenberg_pcb:CONN_HEADER_2.54MM_1x3_REFLOW
- R13: value 470 -> 33K
- R14: value 470 -> 4.7K
- TP8: footprint azonenberg_pcb:CONN_HEADER_2.54MM_1x5 -> azonenberg_pcb:CONN_HEADER_2.54MM_1x5_REFLOW
Changed lines of the file:
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@@
 	(title_block
 		(title "Kintex Ultrascale+ OshPark For The Lulz")
-		(date "2024-11-10")
+		(date "2024-11-13")
 		(rev "0.1")
 		(company "Antikernel Labs")
@@
 			)
 		)
-		(property "Footprint" "azonenberg_pcb:EIA_0603_LED"
+		(property "Footprint" "azonenberg_pcb:EIA_0402_LED"
 			(at 215.9 341.63 0)
 			(effects
@@
 		(fields_autoplaced yes)
 		(property "Reference" "R13"
-			(at 208.28 336.9142 90)
+			(at 208.28 336.4695 90)
 			(effects
 				(font
@@
 			)
 		)
-		(property "Value" "470"
-			(at 208.28 339.4511 90)
+		(property "Value" "33K"
+			(at 208.28 338.8938 90)
 			(effects
 				(font
@@
 			)
 		)
-		(property "Footprint" "azonenberg_pcb:CONN_HEADER_2.54MM_1x3"
+		(property "Footprint" "azonenberg_pcb:CONN_HEADER_2.54MM_1x3_REFLOW"
 			(at 294.64 370.84 0)
 			(effects
@@
 			)
 		)
-		(property "Footprint" "azonenberg_pcb:CONN_HEADER_2.54MM_1x3"
+		(property "Footprint" "azonenberg_pcb:CONN_HEADER_2.54MM_1x3_REFLOW"
 			(at 292.1 396.24 0)
 			(effects
@@
 			)
 		)
-		(property "Footprint" "azonenberg_pcb:EIA_0603_LED"
+		(property "Footprint" "azonenberg_pcb:EIA_0402_LED"
 			(at 215.9 351.79 0)
 			(effects
@@
 		(fields_autoplaced yes)
 		(property "Reference" "R14"
-			(at 208.28 347.0742 90)
+			(at 208.28 346.6295 90)
 			(effects
 				(font
@@
 			)
 		)
-		(property "Value" "470"
-			(at 208.28 349.6111 90)
+		(property "Value" "4.7K"
+			(at 208.28 349.0538 90)
 			(effects
 				(font
@@
 			)
 		)
-		(property "Footprint" "azonenberg_pcb:CONN_HEADER_2.54MM_1x5"
+		(property "Footprint" "azonenberg_pcb:CONN_HEADER_2.54MM_1x5_REFLOW"
 			(at 325.12 398.78 0)
 			(effects
