File: symmetricom-breakout/symmetricom-breakout.kicad_pcb (KiCad board)
At the start: 4 copper layers, 77 x 56.5 mm, 42 parts, among them J1 BARREL_JACK, J2 SMA, J3 SMA, J4 SMA, J5 CONN_01X03, M1 SCREWHOLE, M2 SCREWHOLE, M3 SCREWHOLE, M4 SCREWHOLE, M5 LOGO, M6 LOGO, M7 LOGO, M8 LOGO, U1 SA22C, U2 MUN12AD03-SE, U3 74LVC1T45, U4 74LVC1T45, U5 MIC5353

Commit message: Updated symmetricom breakout after review
Parts:
- moved R2 0.25 mm to (113.0, 49.8)
- moved R1 0.15 mm to (113.9, 50.8)
Changed lines of the file:
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@@
 			(outputformat 1)
 			(mirror no)
-			(drillshape 1)
+			(drillshape 0)
 			(scaleselection 1)
-			(outputdirectory "")
+			(outputdirectory "output/")
 		)
 	)
@@
 		(at 131 45.5 90)
 		(property "Reference" "R4"
-			(at 0 1.5 90)
+			(at 0 1.5 -90)
 			(unlocked yes)
 			(layer "F.SilkS")
@@
 	(footprint "azonenberg_pcb:EIA_0402_RES_NOSILK"
 		(layer "F.Cu")
-		(at 113.75 50.75 90)
+		(at 113.9 50.75 90)
 		(property "Reference" "R1"
-			(at 1.75 0 90)
+			(at 1.75 0.25 -90)
 			(unlocked yes)
 			(layer "F.SilkS")
@@
 		(at 111.5 44 180)
 		(property "Reference" "R5"
-			(at 0 1.5 180)
+			(at -1.7 0 0)
 			(unlocked yes)
 			(layer "F.SilkS")
@@
 		(at 112 45.499999 90)
 		(property "Reference" "R3"
-			(at 0 1.5 90)
+			(at 0 0.8 -90)
 			(unlocked yes)
 			(layer "F.SilkS")
@@
 	(footprint "azonenberg_pcb:EIA_0402_RES_NOSILK"
 		(layer "F.Cu")
-		(at 112.75 49.75 90)
+		(at 113 49.75 90)
 		(property "Reference" "R2"
-			(at 1.75 0 90)
+			(at 1.75 0 -90)
 			(unlocked yes)
 			(layer "F.SilkS")
@@
 	)
 	(segment
-		(start 112.75 49.250001)
-		(end 112.75 48.75)
-		(width 0.125)
-		(layer "F.Cu")
-		(net 1)
-	)
-	(segment
 		(start 108.75 54.25)
 		(end 107.1 54.25)
@@
 	)
 	(segment
+		(start 113 49.250001)
+		(end 113 49)
+		(width 0.125)
+		(layer "F.Cu")
+		(net 1)
+	)
+	(segment
 		(start 122 73.5)
 		(end 122 71.5)
@@
 		(width 0.125)
 		(layer "F.Cu")
+		(net 1)
+	)
+	(segment
+		(start 113 49)
+		(end 112.75 48.75)
+		(width 0.125)
+		(layer "F.Cu")
