File: fpga-stm32-ifaces/power-support.kicad_sch (KiCad schematic)
At the start: 2 parts, among them U1 STM32H735-UFBGA176-25, U2 XC7S25-1FTGB196

Commit message: Finished initial schematic of fpga-stm32-ifaces board, waiting for sch review
Parts:
- added C100, C106, C107, C108, C109, C110, C111, C112, C113, C71, C72, C73, C75, C76, C77, C78, C79, C80, C81, C82, C90, C91, C92, C93, C94, C95, C98, C99: 0.47 uF, azonenberg_pcb:EIA_0402_CAP_NOSILK, symbol device:C
- added C101, C83, C84: 100 uF, symbol device:C
- added C102, C103, C104, C105, C62, C63, C66, C68, C70, C86, C87, C88, C89, C97: 4.7 uF, azonenberg_pcb:EIA_0603_CAP_NOSILK, symbol device:C
- added C59, C61, C64: 10 uF, azonenberg_pcb:EIA_0805_CAP_NOSILK, symbol device:C
- added C60: 220 pF, azonenberg_pcb:EIA_0402_CAP_NOSILK, symbol device:C
- added C65, C69: 2.2 uF, azonenberg_pcb:EIA_0805_CAP_NOSILK, symbol device:C
- added C67: 0.1 uF, azonenberg_pcb:EIA_0402_CAP_NOSILK, symbol device:C
- added C74: 22 uF, azonenberg_pcb:EIA_0805_CAP_NOSILK, symbol device:C
- added C85, C96: 47 uF, symbol device:C
- added FB7: MI0603J601R-10, azonenberg_pcb:EIA_0603_INDUCTOR_NOSILK, symbol passive-azonenberg:FERRITE_SMALL2
- added L1: 2.2 uH, azonenberg_pcb:EIA_1210_CAP_NOSILK, symbol passive-azonenberg:INDUCTOR_PWROUT
- added TP12, TP13, TP14: U.FL, azonenberg_pcb:CONN_U.FL_TE_1909763-1, symbol conn:CONN_COAXIAL
Connections:
- net GND: now reaches U1.A1 (VSS)
- net GND: now also U1.A15 (VSS), U1.C2 (VSS), U1.D10 (VSS), U1.D6 (VSS), U1.E1 (VSS), U1.F10 (VSS), U1.F12 (VSS), U1.F2 (VSSSMPS), U1.F6 (VSS), U1.F7 (VSS), U1.F8 (VSS), U1.F9 (VSS), U1.G10 (VSS), U1.G6 (VSS), U1.G7 (VSS), U1.G8 (VSS), U1.G9 (VSS), U1.H10 (VSS), U1.H6 (VSS), U1.H7 (VSS), U1.H8 (VSS), U1.H9 (VSS), U1.J10 (VSS), U1.J14 (VSS), U1.J6 (VSS), U1.J7 (VSS), U1.J8 (VSS), U1.J9 (VSS), U1.K10 (VSS), U1.K12 (VSS), U1.K2 (VSS), U1.K6 (VSS), U1.K7 (VSS), U1.K8 (VSS), U1.K9 (VSS), U1.M10 (VSS), U1.M6 (VSS), U1.N3 (VSSA), U1.R1 (VSS), U1.R15 (VSS), U2.A1 (GND), U2.A11 (GND), U2.A14 (GND), U2.A6 (GND), U2.A9 (GND), U2.B4 (GND), U2.B7 (GND), U2.B9 (GND), U2.C13 (GND), U2.C2 (GND), U2.C6 (GND), U2.C7 (GND), U2.C8 (GND), U2.C9 (GND), U2.D11 (GND), U2.D5 (GND), U2.D7 (GND), U2.D9 (GND), U2.E1 (GND), U2.E10 (GND), U2.E14 (GND), U2.E3 (GND), U2.E6 (GND), U2.E8 (GND), U2.F5 (GND), U2.F7 (GNDADC_0), U2.F9 (GND), U2.G10 (GND), U2.G12 (GND), U2.G3 (GND), U2.G6 (GND), U2.H5 (GND), U2.H9 (GND), U2.J10 (GND), U2.J6 (GND), U2.K1 (GND), U2.K14 (GND), U2.K5 (GND), U2.K7 (GND), U2.K9 (GND), U2.L10 (GND), U2.L11 (GND), U2.L4 (GND), U2.L6 (GND), U2.L8 (GND), U2.N12 (GND), U2.N3 (GND), U2.N5 (GND), U2.N9 (GND), U2.P1 (GND), U2.P14 (GND), C100.2, C101.2, C102.2, C103.2, C104.2, C105.2, C106.2, C107.2, C108.2, C109.2, C110.2, C111.2, C112.2, C113.2, C59.2, C60.2, C61.2, C62.2, C63.2, C64.2, C65.2, C66.2, C67.2, C68.2, C69.2, C70.2, C71.2, C72.1, C73.2, C74.2, C75.2, C76.1, C77.2, C78.1, C79.2, C80.1, C81.2, C82.1, C83.2, C84.2, C85.2, C86.2, C87.2, C88.2, C89.2, C90.2, C91.2, C92.2, C93.2, C94.2, C95.2, C96.2, C97.2, C98.2, C99.2, TP12.2 (Ext), TP13.2 (Ext), TP14.2 (Ext)
- net VSMPS: now reaches U1.A13 (VDDLDO)
- net VSMPS: now also U1.A3 (VDDLDO), U1.G2 (VFBSMPS), U1.R14 (VDDLDO), C59.1, C61.1, C63.1, L1.1, TP13.1 (In)
- net VCORE: now reaches U1.A14 (VCAP)
- net VCORE: now also U1.A4 (VCAP), U1.R13 (VCAP), C65.1, C69.1, TP12.1 (In)
- net 3V3: now reaches U1.D11 (VDD)
- net 3V3: now also U1.D5 (VDD), U1.E12 (VDD), U1.E15 (VDD50USB), U1.E4 (VDD), U1.F13 (VDD33USB), U1.G1 (VDDSMPS), U1.G4 (VDD), U1.H12 (VDD), U1.K4 (VDD), U1.L12 (VDD), U1.M5 (VDD), U1.M9 (VDD), U2.G13 (VCCO_14), U2.G2 (VCCO_34), U2.K13 (VCCO_14), U2.K2 (VCCO_34), U2.N13 (VCCO_14), U2.N2 (VCCO_34), U2.N6 (VCCO_0), U2.N8 (VCCO_0), C101.1, C102.1, C103.1, C104.1, C105.1, C106.1, C107.1, C108.1, C109.1, C110.1, C111.1, C112.1, C113.1, C62.1, C64.1, C66.1, C68.1, C71.1, C72.2, C74.1, C75.1, C76.2, C77.1, C78.2, C79.1, C80.2, C81.1, C82.2, FB7.1
- net 3V3_SB: now reaches U1.E2 (VBAT)
- net 3V3_SB: now also C67.1
- net VLXSMPS: now reaches U1.F1 (VLXSMPS)
- net VLXSMPS: now also C60.1, L1.2
- net MCU_VDDA: now reaches U1.M4 (VDDA)
- net MCU_VDDA: now also C70.1, C73.1, FB7.2, TP14.1 (In)
- net 1V8: now reaches U2.B8 (VCCBATT_0)
- net 1V8: now also U2.F10 (VCCAUX), U2.F8 (VCCADC_0), U2.H10 (VCCAUX), U2.K10 (VCCAUX), U2.L9 (VCCAUX), C100.1, C96.1, C97.1, C98.1, C99.1
- net 1V0: now reaches U2.D6 (VCCINT)
- net 1V0: now also U2.D8 (VCCINT), U2.E5 (VCCBRAM), U2.E7 (VCCINT), U2.E9 (VCCINT), U2.F6 (VCCINT), U2.G5 (VCCBRAM), U2.G9 (VCCINT), U2.H6 (VCCINT), U2.J5 (VCCBRAM), U2.J9 (VCCINT), U2.K6 (VCCINT), U2.K8 (VCCINT), C83.1, C84.1, C85.1, C86.1, C87.1, C88.1, C89.1, C90.1, C91.1, C92.1, C93.1, C94.1, C95.1
Other:
- note added: "FPGA VCCAUX"
- note added: "FPGA VCCINT / VCCBRAM"
- note added: "FPGA VCCO"
- note added: "MCU VBAT decoupling"
- note added: "MCU VCAP decoupling"
- note added: "MCU VDD decoupling"
- note added: "MCU VDDA decoupling"
- note added: "MCU VDDLDO decoupling"
- note added: "MCU VDDSMPS decoupling"
- moved on the sheet: U1I, U2A

Commit message: Continued initial layout of fpga-stm32-ifaces
Parts:
- C101, C83, C84, C85, C96: footprint (none) -> azonenberg_pcb:EIA_1210_CAP_NOSILK
- U1: footprint (none) -> azonenberg_pcb:BGA_201_10x10_DEPOP_0.65MM_OSHPARK
- U2: footprint (none) -> azonenberg_pcb:BGA_196_15x15_FULLARRAY_1MM_FTGB196
Other:
- company: (none) -> Antikernel Labs
- title: (none) -> FPGA - STM32 Interface Test
Changed lines of the file:
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@@
 	(generator_version "8.0")
 	(paper "A3")
+	(title_block
+		(title "FPGA - STM32 Interface Test")
+		(date "2024-06-12")
+		(rev "0.1")
+		(company "Antikernel Labs")
+	)
 	(junction
 		(at 67.31 139.7)
@@
 			)
 		)
-		(property "Footprint" ""
+		(property "Footprint" "azonenberg_pcb:BGA_201_10x10_DEPOP_0.65MM_OSHPARK"
 			(at 71.12 156.21 0)
 			(effects
@@
 			)
 		)
-		(property "Footprint" ""
+		(property "Footprint" "azonenberg_pcb:EIA_1210_CAP_NOSILK"
 			(at 195.2752 104.14 0)
 			(effects
@@
 			)
 		)
-		(property "Footprint" ""
+		(property "Footprint" "azonenberg_pcb:EIA_1210_CAP_NOSILK"
 			(at 167.3352 133.35 0)
 			(effects
@@
 			)
 		)
-		(property "Footprint" ""
+		(property "Footprint" "azonenberg_pcb:EIA_1210_CAP_NOSILK"
 			(at 181.3052 104.14 0)
 			(effects
@@
 			)
 		)
-		(property "Footprint" ""
+		(property "Footprint" "azonenberg_pcb:BGA_201_10x10_DEPOP_0.65MM_OSHPARK"
 			(at 71.12 88.9 0)
 			(effects
@@
 			)
 		)
-		(property "Footprint" ""
+		(property "Footprint" "azonenberg_pcb:BGA_196_15x15_FULLARRAY_1MM_FTGB196"
 			(at 332.74 158.75 0)
 			(effects
@@
 			)
 		)
-		(property "Footprint" ""
+		(property "Footprint" "azonenberg_pcb:EIA_1210_CAP_NOSILK"
 			(at 167.3352 104.14 0)
 			(effects
@@
 			)
 		)
-		(property "Footprint" ""
+		(property "Footprint" "azonenberg_pcb:EIA_1210_CAP_NOSILK"
 			(at 167.3352 148.59 0)
 			(effects
