File: fpga-stm32-ifaces/psu.kicad_sch (KiCad schematic)
At the start: 0 parts

Commit message: Finished initial schematic of fpga-stm32-ifaces board, waiting for sch review
Parts:
- added C34, C37, C38, C39, C53, C54: 0.47 uF, azonenberg_pcb:EIA_0402_CAP_NOSILK, symbol device:C
- added C35: 4.7 uF, azonenberg_pcb:EIA_0603_CAP_NOSILK, symbol device:C
- added C36: 0.1 uF, azonenberg_pcb:EIA_0402_CAP_NOSILK, symbol device:C
- added C40: 25SVPF330M, azonenberg_pcb:CAP_AL_10MM_SMT, symbol device:CP1
- added C41, C44, C47, C50: 10 uF, symbol device:C
- added C42, C43, C45, C46, C48, C49, C51, C52: 22 uF, symbol device:C
- added D10, D9: GREEN, symbol device:LED
- added D11: RED, symbol device:LED
- added F1: 2A, azonenberg_pcb:EIA_0603_CAP_NOSILK, symbol power-azonenberg:FUSE_PWROUT_2
- added FB5: MI0603J601R-10, azonenberg_pcb:EIA_0603_INDUCTOR_NOSILK, symbol passive-azonenberg:INDUCTOR_PWROUT
- added FB6: BLM31KN271SH1L, azonenberg_pcb:EIA_1206_CAP_NOSILK, symbol passive-azonenberg:FERRITE_SMALL2
- added J6: CONN_01X03, azonenberg_pcb:CONN_HEADER_2.54MM_1x3, symbol conn:CONN_01X03
- added J7: CONN_PCIE_PWR_8PIN, azonenberg_pcb:CONN_MOLEX_MINIFITJR_8POS_0039291087, symbol power-azonenberg:CONN_PCIE_PWR_8PIN
- added J8: XILINX_JTAG, symbol xilinx-azonenberg:XILINX_JTAG
- added J9: CONN_IBC_MGMT_DEVICE, symbol power-azonenberg:CONN_IBC_MGMT_DEVICE
- added R58: DNP, azonenberg_pcb:EIA_0402_RES_NOSILK, symbol device:R
- added R59: 10K, azonenberg_pcb:EIA_0402_RES_NOSILK, symbol device:R
- added R60, R64, R65: 100K, symbol device:R
- added R61: 22.1K, symbol device:R
- added R62: 200k, symbol device:R
- added R63: 100k, symbol device:R
- added R66: 187K, symbol device:R
- added R67: 280K, symbol device:R
- added R68: 33, symbol device:R
- added R69: 1K, azonenberg_pcb:EIA_0402_RES_NOSILK, symbol device:R
- added R70, R71, R72: 470, symbol device:R
- added TP10, TP5, TP6, TP7, TP8, TP9: U.Fl, symbol conn:CONN_COAXIAL
- added TP11: CONN_01X03, symbol conn:CONN_01X03
- added U11: STM32L431-QFN48, symbol st-azonenberg:STM32L431-QFN48
- added U12, U13, U14, U15: MUN12AD03-SE, symbol power-azonenberg:MUN12AD03-SE
Connections:
- new net: R62.2, R63.1, U13.6 (FB)
- new net: F1.1, J7.1 (12V0), J7.2 (12V0), J7.3 (12V0), J7.4 (12V0_SENSE)
- new net: F1.2, FB6.1
- new net: R64.2, R65.1, U14.6 (FB)
- new net: R66.2, R67.1, U15.6 (FB)
- new net: R60.2, R61.1, U12.6 (FB)
- new net: D10.2 (A), R71.2
- new net: D11.2 (A), R72.2
- new net: R68.2, U11.39 (PB3)
- new net: D9.2 (A), R70.2
- new net 12V0: C40.1, C41.1, C44.1, C47.1, C50.1, FB6.2, TP6.1 (In), U12.2 (VIN), U13.2 (VIN), U14.2 (VIN), U15.2 (VIN)
- new net 12V0_EN: J9.1 (12V0_OUT_EN), U11.32 (PA11)
- new net 1V0: C51.1, C52.1, R66.1, TP10.1 (In), U15.4 (VOUT), U15.5 (VOUT)
- new net 1V0_EN: U11.13 (PA3), U15.1 (EN)
- new net 1V0_PGOOD: U11.25 (PB12), U15.7 (PGOOD)
- new net 1V2: C48.1, C49.1, R64.1, TP9.1 (In), U14.4 (VOUT), U14.5 (VOUT)
- new net 1V2_EN: U11.33 (PA12), U14.1 (EN)
- new net 1V2_PGOOD: U11.26 (PB13), U14.7 (PGOOD)
- new net 1V8: C45.1, C46.1, R62.1, TP8.1 (In), U13.4 (VOUT), U13.5 (VOUT)
- new net 1V8_EN: U11.18 (PB0), U13.1 (EN)
- new net 1V8_PGOOD: U11.28 (PB15), U13.7 (PGOOD)
- new net 3V3: C42.1, C43.1, R60.1, TP5.1 (In), U12.4 (VOUT), U12.5 (VOUT)
- new net 3V3_EN: U11.29 (PA8), U12.1 (EN)
- new net 3V3_PGOOD: U11.27 (PB14), U12.7 (PGOOD)
- new net 3V3_SB: C34.1, C35.1, C37.1, C39.1, C53.1, C54.1, FB5.2, J8.2 (Vccaux), J9.5 (3V3_SB), R58.1, R69.1, TP7.1 (In), U11.1 (VBAT), U11.24 (VDD), U11.36 (VDD), U11.48 (VDD)
- new net A3V3_SUPER: C38.1, FB5.1, U11.9 (VDDA)
- new net FPGA_DONE: U11.45 (PB8)
- new net FPGA_INIT: U11.11 (PA1)
- new net FPGA_RST_N: U11.10 (PA0)
- new net GND: C34.2, C35.2, C36.2, C37.2, C38.2, C39.2, C40.2, C41.2, C42.2, C43.2, C44.2, C45.2, C46.2, C47.2, C48.2, C49.2, C50.2, C51.2, C52.2, C53.2, C54.2, D10.1 (K), D11.1 (K), D9.1 (K), J6.3 (P3), J7.5 (GND), J7.6 (GND_SENSE), J7.7 (GND), J7.8 (GND), J8.11 (Vss), J8.3 (Vss), J8.5 (Vss), J8.7 (Vss), J8.9 (Vss), J9.4 (GND), R59.2, R61.2, R63.2, R65.2, R67.2, TP10.2 (Ext), TP11.1 (P1), TP5.2 (Ext), TP6.2 (Ext), TP7.2 (Ext), TP8.2 (Ext), TP9.2 (Ext), U11.23 (GND), U11.35 (GND), U11.47 (GND), U11.8 (VSSA), U11.PAD (GND), U12.3 (GND), U12.PAD (GND), U13.3 (GND), U13.PAD (GND), U14.3 (GND), U14.PAD (GND), U15.3 (GND), U15.PAD (GND)
- new net MCU_RST_N: U11.12 (PA2)
- new net SUPER_BOOT0: R59.1, U11.44 (BOOT0)
- new net SUPER_FAULT_LED: R72.1, U11.41 (PB5)
- new net SUPER_I2C_SCL: J9.2 (I2C_SCL), TP11.3 (P3), U11.42 (PB6)
- new net SUPER_I2C_SDA: J9.3 (I2C_SDA), TP11.2 (P2), U11.43 (PB7)
- new net SUPER_JTAG_TCK: J8.6 (TCK), U11.37 (PA14)
- new net SUPER_JTAG_TDI: J8.10 (TDI_OUT), U11.38 (PA15)
- new net SUPER_JTAG_TDO: J8.8 (TDO_IN), R68.1
- new net SUPER_JTAG_TMS: J8.4 (TMS), U11.34 (PA13)
- new net SUPER_JTAG_TRST: R69.2, U11.40 (PB4)
- new net SUPER_PWRGOOD_LED: R70.1, U11.19 (PB1)
- new net SUPER_RST_N: C36.1, R58.2, U11.7 (NRST)
- new net SUPER_SPI_CS_N: U11.14 (PA4)
- new net SUPER_SPI_MISO: U11.16 (PA6)
- new net SUPER_SPI_MOSI: U11.17 (PA7)
- new net SUPER_SPI_SCK: U11.15 (PA5)
- new net SUPER_SYSOK_LED: R71.1, U11.20 (PB2)
- new net SUPER_UART_RX: J6.1 (P1), U11.31 (PA10)
- new net SUPER_UART_TX: J6.2 (P2), U11.30 (PA9)
- no-connect marks 0 -> 14
Other:
- note added: "Vout = 0.6 * 1+Rt/Rb 1.0 = 0.6*(1+Rt/Rb) 1.666 = 1+Rt/Rb 0.666 = Rt/Rb"
- note added: "Vout = 0.6 * 1+Rt/Rb 1.2 = 0.6*(1+Rt/Rb) 2 = 1+Rt/Rb 1 = Rt/Rb"
- note added: "Vout = 0.6 * 1+Rt/Rb 1.8 = 0.6*(1+Rt/Rb) 3 = 1+Rt/Rb 2 = Rt/Rb"
- note added: "Vout = 0.6 * 1+Rt/Rb 3.3 = 0.6*(1+Rt/Rb) 5.5 = 1+Rt/Rb 4.5 = Rt/Rb"

Commit message: Continued initial layout of fpga-stm32-ifaces
Parts:
- added R86, R87, R88, R89: 10K, azonenberg_pcb:EIA_0402_RES_NOSILK, symbol device:R
- C41, C42, C43, C44, C47, C50: footprint (none) -> azonenberg_pcb:EIA_1210_CAP_NOSILK
- C45, C46, C48, C49, C51, C52: footprint (none) -> azonenberg_pcb:EIA_0805_CAP_NOSILK
- D10, D11, D9: footprint (none) -> azonenberg_pcb:EIA_0603_LED
- J8: footprint (none) -> azonenberg_pcb:XILINX_JTAG_PTH_MOLEX_0878311420
- J9: footprint (none) -> azonenberg_pcb:CONN_MOLEX_PICOBLADE_5POS_0532610571
- R60, R61, R62, R63, R64, R65, R66, R67, R68, R70, R71, R72: footprint (none) -> azonenberg_pcb:EIA_0402_RES_NOSILK
- TP10, TP5, TP6, TP7, TP8, TP9: footprint (none) -> azonenberg_pcb:CONN_U.FL_TE_1909763-1
- TP11: footprint (none) -> azonenberg_pcb:CONN_HEADER_2.54MM_1x3
- U11: footprint (none) -> azonenberg_pcb:QFN_48_0.5MM_7x7MM
- U12, U13, U14, U15: footprint (none) -> azonenberg_pcb:MODULE_CYNTEC_MUN12AD03-SE
Connections:
- net 12V0_EN: now also U11.33 (PA12); no longer U11.32 (PA11)
- net 1V0_EN: now also R89.1
- net 1V2_EN: now also U11.32 (PA11), R88.1; no longer U11.33 (PA12)
- net 1V8_EN: now also R87.1
- net 3V3_EN: now also R86.1
- net FPGA_DONE: now also U11.20 (PB2); no longer U11.45 (PB8)
- net FPGA_RST_N: now also U11.19 (PB1); no longer U11.10 (PA0)
- net GND: now also R86.2, R87.2, R88.2, R89.2
- net SUPER_FAULT_LED: now also U11.5 (PH0); no longer U11.41 (PB5)
- net SUPER_PWRGOOD_LED: now also U11.10 (PA0); no longer U11.19 (PB1)
- net SUPER_SYSOK_LED: now also U11.6 (PH1); no longer U11.20 (PB2)
Other:
- company: (none) -> Antikernel Labs
- title: (none) -> FPGA - STM32 Interface Test
- moved on the sheet: U11C, U11E

Commit message: Initial routing of FPGA power
Connections:
- net 1V2_EN: now also U11.12 (PA2); no longer U11.32 (PA11)
- net 1V2_PGOOD: now also U11.11 (PA1); no longer U11.26 (PB13)
- net FPGA_INIT: now also U11.32 (PA11); no longer U11.11 (PA1)
- net MCU_RST_N: now also U11.26 (PB13); no longer U11.12 (PA2)
Changed lines of the file:
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@@
 	)
 	(label "1V2_EN"
-		(at 212.09 228.6 180)
+		(at 212.09 205.74 180)
 		(fields_autoplaced yes)
 		(effects
@@
 	)
 	(label "1V2_PGOOD"
-		(at 271.78 233.68 180)
+		(at 212.09 203.2 180)
 		(fields_autoplaced yes)
 		(effects
@@
 	(hierarchical_label "MCU_RST_N"
 		(shape output)
-		(at 212.09 205.74 180)
+		(at 271.78 233.68 180)
 		(fields_autoplaced yes)
 		(effects
@@
 	(hierarchical_label "FPGA_INIT"
 		(shape bidirectional)
-		(at 212.09 203.2 180)
-		(fields_autoplaced yes)
-		(effects
+		(at 212.09 228.6 180)
+		(fields_autoplaced yes)
+		(effects

Commit message: Continued layout, 283 now unrouted
Connections:
- net 1V0_EN: now also U11.26 (PB13); no longer U11.13 (PA3)
- net MCU_RST_N: now also U11.13 (PA3); no longer U11.26 (PB13)
Changed lines of the file:
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@@
 	(title_block
 		(title "FPGA - STM32 Interface Test")
-		(date "2024-06-12")
+		(date "2024-06-13")
 		(rev "0.1")
 		(company "Antikernel Labs")
@@
 	)
 	(label "1V0_EN"
-		(at 212.09 208.28 180)
+		(at 271.78 233.68 180)
 		(fields_autoplaced yes)
 		(effects
@@
 	(hierarchical_label "MCU_RST_N"
 		(shape output)
-		(at 271.78 233.68 180)
-		(fields_autoplaced yes)
-		(effects
+		(at 212.09 208.28 180)
+		(fields_autoplaced yes)
+		(effects

Commit message: Continued fpga-stm32-ifaces layout
Connections:
- net 1V0_EN: now also U11.28 (PB15); no longer U11.26 (PB13)
- net 1V0_PGOOD: now also U11.29 (PA8); no longer U11.25 (PB12)
- net 1V8_EN: now also U11.32 (PA11); no longer U11.18 (PB0)
- net 1V8_PGOOD: now also U11.27 (PB14); no longer U11.28 (PB15)
- net 3V3_EN: now also U11.25 (PB12); no longer U11.29 (PA8)
- net 3V3_PGOOD: now also U11.26 (PB13); no longer U11.27 (PB14)
- net FPGA_INIT: now also U11.19 (PB1); no longer U11.32 (PA11)
- net FPGA_RST_N: now also U11.18 (PB0); no longer U11.19 (PB1)
Changed lines of the file:
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@@
 	)
 	(label "3V3_PGOOD"
-		(at 271.78 236.22 180)
+		(at 271.78 233.68 180)
 		(fields_autoplaced yes)
 		(effects
@@
 	)
 	(label "1V0_EN"
-		(at 271.78 233.68 180)
+		(at 271.78 238.76 180)
 		(fields_autoplaced yes)
 		(effects
@@
 	)
 	(label "1V0_PGOOD"
-		(at 271.78 231.14 180)
+		(at 212.09 220.98 180)
 		(fields_autoplaced yes)
 		(effects
@@
 	)
 	(label "1V8_PGOOD"
-		(at 271.78 238.76 180)
+		(at 271.78 236.22 180)
 		(fields_autoplaced yes)
 		(effects
@@
 	)
 	(label "1V8_EN"
-		(at 271.78 200.66 180)
+		(at 212.09 228.6 180)
 		(fields_autoplaced yes)
 		(effects
@@
 	)
 	(label "3V3_EN"
-		(at 212.09 220.98 180)
+		(at 271.78 231.14 180)
 		(fields_autoplaced yes)
 		(effects
@@
 	(hierarchical_label "FPGA_RST_N"
 		(shape output)
-		(at 271.78 203.2 180)
+		(at 271.78 200.66 180)
 		(fields_autoplaced yes)
 		(effects
@@
 	(hierarchical_label "FPGA_INIT"
 		(shape bidirectional)
-		(at 212.09 228.6 180)
-		(fields_autoplaced yes)
-		(effects
+		(at 271.78 203.2 180)
+		(fields_autoplaced yes)
+		(effects
