File: fpga-stm32-ifaces/mcu.kicad_sch (KiCad schematic)
At the start: 58 parts, among them J10 CORTEX_DEBUG_ETM, J3 PMOD_HOST, J4 XILINX_JTAG, J5 CONN_01X03, U1 STM32H735-UFBGA176-25, U16 W25Q128JV, U2 XC7S25-1FTGB196, U8 AT24MAC402, U9 ECS-1612MV-250-CN

Commit message: Finished FPGA and MCU escape and interconnect routing
Connections:
- net FMC_NBL1: now also U2.A5 (IO_L4N_T0_34); no longer U2.B5 (IO_L4P_T0_34)
- net FPGA_QSPI_CS_N: now also U2.B3 (IO_L3P_T0_DQS_34); no longer U2.A3 (IO_L2N_T0_34)
- net FPGA_QSPI_DQ0: now also U2.C4 (IO_L6N_T0_VREF_34); no longer U2.B3 (IO_L3P_T0_DQS_34)
- net FPGA_QSPI_DQ1: now also U2.B5 (IO_L4P_T0_34); no longer U2.C4 (IO_L6N_T0_VREF_34)
- net FPGA_QSPI_DQ2: now also U2.B6 (IO_0_34); no longer U2.C5 (IO_L6P_T0_34)
- net FPGA_QSPI_DQ3: now also U2.C5 (IO_L6P_T0_34); no longer U2.B6 (IO_0_34)
- net FPGA_QSPI_DQ6: now also U2.A3 (IO_L2N_T0_34); no longer U2.A5 (IO_L4N_T0_34)
- net MCU_LED_0: now also U1.N15 (PH12); no longer U1.H1 (PF6)
- net MCU_LED_1: now also U1.P15 (PH6); no longer U1.J3 (PF7)
- net MCU_LED_2: now also U1.J4 (PF9); no longer U1.J2 (PF8)
- net MCU_LED_3: now also U1.M1 (PC2); no longer U1.J4 (PF9)
Changed lines of the file:
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@@
+	)
+	(no_connect
+		(at 91.44 107.95)
 	)
 	(no_connect
@@
 	)
 	(no_connect
+		(at 134.62 97.79)
+	)
+	(no_connect
+		(at 40.64 38.1)
+	)
+	(no_connect
+		(at 134.62 58.42)
+	)
+	(no_connect
+		(at 134.62 60.96)
+	)
+	(no_connect
+		(at 186.69 95.25)
+	)
+	(no_connect
+		(at 134.62 43.18)
+	)
+	(no_connect
+		(at 91.44 123.19)
+	)
+	(no_connect
+		(at 134.62 113.03)
+	)
+	(no_connect
+		(at 134.62 63.5)
+	)
+	(no_connect
+		(at 91.44 115.57)
+	)
+	(no_connect
+		(at 91.44 128.27)
+	)
+	(no_connect
+		(at 40.64 55.88)
+	)
+	(no_connect
+		(at 91.44 125.73)
+	)
+	(no_connect
+		(at 91.44 55.88)
+	)
+	(no_connect
+		(at 134.62 95.25)
+	)
+	(no_connect
 		(at 134.62 40.64)
 	)
 	(no_connect
-		(at 134.62 97.79)
-	)
-	(no_connect
-		(at 40.64 38.1)
-	)
-	(no_connect
-		(at 134.62 58.42)
-	)
-	(no_connect
-		(at 134.62 60.96)
-	)
-	(no_connect
-		(at 186.69 95.25)
-	)
-	(no_connect
-		(at 134.62 105.41)
-	)
-	(no_connect
-		(at 134.62 43.18)
-	)
-	(no_connect
-		(at 91.44 123.19)
-	)
-	(no_connect
-		(at 134.62 113.03)
-	)
-	(no_connect
-		(at 134.62 63.5)
-	)
-	(no_connect
-		(at 91.44 115.57)
-	)
-	(no_connect
-		(at 134.62 120.65)
-	)
-	(no_connect
-		(at 91.44 128.27)
-	)
-	(no_connect
-		(at 40.64 55.88)
-	)
-	(no_connect
-		(at 91.44 125.73)
-	)
-	(no_connect
-		(at 91.44 55.88)
-	)
-	(no_connect
-		(at 134.62 95.25)
-	)
-	(no_connect
 		(at 40.64 123.19)
 	)
@@
 	)
 	(no_connect
-		(at 134.62 35.56)
-	)
-	(no_connect
 		(at 134.62 115.57)
 	)
@@
 	)
 	(no_connect
+		(at 91.44 110.49)
+	)
+	(no_connect
 		(at 134.62 92.71)
 	)
@@
 	(no_connect
 		(at 91.44 58.42)
+	)
+	(no_connect
+		(at 91.44 105.41)
 	)
 	(no_connect
@@
 	)
 	(label "FMC_NBL1"
-		(at 339.09 54.61 180)
+		(at 339.09 57.15 180)
 		(fields_autoplaced yes)
 		(effects
@@
 	)
 	(label "MCU_LED_2"
-		(at 91.44 110.49 180)
+		(at 91.44 113.03 180)
 		(fields_autoplaced yes)
 		(effects
@@
 	)
 	(label "FPGA_QSPI_DQ0"
-		(at 339.09 49.53 180)
+		(at 339.09 67.31 180)
 		(fields_autoplaced yes)
 		(effects
@@
 	)
 	(label "MCU_LED_3"
-		(at 91.44 113.03 180)
+		(at 134.62 35.56 180)
 		(fields_autoplaced yes)
 		(effects
@@
 	)
 	(label "MCU_LED_0"
-		(at 91.44 105.41 180)
+		(at 134.62 120.65 180)
 		(fields_autoplaced yes)
 		(effects
@@
 	)
 	(label "FPGA_QSPI_CS_N"
-		(at 339.09 46.99 180)
+		(at 339.09 49.53 180)
 		(fields_autoplaced yes)
 		(effects
@@
 	)
 	(label "FPGA_QSPI_DQ1"
-		(at 339.09 67.31 180)
+		(at 339.09 54.61 180)
 		(fields_autoplaced yes)
 		(effects
@@
 	)
 	(label "FPGA_QSPI_DQ2"
-		(at 339.09 64.77 180)
+		(at 339.09 36.83 180)
 		(fields_autoplaced yes)
 		(effects
@@
 	)
 	(label "FPGA_QSPI_DQ3"
-		(at 339.09 36.83 180)
+		(at 339.09 64.77 180)
 		(fields_autoplaced yes)
 		(effects
@@
 	)
 	(label "FPGA_QSPI_DQ6"
-		(at 339.09 57.15 180)
+		(at 339.09 46.99 180)
 		(fields_autoplaced yes)
 		(effects
@@
 	)
 	(label "MCU_LED_1"
-		(at 91.44 107.95 180)
-		(fields_autoplaced yes)
-		(effects
+		(at 134.62 105.41 180)
+		(fields_autoplaced yes)
+		(effects
