File: lpr-rgmii-phy/lpr-rgmii-phy.kicad_sch (KiCad schematic)
At the start: 15 parts, among them U1 MUN12AD03-SE, U2 MUN12AD03-SE

Commit message: lpr-rgmii-phy: Finished initial layout, ready for review
Parts:
- added C10, C11, C12, C19, C20, C21, C22, C8, C9: 4.7 uF, azonenberg_pcb:EIA_0603_CAP_NOSILK, symbol device:C
- added C13, C14, C15, C16: 0.1 uF, azonenberg_pcb:EIA_0402_CAP_NOSILK, symbol device:C
- added C17, C18, C23, C24, C25, C26, C27, C28, C29, C30, C31, C32, C33, C34, C35, C7: 0.47 uF, azonenberg_pcb:EIA_0402_CAP_NOSILK, symbol device:C
- added FB1, FB2, FB3, FB4: MI0603J601R-10, azonenberg_pcb:EIA_0603_INDUCTOR_NOSILK, symbol passive-azonenberg:FERRITE_SMALL2
- added J2: 0826-1G1T-23-F, azonenberg_pcb:CONN_BELFUSE_0826_1G1T_23_F, symbol special-azonenberg:BEL_FUSE_0826-1G1T-23-F
- added M1: LOGO, azonenberg_pcb:LONGTHING-1200DPI, symbol special-azonenberg:MECHANICAL
- added M2: LOGO, w_logo:Logo_silk_OSHW_6x6mm, symbol special-azonenberg:MECHANICAL
- added M3: LOGO, w_logo:Logo_silk_ROHS_5x2.8mm, symbol special-azonenberg:MECHANICAL
- added M4: LOGO, w_logo:Logo_silk_WEEE_3.4x5mm, symbol special-azonenberg:MECHANICAL
- added R10, R11, R12, R13, R14, R7, R9: 33, azonenberg_pcb:EIA_0402_RES_NOSILK, symbol device:R
- added R15: 12.1K 1%, azonenberg_pcb:EIA_0402_RES_NOSILK, symbol device:R
- added R16, R24, R8: 1K, azonenberg_pcb:EIA_0402_RES_NOSILK, symbol device:R
- added R17, R18, R19, R20, R21, R22, R23, R25, R26: 10K, azonenberg_pcb:EIA_0402_RES_NOSILK, symbol device:R
- added R5, R6: 470, azonenberg_pcb:EIA_0402_RES_NOSILK, symbol device:R
- added TP3, TP4, TP5, TP6: U.FL, azonenberg_pcb:CONN_U.FL_TE_1909763-1, symbol conn:CONN_COAXIAL
- added TP7, TP9: TESTPOINT, azonenberg_pcb:TESTPOINT_SMT_0.5MM, symbol conn:CONN_01X01
- added TP8: TESTCLIP, azonenberg_pcb:TESTPOINT_SMT_KEYSTONE_5016, symbol conn:CONN_01X01
- added U3: ECS-1612MV-250-CN, azonenberg_pcb:OSCILLATOR_1.6x1.2, symbol osc-azonenberg:OSC
- added U4: KSZ9031RN, azonenberg_pcb:QFN_48_0.5MM_7x7MM, symbol special-azonenberg:KSZ9031RN
- added U5, U6: RCLAMP0514M, azonenberg_pcb:SOP_10_0.5MM_3MM, symbol special-azonenberg:RCLAMP0514M
- J1: value ~ -> LPR_HEADER; footprint (none) -> azonenberg_pcb:CONN_HEADER_2.0MM_2x20_SMT_MOLEX_0877594014
- R1, R3, R4: value FIXME -> 100K
- R2: value FIXME -> 22.1K
Connections:
- net 1V2: now also C11.1, C8.1, FB1.1, FB3.1, FB4.1
- net 3V3: now also C10.1, C17.1, C23.1, C28.1, C7.1, C9.1, FB2.1, R17.1, R18.1, R19.1, R20.1, R24.1, R5.1, R6.1, U3.1 (E/D#), U3.4 (Vdd), U4.16 (DVDDH), U4.34 (DVDDH), U4.40 (DVDDH)
- net 5V5: now also R25.1, R26.1
- net GND: now also U1.PAD (GND), U2.PAD (GND), C10.2, C11.2, C12.2, C13.1, C14.1, C15.1, C16.1, C17.2, C18.2, C19.2, C20.2, C21.2, C22.2, C23.2, C24.2, C25.2, C26.2, C27.2, C28.2, C29.2, C30.2, C31.2, C32.2, C33.2, C34.2, C35.2, C7.2, C8.2, C9.2, J2.17 (SHLD), R15.1, R16.1, R21.1, R22.1, R23.1, R8.1, TP3.2 (Ext), TP4.2 (Ext), TP5.2 (Ext), TP6.2 (Ext), TP8.1 (P1), U3.2 (Vss), U4.13 (NC/GND), U4.29 (VSS), U4.PAD, U5.8 (Gnd), U6.8 (Gnd)
- net ETH_RST_N: now reaches J1.19 (RFE_GPIO14)
- net ETH_RST_N: now also U4.42 (RESET_N)
- net ETH_MDIO: now reaches J1.23 (RFE_GPIO12)
- net ETH_MDIO: now also R24.2, U4.37 (MDIO)
- net ETH_MDC: now reaches J1.24 (RFE_GPIO3)
- net ETH_MDC: now also U4.36 (MDC)
- net RGMII_TX_CLK: now reaches J1.25 (RFE_GPIO11)
- net RGMII_TX_CLK: now also U4.24 (GTX_CLK)
- net RGMII_TX_EN: now reaches J1.26 (RFE_GPIO2)
- net RGMII_TX_EN: now also U4.25 (TX_EN)
- net RGMII_TXD2: now reaches J1.27 (RFE_GPIO10)
- net RGMII_TXD2: now also U4.21 (TXD2)
- net RGMII_TXD3: now reaches J1.28 (RFE_GPIO1)
- net RGMII_TXD3: now also U4.22 (TXD3)
- net ETH_RX_DV: now reaches J1.3 (RFE_GPIO17)
- net ETH_RX_DV: now also R13.1, R22.2
- net RGMII_TXD0: now reaches J1.31 (RFE_GPIO9)
- net RGMII_TXD0: now also U4.19 (TXD0)
- net RGMII_TXD1: now reaches J1.32 (RFE_GPIO0)
- net RGMII_TXD1: now also U4.20 (TXD1)
- net ETH_RX_CLK: now reaches J1.4 (RFE_GPIO8_CC)
- net ETH_RX_CLK: now also R14.1, R23.2
- net ETH_RXD1: now reaches J1.5 (RFE_GPIO16)
- net ETH_RXD1: now also R11.1, R20.2
- net ETH_RXD0: now reaches J1.6 (RFE_GPIO7)
- net ETH_RXD0: now also R12.1, R21.2
- net ETH_RXD3: now reaches J1.7 (RFE_GPIO15)
- net ETH_RXD3: now also R18.2, R9.1
- net ETH_RXD2: now reaches J1.8 (RFE_GPIO6)
- net ETH_RXD2: now also R10.1, R19.2
- net 1V2_PGOOD: now reaches U2.7 (PGOOD)
- net 1V2_PGOOD: now also R26.2, TP7.1 (P1)
- net 3V3_PGOOD: now reaches U1.7 (PGOOD)
- net 3V3_PGOOD: now also R25.2, TP9.1 (P1)
- new net: R12.2, U4.32 (RXD0/MODE0)
- new net: J2.16 (LED2_P), R6.2
- new net: C16.2, J2.7 (CH4_TAP)
- new net: C15.2, J2.1 (CH3_TAP)
- new net: C13.2, J2.12 (CH1_TAP)
- new net: J2.14 (LED1_P), R5.2
- new net: C14.2, J2.6 (CH2_TAP)
- new net: R17.2, U4.41 (CLK125_NDO/LED_MODE)
- new net: R9.2, U4.27 (RXD3/MODE3)
- new net: R10.2, U4.28 (RXD2/MODE2)
- new net: R11.2, U4.31 (RXD1/MODE1)
- new net: R13.2, U4.33 (RX_DV/CLK125_EN)
- new net: R14.2, U4.35 (RX_CLK/PHYAD2)
- new net: R15.2, U4.48 (ISET)
- new net: R7.2, U3.3 (CLK)
- new net A1V2: C21.1, C25.1, C31.1, FB3.2, TP5.1 (In), U4.4 (AVDDL), U4.9 (AVDDL)
- new net A1V2_PLL: C22.1, C26.1, FB4.2, TP4.1 (In), U4.44 (AVDDL_PLL)
- new net A3V3: C20.1, C27.1, C30.1, C33.1, FB2.2, TP6.1 (In), U4.1 (AVDDH), U4.12 (AVDDH), U4.47 (NC/AVDDH), U5.3 (Vcc), U6.3 (Vcc)
- new net D1V2: C12.1, C18.1, C19.1, C24.1, C29.1, C32.1, C34.1, C35.1, FB1.2, TP3.1 (In), U4.14 (DVDDL), U4.18 (DVDDL), U4.23 (DVDDL), U4.26 (DVDDL), U4.30 (DVDDL), U4.39 (DVDDL)
- new net ETH_A_N: J2.10 (CH1_N), U4.3 (TXRXM_A), U5.4 (LINE_3), U5.7 (NC_3)
- new net ETH_A_P: J2.11 (CH1_P), U4.2 (TXRXP_A), U5.5 (NC_4), U5.6 (LINE_4)
- new net ETH_B_N: J2.4 (CH2_P), U4.6 (TXRXM_B), U5.1 (LINE_1), U5.10 (NC_1)
- new net ETH_B_P: J2.5 (CH2_N), U4.5 (TXRXP_B), U5.2 (NC_2), U5.9 (LINE_2)
- new net ETH_CLK_25MHZ: R7.1, U4.46 (XI)
- new net ETH_C_N: J2.2 (CH3_N), U4.8 (TXRXM_C), U6.4 (LINE_3), U6.7 (NC_3)
- new net ETH_C_P: J2.3 (CH3_P), U4.7 (TXRXP_C), U6.5 (NC_4), U6.6 (LINE_4)
- new net ETH_D_N: J2.8 (CH4_P), U4.11 (TXRXM_D), U6.1 (LINE_1), U6.10 (NC_1)
- new net ETH_D_P: J2.9 (CH4_N), U4.10 (TXRXP_D), U6.2 (NC_2), U6.9 (LINE_2)
- new net ETH_LED1_N: J2.13 (LED1_N), R16.2, U4.17 (LED1/PHYAD0)
- new net ETH_LED2_N: J2.15 (LED2_N), R8.2, U4.15 (LED2/PHYAD1)
- no-connect marks 10 -> 12
Other:
- note added: "Polarity swap KSZ9031 auto corrects"
- note added: "Strap: Disable CLK125_NDO we don't use"
- note added: "Strap: PHYADDR[2] = 0"
- note added: "Strap: PHYADR[1:0] = 2'b00"
- note added: "Strap: advertise everything but gig/half"
- note added: "Strap: dual LEDs"
- note added: "Vout = 0.6 * (1 + RfbT / RfbB) 1.2 = 0.6 * (1 + Rtop / Rbot) Rtop/Rbot = 1 Datasheet suggests 124K / 124K We can do 100k / 100k with what we have in stock"
- note added: "Vout = 0.6 * (1 + RfbT / RfbB) 3.3 = 0.6 * (1 + Rtop / Rbot) Rtop/Rbot = 4.5 Datasheet suggests 124K / 27.4K We can do 100k / 22.1k with what we have in stock"
- note removed: "Vout = 0.6 * (1 + RfbT / RfbB) 5 = 0.6 * (1 + Rtop / Rbot) Rtop/Rbot = 7.333 Datasheet suggests 124 / 16.9K We can do 174k / 27.4k with what we have in stock"
- moved on the sheet: C1, C2, C3, C4, C5, C6, J1A, J1B, J1C, R1, R2, R3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
