File: paste-test/paste-test.kicad_pcb (KiCad board)
At the start: 2 copper layers, 67 x 40 mm, 17 parts, among them M1 MECHANICAL, M10 MECHANICAL, M11 MECHANICAL, M12 MECHANICAL, M13 MECHANICAL, M14 MECHANICAL, M15 MECHANICAL, M16 MECHANICAL, M17 MECHANICAL, M2 MECHANICAL, M3 MECHANICAL, M4 MECHANICAL, M5 MECHANICAL, M6 MECHANICAL, M7 MECHANICAL, M8 MECHANICAL, M9 MECHANICAL

Commit message: Initial test version of paste-test board ready for fab
Changed lines of the file:
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@@
 			(outputformat 1)
 			(mirror no)
-			(drillshape 1)
+			(drillshape 0)
 			(scaleselection 1)
-			(outputdirectory "")
+			(outputdirectory "output/")
 		)
 	)
@@
 			)
 		)
+	)
+	(zone
+		(net 0)
+		(net_name "")
+		(layer "F.SilkS")
+		(hatch edge 0.5)
+		(connect_pads
+			(clearance 0.5)
+		)
+		(min_thickness 0.25)
+		(filled_areas_thickness no)
+		(fill yes
+			(thermal_gap 0.5)
+			(thermal_bridge_width 0.5)
+			(island_removal_mode 1)
+			(island_area_min 10)
+		)
+		(polygon
+			(pts
+				(xy 85.75 66.25) (xy 85.75 78.5) (xy 88.75 78.5) (xy 88.75 66.25)
+			)
+		)
