File: christmas-tree/christmas-tree.kicad_sch (KiCad schematic)
At the start: 62 parts, among them J1 USB_C_Receptacle_USB2.0, J2 CORTEX_DEBUG_ETM, J3 CONN_01X03, M1 MECHANICAL, U1 NCP45525IMNTWG-H, U10 19-C47/RSGHBHC-5V01/2T, U11 19-C47/RSGHBHC-5V01/2T, U12 ZLDO1117-33, U2 74LVC1T45, U3 19-C47/RSGHBHC-5V01/2T, U4 19-C47/RSGHBHC-5V01/2T, U5 19-C47/RSGHBHC-5V01/2T, U6 19-C47/RSGHBHC-5V01/2T, U7 19-C47/RSGHBHC-5V01/2T, U8 19-C47/RSGHBHC-5V01/2T, U9 STM32L031-QFN32

Commit message: Removed stale todo comment from schematic
Other:
- note removed: "TODO: 3V3 regulator"
Changed lines of the file:
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@@
-		)
-	)
-	(text "TODO: 3V3 regulator"
-		(exclude_from_sim no)
-		(at 172.212 195.326 0)
-		(effects
-			(font
-				(size 1.27 1.27)
-			)
 		)
 	)
