File: fpga-test-kintex676-artix484/fpga-test-kintex676-artix484.kicad_pcb (KiCad board)
At the start: 4 copper layers, 73 x 88 mm, 161 parts, among them J1 SMPM, J10 SMPM, J11 BARREL_JACK, J2 SMPM, J3 SMPM, J4 SMPM, J5 XILINX_JTAG, J6 XILINX_JTAG, J7 SMPM, J8 SMPM, J9 SMPM, M1 SCREWHOLE, M2 SCREWHOLE, M3 SCREWHOLE, M4 SCREWHOLE, M5 MECHANICAL, M6 MECHANICAL, M7 MECHANICAL, M8 MECHANICAL, M9 MECHANICAL, U1 XC7A35T-2FBG484C, U10 MUN12AD03-SE, U11 SIT9121AI-2BF-XXS156.250000G, U2 SIT9121AI-2BF-XXS156.250000G, U3 ECS-1612MV-250-CN, U4 XC7K160T-2FFG676, U5 ECS-1612MV-250-CN, U6 ZLDO1117-33, U7 MUN12AD03-SE, U8 SIT9121AI-2BF-XXS156.250000G, U9 MUN12AD03-SE

Commit message: Finished fpga test
Parts:
- moved M6 82.2 mm to (70.0, 93.0)
- moved M7 82.1 mm to (78.0, 92.0)
- moved M9 73.0 mm to (85.0, 93.0)
- moved M8 71.9 mm to (91.0, 93.0)
- moved C55 70.0 mm to (109.2, 122.8), turned to 90 degrees
- moved C54 67.2 mm to (106.0, 122.8), turned to 90 degrees
- moved R22 61.5 mm to (105.2, 127.2), turned to 180 degrees
- moved R23 59.5 mm to (105.6, 126.0), turned to -90 degrees
- moved R24 59.5 mm to (104.7, 126.0), turned to 90 degrees
- moved C51 55.2 mm to (128.4, 116.6), turned to 180 degrees
- moved U10 55.0 mm to (107.8, 126.7), turned to 180 degrees
- moved C52 52.9 mm to (128.4, 120.0), turned to 180 degrees
- moved C53 49.9 mm to (111.2, 129.6), turned to -90 degrees
- moved R21 48.1 mm to (132.4, 121.0), turned to -90 degrees
- moved C48 47.1 mm to (125.0, 82.0)
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Connections:
- C60 pad 1: /Kintex FFG676/1V8 -> /Kintex FFG676/Kintex Power/1V8
- C61 pad 1: /Kintex FFG676/1V8 -> /Kintex FFG676/Kintex Power/1V8
- C62 pad 1: /Kintex FFG676/1V8 -> /Kintex FFG676/Kintex Power/1V8
- C65 pad 1: /Kintex FFG676/Kintex Power/1V2 -> /Kintex FFG676/1V2
- C66 pad 1: /Kintex FFG676/1V8 -> /Kintex FFG676/Kintex Power/1V8
- J6 pad 2: /Kintex FFG676/1V8 -> /Kintex FFG676/3V3
- R13 pad 1: /Kintex FFG676/1V8 -> /Kintex FFG676/Kintex Power/1V8
- R14 pad 1: /Kintex FFG676/Kintex Power/1V2 -> /Kintex FFG676/1V2
- R35 pad 2: /Kintex FFG676/Kintex Transceivers/1V2 -> /Kintex FFG676/1V2
- U4 pad A11: /Kintex FFG676/1V8 -> /Kintex FFG676/Kintex Power/1V8
- U4 pad AA1: /Kintex FFG676/1V8 -> /Kintex FFG676/Kintex Power/1V8
- U4 pad AA11: /Kintex FFG676/1V8 -> /Kintex FFG676/Kintex Power/1V8
- U4 pad AA21: /Kintex FFG676/1V8 -> /Kintex FFG676/Kintex Power/1V8
- U4 pad AB18: /Kintex FFG676/1V8 -> /Kintex FFG676/Kintex Power/1V8
- U4 pad AB8: /Kintex FFG676/1V8 -> /Kintex FFG676/Kintex Power/1V8
- U4 pad AC15: /Kintex FFG676/1V8 -> /Kintex FFG676/Kintex Power/1V8
- U4 pad AC25: /Kintex FFG676/1V8 -> /Kintex FFG676/Kintex Power/1V8
- U4 pad AC5: /Kintex FFG676/1V8 -> /Kintex FFG676/Kintex Power/1V8
- U4 pad AD12: /Kintex FFG676/1V8 -> /Kintex FFG676/Kintex Power/1V8
- U4 pad AD2: /Kintex FFG676/1V8 -> /Kintex FFG676/Kintex Power/1V8
- U4 pad AD22: /Kintex FFG676/1V8 -> /Kintex FFG676/Kintex Power/1V8
- U4 pad AE19: /Kintex FFG676/1V8 -> /Kintex FFG676/Kintex Power/1V8
- U4 pad AE9: /Kintex FFG676/1V8 -> /Kintex FFG676/Kintex Power/1V8
- U4 pad AF16: /Kintex FFG676/1V8 -> /Kintex FFG676/Kintex Power/1V8
- U4 pad AF26: /Kintex FFG676/1V8 -> /Kintex FFG676/Kintex Power/1V8
- U4 pad AF6: /Kintex FFG676/1V8 -> /Kintex FFG676/Kintex Power/1V8
- U4 pad B18: /Kintex FFG676/1V8 -> /Kintex FFG676/Kintex Power/1V8
- U4 pad B3: /Kintex FFG676/Kintex Power/1V2 -> /Kintex FFG676/1V2
- U4 pad B8: /Kintex FFG676/1V8 -> /Kintex FFG676/Kintex Power/1V8
- U4 pad C15: /Kintex FFG676/1V8 -> /Kintex FFG676/Kintex Power/1V8
- U4 pad C2: /Kintex FFG676/Kintex Power/1V2 -> /Kintex FFG676/1V2
- U4 pad D12: /Kintex FFG676/1V8 -> /Kintex FFG676/Kintex Power/1V8
- U4 pad D3: /Kintex FFG676/Kintex Power/1V2 -> /Kintex FFG676/1V2
- U4 pad E19: /Kintex FFG676/1V8 -> /Kintex FFG676/Kintex Power/1V8
- U4 pad E8: /Kintex FFG676/1V8 -> /Kintex FFG676/Kintex Power/1V8
- U4 pad E9: /Kintex FFG676/1V8 -> /Kintex FFG676/Kintex Power/1V8
- U4 pad F16: /Kintex FFG676/1V8 -> /Kintex FFG676/Kintex Power/1V8
- U4 pad G13: /Kintex FFG676/1V8 -> /Kintex FFG676/Kintex Power/1V8
- U4 pad G2: /Kintex FFG676/Kintex Power/1V2 -> /Kintex FFG676/1V2
- U4 pad H10: /Kintex FFG676/1V8 -> /Kintex FFG676/Kintex Power/1V8
- U4 pad H20: /Kintex FFG676/1V8 -> /Kintex FFG676/Kintex Power/1V8
- U4 pad H3: /Kintex FFG676/Kintex Power/1V2 -> /Kintex FFG676/1V2
- U4 pad J17: /Kintex FFG676/1V8 -> /Kintex FFG676/Kintex Power/1V8
- U4 pad K24: /Kintex FFG676/1V8 -> /Kintex FFG676/Kintex Power/1V8
- U4 pad L11: /Kintex FFG676/1V8 -> /Kintex FFG676/Kintex Power/1V8
- U4 pad L2: /Kintex FFG676/Kintex Power/1V2 -> /Kintex FFG676/1V2
- U4 pad M10: /Kintex FFG676/1V8 -> /Kintex FFG676/Kintex Power/1V8
- U4 pad M12: /Kintex FFG676/1V8 -> /Kintex FFG676/Kintex Power/1V8
- U4 pad M18: /Kintex FFG676/1V8 -> /Kintex FFG676/Kintex Power/1V8
- U4 pad M3: /Kintex FFG676/Kintex Power/1V2 -> /Kintex FFG676/1V2
- U4 pad M5: /Kintex FFG676/Kintex Transceivers/1V2 -> /Kintex FFG676/1V2
- U4 pad N25: /Kintex FFG676/1V8 -> /Kintex FFG676/Kintex Power/1V8
- U4 pad N6: /Kintex FFG676/1V8 -> /Kintex FFG676/Kintex Power/1V8
- U4 pad P10: /Kintex FFG676/1V8 -> /Kintex FFG676/Kintex Power/1V8
- U4 pad P22: /Kintex FFG676/1V8 -> /Kintex FFG676/Kintex Power/1V8
- U4 pad P8: /Kintex FFG676/1V8 -> /Kintex FFG676/Kintex Power/1V8
- U4 pad R19: /Kintex FFG676/1V8 -> /Kintex FFG676/Kintex Power/1V8
- U4 pad R9: /Kintex FFG676/1V8 -> /Kintex FFG676/Kintex Power/1V8
- U4 pad T10: /Kintex FFG676/1V8 -> /Kintex FFG676/Kintex Power/1V8
- U4 pad T16: /Kintex FFG676/1V8 -> /Kintex FFG676/Kintex Power/1V8
- U4 pad T26: /Kintex FFG676/1V8 -> /Kintex FFG676/Kintex Power/1V8
- U4 pad T8: /Kintex FFG676/1V8 -> /Kintex FFG676/Kintex Power/1V8
- U4 pad U11: /Kintex FFG676/1V8 -> /Kintex FFG676/Kintex Power/1V8
- U4 pad U23: /Kintex FFG676/1V8 -> /Kintex FFG676/Kintex Power/1V8
- U4 pad U3: /Kintex FFG676/1V8 -> /Kintex FFG676/Kintex Power/1V8
- U4 pad V10: /Kintex FFG676/1V8 -> /Kintex FFG676/Kintex Power/1V8
- U4 pad V20: /Kintex FFG676/1V8 -> /Kintex FFG676/Kintex Power/1V8
- U4 pad W17: /Kintex FFG676/1V8 -> /Kintex FFG676/Kintex Power/1V8
- U4 pad W7: /Kintex FFG676/1V8 -> /Kintex FFG676/Kintex Power/1V8
- U4 pad Y14: /Kintex FFG676/1V8 -> /Kintex FFG676/Kintex Power/1V8
- U4 pad Y24: /Kintex FFG676/1V8 -> /Kintex FFG676/Kintex Power/1V8
- U4 pad Y4: /Kintex FFG676/1V8 -> /Kintex FFG676/Kintex Power/1V8
Routing:
- net /Kintex FFG676/1V8: track 273.4 -> 0.00 mm, vias 72 -> 0
- net /Kintex FFG676/Kintex Power/1V8: track 0.00 -> 246.2 mm, vias 0 -> 69
- net /GND: track 1227.1 -> 1384.5 mm, vias 449 -> 641
- net /Power Supply/12V0: track 2.52 -> 112.1 mm
- net /Kintex FFG676/1V2: track 0.00 -> 70.0 mm, vias 0 -> 14
- net /Kintex FFG676/Kintex Power/1V2: track 63.9 -> 0.00 mm, vias 13 -> 0
- net /3V3: track 58.2 -> 116.2 mm, vias 8 -> 13
- net /1V2: track 145.2 -> 173.0 mm, vias 8 -> 18
- net /1V8: track 51.7 -> 74.7 mm, vias 8 -> 14
- net /1V0: track 117.7 -> 138.5 mm, vias 8 -> 14
- net /Kintex FFG676/3V3: track 168.2 -> 179.3 mm
- net /Artix FGG484/3V3: track 119.7 -> 124.0 mm
- net /Power Supply/1V8_FB: track 0.00 -> 2.55 mm
- net /Kintex FFG676/KINTEX_TCK: track 29.4 -> 26.9 mm, vias 3 -> 2
- net /Power Supply/1V2_FB: track 0.00 -> 1.98 mm
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- added copper zone on F.Cu, net /1V0
- added copper zone on In2.Cu, net /1V0
- added copper zone on F.Cu, net /1V2
- added copper zone on In2.Cu, net /1V2
- added copper zone on F.Cu, net /1V8
- added copper zone on In2.Cu, net /1V8
- added copper zone on F.Cu, net /3V3
- added copper zone on In2.Cu, net /3V3
- added copper zone on B.Cu, net /Artix FGG484/1V2
- added copper zone on B.Cu, net /Artix FGG484/3V3
- added copper zone on F.Cu, net /Artix FGG484/3V3
- added copper zone on In2.Cu, net /Artix FGG484/3V3
- added copper zone on In2.Cu, net /Artix FGG484/Artix Power/1V0
- added copper zone on B.Cu, net /Artix FGG484/Artix Power/1V8
- added copper zone on In2.Cu, net /Artix FGG484/Artix Power/1V8
- added copper zone on In1.Cu, net /GND
- added copper zone on In2.Cu, net /GND
- added copper zone on B.Cu, net /Kintex FFG676/1V2
- added copper zone on In2.Cu, net /Kintex FFG676/1V2
- added copper zone on In2.Cu, net /Kintex FFG676/3V3
- added copper zone on F.Cu, net /Kintex FFG676/Kintex Power/1V0
- added copper zone on In2.Cu, net /Kintex FFG676/Kintex Power/1V0
- added copper zone on In2.Cu, net /Kintex FFG676/Kintex Power/1V8
- added copper zone on F.Cu, net /Power Supply/12V0
Other:
- board text added: "+12VDC"
- board text added: "Artix-7 FGG484 + Kintex-7 FFG676 Minimal Testbed A. Zonenberg v0.1 / 2024-11-17"
- board text added: "RX_N"
- board text added: "RX_P"
- board text added: "TX_N"
- board text added: "TX_P"
