File: fpga-test-kintex676-artix484/kintex-transceivers.kicad_sch (KiCad schematic)
At the start: 28 parts, among them J10 SMPM, J7 SMPM, J8 SMPM, J9 SMPM, U11 SIT9121AI-2BF-XXS156.250000G, U4 XC7K160T-2FFG676, U8 SIT9121AI-2BF-XXS156.250000G

Commit message: Finished fpga test
Changed lines of the file:
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@@
+	)
+	(junction
+		(at 199.39 21.59)
+		(diameter 0)
+		(color 0 0 0 0)
 	)
 	(junction
@@
 	(wire
 		(pts
+			(xy 199.39 24.13) (xy 199.39 21.59)
+		)
+		(stroke
+			(width 0)
+			(type default)
+		)
+	)
+	(wire
+		(pts
 			(xy 43.18 142.24) (xy 43.18 144.78)
 		)
@@
 		(pts
 			(xy 73.66 160.02) (xy 73.66 163.83)
+		)
+		(stroke
+			(width 0)
+			(type default)
+		)
+	)
+	(wire
+		(pts
+			(xy 180.34 24.13) (xy 199.39 24.13)
 		)
 		(stroke
@@
 		)
 	)
-	(label "1V2"
-		(at 194.31 21.59 0)
-		(fields_autoplaced yes)
-		(effects
-			(font
-				(size 1.27 1.27)
-			)
-			(justify left bottom)
-		)
-	)
 	(label "GTX7_TX_AC_N"
 		(at 95.25 90.17 180)
@@
 		(fields_autoplaced yes)
 		(effects
+			(font
+				(size 1.27 1.27)
+			)
+			(justify right)
+		)
+	)
+	(hierarchical_label "1V2"
+		(shape input)
+		(at 180.34 24.13 180)
+		(fields_autoplaced yes)
+		(effects
