File: fpga-test-kintex676-artix484/kintex.kicad_sch (KiCad schematic)
At the start: 23 parts, among them J6 XILINX_JTAG, M1 SCREWHOLE, M2 SCREWHOLE, M3 SCREWHOLE, M4 SCREWHOLE, U4 XC7K160T-2FFG676, U5 ECS-1612MV-250-CN

Commit message: Finished fpga test
Connections:
- net 1V8: no longer J6.2 (Vccaux)
- net 3V3: now also J6.2 (Vccaux)
Other:
- sheet Kintex Transceivers ports: added 1V2; removed none
Changed lines of the file:
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@@
 	)
 	(label "GND"
-		(at 22.86 39.37 180)
+		(at 22.86 41.91 180)
 		(fields_autoplaced yes)
 		(effects
@@
 		)
 	)
+	(label "1V2"
+		(at 22.86 39.37 180)
+		(fields_autoplaced yes)
+		(effects
+			(font
+				(size 1.27 1.27)
+			)
+			(justify right bottom)
+		)
+	)
 	(label "3V3"
 		(at 45.72 157.48 180)
@@
 		)
 	)
-	(label "1V8"
+	(label "3V3"
 		(at 43.18 179.07 180)
 		(fields_autoplaced yes)
@@
 		)
 		(pin "GND" input
+			(at 22.86 41.91 180)
+			(effects
+				(font
+					(size 1.27 1.27)
+				)
+				(justify left)
+			)
+		)
+		(pin "1V2" input
 			(at 22.86 39.37 180)
 			(effects
