File: quad-relay-mux/quad-relay-mux.kicad_pcb (KiCad board)
At the start: 4 copper layers, 42 x 157.5 mm, 102 parts, among them J1 CONN_01X03, J10 SMA, J11 SMA, J12 SMA, J13 SMA, J14 USB_C_Receptacle_USB2.0, J15 SMA, J16 SMA, J17 SMA, J2 CORTEX_DEBUG_ETM, J3 CONN_01X03, J4 CONN_01X03, J5 SMA, J6 SMA, J7 SMA, J8 SMA, J9 SMA, K1 RELAY_TE_HF3_96, K2 RELAY_TE_HF3_96, K3 RELAY_TE_HF3_96, K4 RELAY_TE_HF3_96, M1 SCREWHOLE, M10 LOGO, M2 SCREWHOLE, M3 SCREWHOLE, M4 SCREWHOLE, M5 SCREWHOLE, M6 SCREWHOLE, M7 LOGO, M8 LOGO, M9 LOGO, U1 STM32L431-QFN32, U2 FT234XD, U3 TCA6424A, U39 NCP45525IMNTWG-H, U55 BD63573NUV, U56 BD63573NUV, U57 BD63573NUV, U58 BD63573NUV

Commit message: Updated relay mux board config for fab
Other:
- rule pad_to_mask_clearance: 0 -> 0.05
Changed lines of the file:
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@@
 			(dielectric_constraints no)
 		)
-		(pad_to_mask_clearance 0)
+		(pad_to_mask_clearance 0.05)
 		(allow_soldermask_bridges_in_footprints no)
 		(tenting front back)
@@
 			(usegerberattributes yes)
 			(usegerberadvancedattributes yes)
-			(creategerberjobfile yes)
+			(creategerberjobfile no)
 			(dashed_line_dash_ratio 12.000000)
 			(dashed_line_gap_ratio 3.000000)
@@
 			(outputformat 1)
 			(mirror no)
-			(drillshape 1)
+			(drillshape 0)
 			(scaleselection 1)
-			(outputdirectory "")
+			(outputdirectory "output/")
 		)
 	)
