File: t20-l431-som/fpga-config.kicad_sch (KiCad schematic)
At the start: 3 parts, among them U2 T20W80, U3 MX25U3232F

Commit message: Continued initial layout
Parts:
- added R1: 10K, azonenberg_pcb:EIA_0201_RES_NOSILK, symbol device:R
- added U4: MODULE_INTERNAL_T20_L431_HOST, azonenberg_pcb:MODULE_INTERNAL_T20_L431_HOST, symbol special-azonenberg:MODULE_INTERNAL_T20_L431_HOST
Connections:
- net 1V8: now also R1.2
- net FPGA_FLASH_CS_N: now also R1.1
- net FPGA_JTAG_TCK: now also U4.C8 (FPGA_JTAG_TCK)
- net FPGA_JTAG_TDI: now also U4.B8 (FPGA_JTAG_TDI)
- net FPGA_JTAG_TDO: now also U4.B7 (FPGA_JTAG_TDO)
- net FPGA_JTAG_TMS: now also U4.D7 (FPGA_JTAG_TMS)
Other:
- note removed: "TODO: JTAG pins to host board"
Changed lines of the file:
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@@
-		)
-	)
-	(text "TODO: JTAG pins to host board"
-		(exclude_from_sim no)
-		(at 113.03 24.13 0)
-		(effects
-			(font
-				(size 1.27 1.27)
-			)
-			(justify left)
 		)
 	)
@@
 		)
 	)
+	(label "FPGA_JTAG_TCK"
+		(at 45.72 110.49 180)
+		(effects
+			(font
+				(size 1.27 1.27)
+			)
+			(justify right bottom)
+		)
+	)
+	(label "FPGA_JTAG_TDI"
+		(at 45.72 115.57 180)
+		(effects
+			(font
+				(size 1.27 1.27)
+			)
+			(justify right bottom)
+		)
+	)
 	(label "FPGA_FLASH_CS_N"
 		(at 45.72 74.93 180)
@@
 		)
 	)
+	(label "FPGA_JTAG_TDO"
+		(at 45.72 118.11 180)
+		(effects
+			(font
+				(size 1.27 1.27)
+			)
+			(justify right bottom)
+		)
+	)
 	(label "FPGA_FLASH_SCK"
 		(at 45.72 77.47 180)
@@
 		)
 	)
+	(label "FPGA_FLASH_CS_N"
+		(at 118.11 67.31 180)
+		(effects
+			(font
+				(size 1.27 1.27)
+			)
+			(justify right bottom)
+		)
+	)
 	(label "FPGA_FLASH_DQ0"
 		(at 45.72 80.01 180)
@@
 		)
 	)
+	(label "FPGA_JTAG_TMS"
+		(at 45.72 113.03 180)
+		(effects
+			(font
+				(size 1.27 1.27)
+			)
+			(justify right bottom)
+		)
+	)
 	(label "FPGA_JTAG_TCK"
 		(at 45.72 41.91 180)
@@
 			)
 			(justify right bottom)
+		)
+	)
+	(label "1V8"
+		(at 125.73 67.31 0)
+		(effects
+			(font
+				(size 1.27 1.27)
+			)
+			(justify left bottom)
 		)
 	)
@@
 				)
 			)
+		)
+	)
+	(symbol
+		(lib_id "device:R")
+		(at 121.92 67.31 90)
+		(unit 1)
+		(exclude_from_sim no)
+		(in_bom yes)
+		(on_board yes)
+		(dnp no)
+		(property "Reference" "R1"
+			(at 121.92 64.77 90)
+			(effects
+				(font
+					(size 1.27 1.27)
+				)
+			)
+		)
+		(property "Value" "10K"
+			(at 121.92 67.31 90)
+			(effects
+				(font
+					(size 1.27 1.27)
+				)
+			)
+		)
+		(property "Footprint" "azonenberg_pcb:EIA_0201_RES_NOSILK"
+			(at 121.92 69.088 90)
+			(effects
+				(font
+					(size 1.27 1.27)
+				)
+				(hide yes)
+			)
+		)
+		(property "Datasheet" ""
+			(at 121.92 67.31 0)
+			(effects
+				(font
+					(size 1.27 1.27)
+				)
+				(hide yes)
+			)
+		)
+		(property "Description" "Resistor"
+			(at 121.92 67.31 0)
+			(effects
+				(font
+					(size 1.27 1.27)
+				)
+				(hide yes)
+			)
+		)
+		(pin "1"
+		)
+		(pin "2"
+		)
+		(instances
+			(project "t20-l431-som"
+				(path "/c9028163-a5a7-4e78-bba9-fb79df7846cd/bd86606c-2acb-477c-972b-5bc80fa54b47"
+					(reference "R1")
+					(unit 1)
+				)
+			)
+		)
+	)
+	(symbol
+		(lib_id "special-azonenberg:MODULE_INTERNAL_T20_L431_HOST")
+		(at 49.53 157.48 0)
+		(unit 2)
+		(exclude_from_sim no)
+		(in_bom yes)
+		(on_board yes)
+		(dnp no)
+		(property "Reference" "U4"
+			(at 49.53 158.8657 0)
+			(effects
+				(font
+					(size 1.27 1.27)
+				)
+				(justify left)
+			)
+		)
+		(property "Value" "MODULE_INTERNAL_T20_L431_HOST"
+			(at 49.53 161.29 0)
+			(effects
+				(font
+					(size 1.27 1.27)
+				)
+				(justify left)
+			)
+		)
+		(property "Footprint" "azonenberg_pcb:MODULE_INTERNAL_T20_L431_HOST"
+			(at 49.53 157.48 0)
+			(effects
+				(font
+					(size 1.27 1.27)
+				)
+				(hide yes)
+			)
+		)
+		(property "Datasheet" ""
+			(at 49.53 157.48 0)
+			(effects
+				(font
+					(size 1.27 1.27)
+				)
+				(hide yes)
+			)
+		)
+		(property "Description" ""
+			(at 49.53 157.48 0)
+			(effects
+				(font
+					(size 1.27 1.27)
+				)
+				(hide yes)
+			)
+		)
+		(pin "B7"
+		)
+		(pin "D6"
+		)
+		(pin "B8"
+		)
+		(pin "C6"
+		)
+		(pin "C8"
+		)
+		(pin "D5"
+		)
+		(pin "D7"
+		)
+		(pin "B3"
+		)
+		(pin "A3"
+		)
+		(pin "B2"
+		)
+		(pin "C2"
+		)
+		(pin "C3"
+		)
+		(pin "B4"
+		)
+		(pin "A4"
+		)
+		(pin "B5"
+		)
+		(pin "C5"
+		)
+		(pin "E5"
+		)
+		(pin "A5"
+		)
+		(pin "B1"
+		)
+		(pin "B6"
+		)
+		(pin "G4"
+		)
+		(pin "A6"
+		)
+		(pin "E7"
+		)
+		(pin "A7"
+		)
+		(pin "A8"
+		)
+		(pin "C2"
+		)
+		(pin "E2"
+		)
+		(pin "A3"
+		)
+		(pin "E8"
+		)
+		(pin "D4"
+		)
+		(pin "D2"
+		)
+		(pin "F2"
+		)
+		(instances
+			(project "t20-l431-som"
+				(path "/c9028163-a5a7-4e78-bba9-fb79df7846cd/bd86606c-2acb-477c-972b-5bc80fa54b47"
+					(reference "U4")
+					(unit 2)
+				)
+			)

Commit message: Continued initial layout
Other:
- moved on the sheet: U4B
Changed lines of the file:
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@@
 	(symbol
 		(lib_id "special-azonenberg:MODULE_INTERNAL_T20_L431_HOST")
-		(at 49.53 157.48 0)
+		(at 49.53 119.38 0)
 		(unit 2)
 		(exclude_from_sim no)
@@
 		(dnp no)
 		(property "Reference" "U4"
-			(at 49.53 158.8657 0)
+			(at 49.53 120.7657 0)
 			(effects
 				(font
@@
 		)
 		(property "Value" "MODULE_INTERNAL_T20_L431_HOST"
-			(at 49.53 161.29 0)
+			(at 49.53 123.19 0)
 			(effects
 				(font
@@
 		)
 		(property "Footprint" "azonenberg_pcb:MODULE_INTERNAL_T20_L431_HOST"
-			(at 49.53 157.48 0)
+			(at 49.53 119.38 0)
 			(effects
 				(font
@@
 		)
 		(property "Datasheet" ""
-			(at 49.53 157.48 0)
+			(at 49.53 119.38 0)
 			(effects
 				(font
@@
 		)
 		(property "Description" ""
-			(at 49.53 157.48 0)
+			(at 49.53 119.38 0)
 			(effects
 				(font
@@
 		(pin "F2"
 		)
+		(pin "F7"
+		)
+		(pin "G6"
+		)
+		(pin "D8"
+		)
+		(pin "E6"
+		)
+		(pin "G12"
+		)
+		(pin "E9"
+		)
+		(pin "F8"
+		)
+		(pin "G11"
+		)
+		(pin "J2"
+		)
+		(pin "G8"
+		)
+		(pin "F6"
+		)
+		(pin "G10"
+		)
+		(pin "F5"
+		)
+		(pin "C4"
+		)
+		(pin "K3"
+		)
+		(pin "H4"
+		)
+		(pin "H3"
+		)
+		(pin "H5"
+		)
+		(pin "J5"
+		)
+		(pin "J3"
+		)
+		(pin "J4"
+		)
+		(pin "J6"
+		)
+		(pin "H6"
+		)
+		(pin "H2"
+		)
+		(pin "F4"
+		)
+		(pin "G5"
+		)
+		(pin "H7"
+		)
+		(pin "N4"
+		)
+		(pin "G7"
+		)
+		(pin "G3"
+		)
+		(pin "K1"
+		)
+		(pin "N6"
+		)
+		(pin "L1"
+		)
+		(pin "J1"
+		)
+		(pin "N3"
+		)
+		(pin "H1"
+		)
+		(pin "G1"
+		)
+		(pin "G2"
+		)
 		(instances

Commit message: Added oscillator
Parts:
- added R6, R7: 10K, azonenberg_pcb:EIA_0201_RES_NOSILK, symbol device:R
Connections:
- net 1V8: now also R6.2, R7.2
- net FPGA_DONE: now also R7.1
- net FPGA_RESET_N: now also R6.1
Changed lines of the file:
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@@
 		)
+	)
+	(junction
+		(at 125.73 67.31)
+		(diameter 0)
+		(color 0 0 0 0)
 	)
 	(no_connect
@@
 		(at 45.72 87.63)
 	)
+	(wire
+		(pts
+			(xy 125.73 67.31) (xy 125.73 72.39)
+		)
+		(stroke
+			(width 0)
+			(type default)
+		)
+	)
+	(wire
+		(pts
+			(xy 125.73 62.23) (xy 125.73 67.31)
+		)
+		(stroke
+			(width 0)
+			(type default)
+		)
+	)
 	(label "FPGA_JTAG_TDI"
 		(at 45.72 39.37 180)
@@
 		)
 	)
+	(label "FPGA_DONE"
+		(at 118.11 62.23 180)
+		(effects
+			(font
+				(size 1.27 1.27)
+			)
+			(justify right bottom)
+		)
+	)
 	(label "FPGA_FLASH_DQ0"
 		(at 45.72 80.01 180)
@@
 	(label "FPGA_FLASH_DQ1"
 		(at 45.72 29.21 180)
+		(effects
+			(font
+				(size 1.27 1.27)
+			)
+			(justify right bottom)
+		)
+	)
+	(label "FPGA_RESET_N"
+		(at 118.11 72.39 180)
 		(effects
 			(font
@@
 	(symbol
 		(lib_id "device:R")
+		(at 121.92 72.39 90)
+		(unit 1)
+		(exclude_from_sim no)
+		(in_bom yes)
+		(on_board yes)
+		(dnp no)
+		(property "Reference" "R6"
+			(at 121.92 69.85 90)
+			(effects
+				(font
+					(size 1.27 1.27)
+				)
+			)
+		)
+		(property "Value" "10K"
+			(at 121.92 72.39 90)
+			(effects
+				(font
+					(size 1.27 1.27)
+				)
+			)
+		)
+		(property "Footprint" "azonenberg_pcb:EIA_0201_RES_NOSILK"
+			(at 121.92 74.168 90)
+			(effects
+				(font
+					(size 1.27 1.27)
+				)
+				(hide yes)
+			)
+		)
+		(property "Datasheet" ""
+			(at 121.92 72.39 0)
+			(effects
+				(font
+					(size 1.27 1.27)
+				)
+				(hide yes)
+			)
+		)
+		(property "Description" "Resistor"
+			(at 121.92 72.39 0)
+			(effects
+				(font
+					(size 1.27 1.27)
+				)
+				(hide yes)
+			)
+		)
+		(pin "1"
+		)
+		(pin "2"
+		)
+		(instances
+			(project "t20-l431-som"
+				(path "/c9028163-a5a7-4e78-bba9-fb79df7846cd/bd86606c-2acb-477c-972b-5bc80fa54b47"
+					(reference "R6")
+					(unit 1)
+				)
+			)
+		)
+	)
+	(symbol
+		(lib_id "device:R")
+		(at 121.92 62.23 90)
+		(unit 1)
+		(exclude_from_sim no)
+		(in_bom yes)
+		(on_board yes)
+		(dnp no)
+		(property "Reference" "R7"
+			(at 121.92 59.69 90)
+			(effects
+				(font
+					(size 1.27 1.27)
+				)
+			)
+		)
+		(property "Value" "10K"
+			(at 121.92 62.23 90)
+			(effects
+				(font
+					(size 1.27 1.27)
+				)
+			)
+		)
+		(property "Footprint" "azonenberg_pcb:EIA_0201_RES_NOSILK"
+			(at 121.92 64.008 90)
+			(effects
+				(font
+					(size 1.27 1.27)
+				)
+				(hide yes)
+			)
+		)
+		(property "Datasheet" ""
+			(at 121.92 62.23 0)
+			(effects
+				(font
+					(size 1.27 1.27)
+				)
+				(hide yes)
+			)
+		)
+		(property "Description" "Resistor"
+			(at 121.92 62.23 0)
+			(effects
+				(font
+					(size 1.27 1.27)
+				)
+				(hide yes)
+			)
+		)
+		(pin "1"
+		)
+		(pin "2"
+		)
+		(instances
+			(project "t20-l431-som"
+				(path "/c9028163-a5a7-4e78-bba9-fb79df7846cd/bd86606c-2acb-477c-972b-5bc80fa54b47"
+					(reference "R7")
+					(unit 1)
+				)
+			)
+		)
+	)
+	(symbol
+		(lib_id "device:R")
 		(at 121.92 67.31 90)
 		(unit 1)
@@
 		(pin "R1"
 		)
+		(pin "K8"
+		)
+		(pin "J7"
+		)
+		(pin "L7"
+		)
+		(pin "N7"
+		)
+		(pin "P7"
+		)
+		(pin "M7"
+		)
+		(pin "M7"
+		)
+		(pin "P5"
+		)
+		(pin "R5"
+		)
+		(pin "R4"
+		)
+		(pin "R7"
+		)
+		(pin "P6"
+		)
+		(pin "R6"
+		)
+		(pin "N8"
+		)
+		(pin "R8"
+		)
+		(pin "P8"
+		)
+		(pin "P9"
+		)
+		(pin "R9"
+		)
+		(pin "M8"
+		)
+		(pin "J12"
+		)
+		(pin "L12"
+		)
 		(instances
