File: t20-l431-carrier/t20-l431-carrier.kicad_sch (KiCad schematic)
At the start: 39 parts, among them J1 XILINX_JTAG, J2 CORTEX_DEBUG_ETM, J3 CONN_01X02, J4 PMOD_HOST, J5 PMOD_HOST, J6 PMOD_HOST, J7 PMOD_HOST, M10 LOGO, M7 LOGO, M8 LOGO, M9 LOGO, U1 MODULE_INTERNAL_T20_L431_CARR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, U7 ECS-1612MV-250-CN

Commit message: Began top right corner fanout
Connections:
- net FPGA_PMOD0_DQ3: now also U1.A7 (GPIOL_12_CDI2); no longer U1.E7 (GPIOR_117_CTRL14)
- net FPGA_PMOD0_DQ7: now also U1.A8 (GPIOL_13_CDI3); no longer U1.G5 (GPIOR_78_EXTFB0_CDI31)
- net FPGA_PMOD1_DQ0: now also U1.E9 (GPIOR_155); no longer U1.E8 (GPIOR_154)
- net FPGA_PMOD1_DQ1: now also U1.F7 (GPIOR_133_CDI18); no longer U1.E9 (GPIOR_155)
- net FPGA_PMOD1_DQ2: now also U1.E7 (GPIOR_117_CTRL14); no longer U1.F7 (GPIOR_133_CDI18)
- net FPGA_PMOD1_DQ3: now also U1.G5 (GPIOR_78_EXTFB0_CDI31); no longer U1.G7 (GPIOR_132_CDI19)
- net FPGA_PMOD1_DQ5: now also U1.E8 (GPIOR_154); no longer U1.A7 (GPIOL_12_CDI2)
- net FPGA_PMOD1_DQ6: now also U1.G7 (GPIOR_132_CDI19); no longer U1.A8 (GPIOL_13_CDI3)
Changed lines of the file:
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@@
 	)
 	(label "FPGA_PMOD0_DQ3"
-		(at 99.06 193.04 180)
+		(at 99.06 175.26 180)
 		(effects
 			(font
@@
 	)
 	(label "FPGA_PMOD0_DQ7"
-		(at 99.06 208.28 180)
+		(at 99.06 177.8 180)
 		(effects
 			(font
@@
 	)
 	(label "FPGA_PMOD1_DQ2"
-		(at 99.06 223.52 180)
+		(at 99.06 193.04 180)
 		(effects
 			(font
@@
 	)
 	(label "FPGA_PMOD1_DQ0"
-		(at 99.06 218.44 180)
+		(at 99.06 220.98 180)
 		(effects
 			(font
@@
 	)
 	(label "FPGA_PMOD1_DQ6"
-		(at 99.06 177.8 180)
+		(at 99.06 226.06 180)
 		(effects
 			(font
@@
 	)
 	(label "FPGA_PMOD1_DQ3"
-		(at 99.06 226.06 180)
+		(at 99.06 208.28 180)
 		(effects
 			(font
@@
 	)
 	(label "FPGA_PMOD1_DQ5"
-		(at 99.06 175.26 180)
+		(at 99.06 218.44 180)
 		(effects
 			(font
@@
 	)
 	(label "FPGA_PMOD1_DQ1"
-		(at 99.06 220.98 180)
-		(effects
-			(font
+		(at 99.06 223.52 180)
+		(effects
+			(font

Commit message: Continued routing t20/l431 test board
Connections:
- net FPGA_PMOD1_DQ2: now also U1.G5 (GPIOR_78_EXTFB0_CDI31); no longer U1.E7 (GPIOR_117_CTRL14)
- net FPGA_PMOD1_DQ3: now also U1.E7 (GPIOR_117_CTRL14); no longer U1.G5 (GPIOR_78_EXTFB0_CDI31)
- net MCU_PMOD1_DQ0: now also U1.H7 (PC8); no longer U1.H6 (PB0)
- net MCU_PMOD1_DQ1: now also U1.L7 (PC9); no longer U1.N6 (PC11)
- net MCU_PMOD1_DQ2: now also U1.R9 (PC12); no longer U1.J5 (PB2)
- net MCU_PMOD1_DQ3: now also U1.R7 (PB5); no longer U1.P5 (PB4)
- net MCU_PMOD1_DQ4: now also U1.K8 (PA8); no longer U1.R7 (PB5)
- net MCU_PMOD1_DQ5: now also U1.M8 (PC4); no longer U1.R5 (PB6)
- net MCU_PMOD1_DQ6: now also U1.R8 (PD2); no longer U1.R4 (PB8)
- net MCU_PMOD1_DQ7: now also U1.R5 (PB6); no longer U1.G6 (PB11)
- no-connect marks 27 -> 28
Changed lines of the file:
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@@
-	)
-	(no_connect
-		(at 38.1 248.92)
-	)
-	(no_connect
-		(at 99.06 86.36)
 	)
 	(no_connect
@@
 	)
 	(no_connect
-		(at 99.06 91.44)
-	)
-	(no_connect
 		(at 38.1 209.55)
 	)
 	(no_connect
-		(at 99.06 93.98)
-	)
-	(no_connect
 		(at 186.69 88.9)
 	)
@@
 	)
 	(no_connect
+		(at 99.06 118.11)
+	)
+	(no_connect
 		(at 38.1 246.38)
 	)
@@
 	)
 	(no_connect
+		(at 99.06 99.06)
+	)
+	(no_connect
 		(at 38.1 241.3)
 	)
 	(no_connect
+		(at 99.06 123.19)
+	)
+	(no_connect
 		(at 99.06 140.97)
 	)
 	(no_connect
+		(at 99.06 135.89)
+	)
+	(no_connect
+		(at 99.06 143.51)
+	)
+	(no_connect
+		(at 166.37 102.87)
+	)
+	(no_connect
 		(at 186.69 91.44)
 	)
@@
 	)
 	(no_connect
+		(at 99.06 125.73)
+	)
+	(no_connect
 		(at 99.06 138.43)
 	)
 	(no_connect
-		(at 99.06 101.6)
-	)
-	(no_connect
 		(at 38.1 243.84)
 	)
@@
 	(no_connect
 		(at 99.06 162.56)
-	)
-	(no_connect
-		(at 38.1 220.98)
 	)
 	(no_connect
@@
 	)
 	(label "MCU_PMOD1_DQ6"
-		(at 99.06 135.89 180)
+		(at 38.1 220.98 180)
 		(effects
 			(font
@@
 	)
 	(label "MCU_PMOD1_DQ0"
-		(at 99.06 118.11 180)
+		(at 99.06 91.44 180)
 		(effects
 			(font
@@
 	)
 	(label "MCU_PMOD1_DQ7"
-		(at 99.06 143.51 180)
+		(at 99.06 130.81 180)
 		(effects
 			(font
@@
 	)
 	(label "FPGA_PMOD1_DQ2"
-		(at 99.06 193.04 180)
+		(at 99.06 208.28 180)
 		(effects
 			(font
@@
 	)
 	(label "MCU_PMOD1_DQ4"
-		(at 99.06 128.27 180)
+		(at 38.1 248.92 180)
 		(effects
 			(font
@@
 	)
 	(label "MCU_PMOD1_DQ5"
-		(at 99.06 130.81 180)
+		(at 99.06 86.36 180)
 		(effects
 			(font
@@
 	)
 	(label "FPGA_PMOD1_DQ3"
-		(at 99.06 208.28 180)
+		(at 99.06 193.04 180)
 		(effects
 			(font
@@
 	)
 	(label "MCU_PMOD1_DQ3"
-		(at 99.06 125.73 180)
+		(at 99.06 128.27 180)
 		(effects
 			(font
@@
 	)
 	(label "MCU_PMOD1_DQ2"
-		(at 99.06 123.19 180)
+		(at 99.06 101.6 180)
 		(effects
 			(font
@@
 	)
 	(label "MCU_PMOD1_DQ1"
-		(at 99.06 99.06 180)
-		(effects
-			(font
+		(at 99.06 93.98 180)
+		(effects
+			(font
