File: t20-l431-carrier/t20-l431-carrier.kicad_pcb (KiCad board)
At the start: 4 copper layers, 57 x 60 mm, 60 parts, among them J1 XILINX_JTAG, J14 USB_C_Receptacle_USB2.0, J2 CORTEX_DEBUG_ETM, J3 CONN_01X02, J4 PMOD_HOST, J5 PMOD_HOST, J6 PMOD_HOST, J7 PMOD_HOST, M10 LOGO, M7 LOGO, M8 LOGO, M9 LOGO, U1 MODULE_INTERNAL_T20_L431_CARR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, U2 FT234XD, U3 LDO1117-33, U39 NCP45525IMNTWG-H, U7 ECS-1612MV-250-CN

Commit message: Began top right corner fanout
Parts:
- moved TP19 67.8 mm to (50.0, 55.5)
- moved U3 38.5 mm to (76.5, 64.2)
- moved C13 32.7 mm to (76.5, 71.8)
- moved C12 32.7 mm to (76.5, 70.0)
- moved TP18 21.1 mm to (84.5, 92.0)
Connections:
- U1 pad A7: /FPGA_PMOD1_DQ5 -> /FPGA_PMOD0_DQ3
- U1 pad A8: /FPGA_PMOD1_DQ6 -> /FPGA_PMOD0_DQ7
- U1 pad E7: /FPGA_PMOD0_DQ3 -> /FPGA_PMOD1_DQ2
- U1 pad E8: /FPGA_PMOD1_DQ0 -> /FPGA_PMOD1_DQ5
- U1 pad E9: /FPGA_PMOD1_DQ1 -> /FPGA_PMOD1_DQ0
- U1 pad F7: /FPGA_PMOD1_DQ2 -> /FPGA_PMOD1_DQ1
- U1 pad G5: /FPGA_PMOD0_DQ7 -> /FPGA_PMOD1_DQ3
- U1 pad G7: /FPGA_PMOD1_DQ3 -> /FPGA_PMOD1_DQ6
Routing:
- net /FPGA_PMOD1_DQ6: track 1.90 -> 32.7 mm
- net /FPGA_PMOD1_DQ5: track 1.90 -> 29.1 mm
- net /FPGA_PMOD1_DQ1: track 2.97 -> 28.3 mm
- net /FPGA_PMOD1_DQ4: track 3.67 -> 26.5 mm
- net /FPGA_PMOD1_DQ0: track 3.77 -> 23.9 mm
- net /MCU_PMOD1_DQ2: track 0.00 -> 6.17 mm, vias 0 -> 1
- net /GND: track 292.5 -> 298.1 mm, vias 91 -> 92
- net /MCU_PMOD1_DQ0: track 0.00 -> 5.57 mm, vias 0 -> 1
- net /MCU_PMOD1_DQ7: track 0.00 -> 5.27 mm, vias 0 -> 1
- net /FPGA_PMOD0_DQ7: track 17.4 -> 21.7 mm
- net /1V8: track 34.9 -> 37.0 mm
- net /FPGA_JTAG_TDI: track 2.87 -> 4.70 mm
- net /FPGA_JTAG_TDO: track 2.87 -> 4.47 mm, vias 0 -> 1
- net /FPGA_PMOD1_DQ3: track 4.77 -> 6.17 mm, vias 0 -> 1
- net /FPGA_PMOD0_DQ3: track 19.9 -> 18.9 mm, vias 1 -> 0
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
Commit message: Continued routing t20/l431 test board
Parts:
- moved C4 46.4 mm to (77.0, 90.8)
- moved C10 46.2 mm to (68.2, 90.2)
- moved C11 42.8 mm to (66.4, 78.0), turned to 180 degrees
- moved C9 42.1 mm to (67.0, 73.6), turned to 180 degrees
- moved C7 37.2 mm to (79.8, 85.8), turned to 90 degrees
- moved C8 32.3 mm to (81.0, 81.0)
- moved C6 22.8 mm to (88.2, 70.9)
- moved C5 22.8 mm to (88.2, 69.1)
- moved R29 2.99 mm to (65.2, 76.5), turned to 180 degrees
- moved C12 2.52 mm to (79.0, 70.2), turned to -90 degrees
- moved C13 1.50 mm to (76.5, 70.2), turned to -90 degrees
- moved U7 1.29 mm to (64.2, 75.2), turned to -90 degrees
- moved C61 1.27 mm to (62.8, 75.2), turned to -90 degrees
Connections:
- U1 pad E7: /FPGA_PMOD1_DQ2 -> /FPGA_PMOD1_DQ3
- U1 pad G5: /FPGA_PMOD1_DQ3 -> /FPGA_PMOD1_DQ2
- U1 pad G6: /MCU_PMOD1_DQ7 -> unconnected-(U1G-PB11-PadG6)
- U1 pad H6: /MCU_PMOD1_DQ0 -> unconnected-(U1G-PB0-PadH6)
- U1 pad H7: unconnected-(U1H-PC8-PadH7) -> /MCU_PMOD1_DQ0
- U1 pad J5: /MCU_PMOD1_DQ2 -> unconnected-(U1G-PB2-PadJ5)
- U1 pad K8: unconnected-(U1F-PA8-PadK8) -> /MCU_PMOD1_DQ4
- U1 pad L7: unconnected-(U1H-PC9-PadL7) -> /MCU_PMOD1_DQ1
- U1 pad M8: unconnected-(U1H-PC4-PadM8) -> /MCU_PMOD1_DQ5
- U1 pad N6: /MCU_PMOD1_DQ1 -> unconnected-(U1H-PC11-PadN6)
- U1 pad P5: /MCU_PMOD1_DQ3 -> unconnected-(U1G-PB4-PadP5)
- U1 pad R4: /MCU_PMOD1_DQ6 -> unconnected-(U1G-PB8-PadR4)
- U1 pad R5: /MCU_PMOD1_DQ5 -> /MCU_PMOD1_DQ7
- U1 pad R7: /MCU_PMOD1_DQ4 -> /MCU_PMOD1_DQ3
- U1 pad R8: unconnected-(U1J-PD2-PadR8) -> /MCU_PMOD1_DQ6
- U1 pad R9: unconnected-(U1H-PC12-PadR9) -> /MCU_PMOD1_DQ2
Routing:
- net /GND: track 298.1 -> 348.9 mm, vias 92 -> 106
- net /FPGA_JTAG_TDI: track 4.70 -> 37.4 mm, vias 0 -> 1
- net /FPGA_JTAG_TDO: track 4.47 -> 36.2 mm
- net /FPGA_PMOD1_DQ7: track 5.27 -> 36.2 mm
- net /FPGA_JTAG_TMS: track 4.57 -> 34.9 mm
- net /FPGA_JTAG_TCK: track 3.77 -> 33.9 mm, vias 0 -> 1
- net /FPGA_PMOD1_DQ2: track 4.47 -> 34.1 mm
- net /3V3: track 189.8 -> 217.1 mm, vias 13 -> 20
- net /FPGA_PMOD1_DQ3: track 6.17 -> 32.4 mm
- net /MCU_PMOD1_DQ6: track 0.80 -> 24.9 mm
- net /MCU_PMOD1_DQ7: track 5.27 -> 29.1 mm, vias 1 -> 0
- net /MCU_PMOD1_DQ4: track 0.90 -> 24.1 mm
- net /MCU_PMOD1_DQ5: track 0.70 -> 23.8 mm
- net /USB-UART and PSU/VBUS: track 10.4 -> 33.2 mm, vias 4 -> 7
- net /MCU_PMOD1_DQ1: track 0.00 -> 21.7 mm
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
Commit message: Updated t20-l431-carrier design
Parts:
- moved C5 27.6 mm to (70.2, 90.0), turned to -90 degrees
- moved C6 16.4 mm to (81.2, 85.8), turned to 90 degrees
Routing:
- net /3V3: track 217.1 -> 219.8 mm, vias 20 -> 22
- net /GND: track 348.9 -> 350.5 mm, vias 106 -> 108
- net /2V5: track 5.86 -> 6.87 mm
- net /MCU_PMOD0_DQ3: track 16.4 -> 15.6 mm
- net Net-(U2-TXD): track 7.64 -> 6.93 mm, vias 1 -> 0
- net Net-(U2-RXD): vias 1 -> 0
- added copper zone on In2.Cu, net /1V2
- added copper zone on In2.Cu, net /1V8
- added copper zone on In2.Cu, net /2V5
- added copper zone on In2.Cu, net /3V3
- added copper zone on In2.Cu, net /3V3_FPGA
- added copper zone on In1.Cu, net /GND
- added copper zone on In2.Cu, net /USB-UART and PSU/VBUS

Commit message: Updated silkscreen text with connector labels
Other:
- board text added: "FPGA PMOD0"
- board text added: "FPGA PMOD1"
- board text added: "MCU PMOD0"
- board text added: "MCU PMOD1"
- board text added: "STM32L431 / T20 SoM Bringup Carrier A. Zonenberg / v0.1 2026-10-22"
Changed lines of the file:
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@@
 		(layer "Edge.Cuts")
+	)
+	(gr_text "STM32L431 / T20 SoM\nBringup Carrier\nA. Zonenberg / v0.1\n2026-10-22"
+		(at 82.25 97.5 0)
+		(layer "F.SilkS")
+		(effects
+			(font
+				(size 0.75 0.75)
+				(thickness 0.1)
+			)
+			(justify left)
+		)
+	)
+	(gr_text "MCU\nPMOD0"
+		(at 52.5 74.25 0)
+		(layer "F.SilkS")
+		(effects
+			(font
+				(size 0.75 0.75)
+				(thickness 0.1)
+			)
+		)
+	)
+	(gr_text "FPGA\nPMOD0"
+		(at 55.25 58.5 0)
+		(layer "F.SilkS")
+		(effects
+			(font
+				(size 0.75 0.75)
+				(thickness 0.1)
+			)
+		)
 	)
 	(gr_text "MCU\nBOOT0"
@@
 		(layer "F.SilkS")
 		(effects
+			(font
+				(size 0.75 0.75)
+				(thickness 0.1)
+			)
+		)
+	)
+	(gr_text "MCU\nPMOD1"
+		(at 94.75 74.25 0)
+		(layer "F.SilkS")
+		(effects
+			(font
+				(size 0.75 0.75)
+				(thickness 0.1)
+			)
+		)
+	)
+	(gr_text "FPGA\nPMOD1"
+		(at 98.5 58.5 0)
+		(layer "F.SilkS")
+		(effects
