File: process-test-0402/process-test-0402.kicad_pcb (KiCad board)
At the start: 4 copper layers, 107.5 x 115.5 mm, 203 parts

Commit message: Updated silkscreen layout on 0402 test board
Parts:
- added M1: MECHANICAL, azonenberg_pcb:LONGTHING-1200DPI, F.Cu at (120.0, 127.5)
- added M2: MECHANICAL, w_logo:Logo_silk_OSHW_6x6mm, F.Cu at (103.0, 128.0)
- added M3: MECHANICAL, w_logo:Logo_silk_WEEE_3.4x5mm, F.Cu at (110.0, 128.5)
- moved R1 3.00 mm to (33.0, 30.0)
- moved R10 3.00 mm to (34.5, 69.5)
- moved R100 3.00 mm to (74.5, 119.5)
- moved R101 3.00 mm to (83.0, 30.0)
- moved R102 3.00 mm to (84.5, 29.5)
- moved R103 3.00 mm to (83.0, 40.0)
- moved R104 3.00 mm to (84.5, 39.5)
- moved R105 3.00 mm to (83.0, 50.0)
- moved R106 3.00 mm to (84.5, 49.5)
- moved R107 3.00 mm to (83.0, 60.0)
- moved R108 3.00 mm to (84.5, 59.5)
- moved R109 3.00 mm to (83.0, 70.0)
- moved R11 3.00 mm to (33.0, 80.0)
- moved R110 3.00 mm to (84.5, 69.5)
- moved R111 3.00 mm to (83.0, 80.0)
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Other:
- board size 107.5 x 115.5 mm -> 108 x 115.5 mm
- board text added: "0402 Reflow / Thermal Imbalance / Placement Testbed A. Zonenberg / v0.1 / 2026-10-24"

Commit message: Added more 0402 process test variants
Routing:
- added copper zone on In1.Cu, net /GND
- added copper zone on In2.Cu, net /GND
Other:
- rule pad_to_mask_clearance: 0 -> 0.05
- board text added: "0402 Reflow / Thermal Imbalance / Placement Testbed A. Zonenberg / v0.1 / 2026-10-25"
- board text removed: "0402 Reflow / Thermal Imbalance / Placement Testbed A. Zonenberg / v0.1 / 2026-10-24"
Changed lines of the file:
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@@
 			(dielectric_constraints no)
 		)
-		(pad_to_mask_clearance 0)
+		(pad_to_mask_clearance 0.05)
 		(allow_soldermask_bridges_in_footprints no)
 		(tenting front back)
@@
 			(outputformat 1)
 			(mirror no)
-			(drillshape 1)
+			(drillshape 0)
 			(scaleselection 1)
-			(outputdirectory "")
+			(outputdirectory "output/")
 		)
 	)
@@
 		(layer "Edge.Cuts")
 	)
-	(gr_text "0402 Reflow / Thermal Imbalance / Placement Testbed\nA. Zonenberg / v0.1 / 2026-10-24"
+	(gr_text "0402 Reflow / Thermal Imbalance / Placement Testbed\nA. Zonenberg / v0.1 / 2026-10-25"
 		(at 32.5 131 0)
 		(layer "F.SilkS")
@@
 		(net 1)
 	)
+	(zone
+		(net 1)
+		(net_name "/GND")
+		(layers "In1.Cu" "In2.Cu")
+		(hatch edge 0.5)
+		(connect_pads yes
+			(clearance 0.125)
+		)
+		(min_thickness 0.125)
+		(filled_areas_thickness no)
+		(fill yes
+			(thermal_gap 0.5)
+			(thermal_bridge_width 0.5)
+		)
+		(polygon
+			(pts
+				(xy 25.5 17.5) (xy 25.5 132) (xy 132.5 132) (xy 132.5 17.5)
+			)
+		)
+	)
 	(embedded_fonts no)
